File: scan-controller-kicad/_autosave-scan-controller-kicad.kicad_sch (KiCad schematic)
At the start: 103 parts, among them J1 24-30VDC, J10 Motor, J11 Raspi GPIO, J12 Raspi UART, J13 ICSP, J14 FTDI, J2 KSQ In, J3 Shaft Eye, J4 Shaft Eye, J5 Film End Eye, J6 LED, J7 LED, J8 Fan, J9 Film End Eye, Q2 BC817, Q3 BC848, Q4 DMMT5401, Q5 DMG2305UX, Q6 IRF7470, SW1 Power, SW10 Reset, SW2 <, SW3 <<, SW4 Lamp, SW5 Zoom, SW6 REC, SW7 >>, SW8 >, SW9 Stop, U1 74LVC14, U2 QRE1113, U3 QRE1113, U4 LM2576HVS-5, U5 DRV8871DDA, U6 ATmega328P, Y1 8MHz

Commit message: Initial PCB
Other:
- note removed: "Footprint!"
Changed lines of the file:
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@@
-    (effects (font (size 1.27 1.27)) (justify left bottom))
-  )
-  (text "Footprint!" (at 48.895 139.065 0)
     (effects (font (size 1.27 1.27)) (justify left bottom))
   )
