File: scan-controller-kicad/scan-controller-kicad.kicad_sch (KiCad schematic)
At the start: 32 parts, among them CN1 24V in, J1 Raspi GPIO, J2 Raspi UART, J3 ICSP, J4 FTDI, Q1 IRLML2502, Q2 IRLML6402, SW1 Reset, U1 ATmega328P, Y1 8MHz

Commit message: Starting routing
Parts:
- added C6: 100n, Capacitor_SMD:C_0805_2012Metric, symbol Device:C_Small
- renumbered C6 to C7, C7 to C8, C8 to C9
Connections:
- net 3.3V-uC: now also C6.1
- net GND: now also C6.2
Changed lines of the file:
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@@
   (junction (at 108.585 94.615) (diameter 0) (color 0 0 0 0)
   )
+  (junction (at 178.435 66.04) (diameter 0) (color 0 0 0 0)
+  )
   (junction (at 45.72 23.495) (diameter 0) (color 0 0 0 0)
   )
@@
   )
   (junction (at 110.49 130.175) (diameter 0) (color 0 0 0 0)
+  )
+  (junction (at 188.595 58.42) (diameter 0) (color 0 0 0 0)
   )
   (junction (at 113.665 89.535) (diameter 0) (color 0 0 0 0)
@@
     (stroke (width 0) (type default))
   )
-  (wire (pts (xy 188.595 60.96) (xy 188.595 66.04))
+  (wire (pts (xy 188.595 58.42) (xy 188.595 66.04))
     (stroke (width 0) (type default))
   )
@@
     (stroke (width 0) (type default))
   )
+  (wire (pts (xy 188.595 45.72) (xy 188.595 58.42))
+    (stroke (width 0) (type default))
+  )
   (wire (pts (xy 155.575 95.25) (xy 151.765 95.25))
     (stroke (width 0) (type default))
@@
     (stroke (width 0) (type default))
   )
+  (wire (pts (xy 184.785 58.42) (xy 188.595 58.42))
+    (stroke (width 0) (type default))
+  )
   (wire (pts (xy 95.885 104.775) (xy 93.98 104.775))
     (stroke (width 0) (type default))
@@
     (stroke (width 0) (type default))
   )
+  (wire (pts (xy 178.435 58.42) (xy 179.705 58.42))
+    (stroke (width 0) (type default))
+  )
   (wire (pts (xy 41.91 41.275) (xy 26.67 41.275))
     (stroke (width 0) (type default))
@@
   )
   (wire (pts (xy 86.995 140.335) (xy 89.535 140.335))
+    (stroke (width 0) (type default))
+  )
+  (wire (pts (xy 178.435 58.42) (xy 178.435 66.04))
     (stroke (width 0) (type default))
   )
@@
     )
   )
-  (global_label "3.3V-uC" (shape input) (at 188.595 60.96 180) (fields_autoplaced)
+  (global_label "3.3V-uC" (shape input) (at 188.595 45.72 180) (fields_autoplaced)
     (effects (font (size 1.27 1.27)) (justify right))
-    (property "Intersheetrefs" "${INTERSHEET_REFS}" (at 177.506 60.96 0)
+    (property "Intersheetrefs" "${INTERSHEET_REFS}" (at 177.506 45.72 0)
       (effects (font (size 1.27 1.27)) (justify right) hide)
     )
@@
   (symbol (lib_id "Device:C_Small") (at 211.455 80.01 0) (mirror y) (unit 1)
     (in_bom yes) (on_board yes) (dnp no)
-    (property "Reference" "C7" (at 211.455 77.47 0)
+    (property "Reference" "C8" (at 211.455 77.47 0)
       (effects (font (size 1.27 1.27)) (justify right))
     )
@@
       (project "scan-controller-kicad"
         (path "/ab6dbce1-4ecf-44ae-8f33-5f07e4f43ca9"
-          (reference "C7") (unit 1)
+          (reference "C8") (unit 1)
         )
       )
@@
   (symbol (lib_id "Device:C_Small") (at 217.17 111.125 270) (unit 1)
     (in_bom yes) (on_board yes) (dnp no)
-    (property "Reference" "C8" (at 215.9 113.665 90)
+    (property "Reference" "C9" (at 215.9 113.665 90)
       (effects (font (size 1.27 1.27)) (justify right))
     )
@@
       (project "scan-controller-kicad"
         (path "/ab6dbce1-4ecf-44ae-8f33-5f07e4f43ca9"
-          (reference "C8") (unit 1)
+          (reference "C9") (unit 1)
         )
       )
@@
   (symbol (lib_id "Device:C_Small") (at 182.245 66.04 270) (mirror x) (unit 1)
     (in_bom yes) (on_board yes) (dnp no)
-    (property "Reference" "C6" (at 183.515 64.77 90)
-      (effects (font (size 1.27 1.27)) (justify left))
-    )
-    (property "Value" "100n" (at 175.895 64.77 90)
+    (property "Reference" "C7" (at 183.515 64.77 90)
+      (effects (font (size 1.27 1.27)) (justify left))
+    )
+    (property "Value" "100n" (at 179.07 62.865 90)
       (effects (font (size 1.27 1.27)) (justify left))
     )
@@
       (project "scan-controller-kicad"
         (path "/ab6dbce1-4ecf-44ae-8f33-5f07e4f43ca9"
-          (reference "C6") (unit 1)
+          (reference "C7") (unit 1)
         )
       )
@@
         )
       )
+    )
+  )
+  (symbol (lib_id "Device:C_Small") (at 182.245 58.42 270) (mirror x) (unit 1)
+    (in_bom yes) (on_board yes) (dnp no)
+    (property "Reference" "C6" (at 184.15 57.15 90)
+      (effects (font (size 1.27 1.27)) (justify left))
+    )
+    (property "Value" "100n" (at 179.07 55.245 90)
+      (effects (font (size 1.27 1.27)) (justify left))
+    )
+    (property "Footprint" "Capacitor_SMD:C_0805_2012Metric" (at 182.245 58.42 0)
+      (effects (font (size 1.27 1.27)) hide)
+    )
+    (property "Datasheet" "https://datasheet.lcsc.com/lcsc/2304140030_Samsung-Electro-Mechanics-CL21B104KCFNNNE_C28233.pdf" (at 182.245 58.42 0)
+      (effects (font (size 1.27 1.27)) hide)
+    )
+    (property "LCSC" "C28233" (at 182.245 58.42 0)
+      (effects (font (size 1.27 1.27)) hide)
+    )
+    (property "Inventory" "B" (at 182.245 58.42 0)
+      (effects (font (size 1.27 1.27)) hide)
+    )
+    (pin "1")
+    (pin "2")
+    (instances
+      (project "scan-controller-kicad"
+        (path "/ab6dbce1-4ecf-44ae-8f33-5f07e4f43ca9"
+          (reference "C6") (unit 1)
+        )
+      )
