File: scan-controller-kicad/scan-controller-kicad.kicad_sch (KiCad schematic)
At the start: 34 parts, among them CN1 24V in, J1 Raspi GPIO, J2 Raspi UART, J3 ICSP, J4 FTDI, Q1 IRLML2502, Q2 IRLML6402, SW1 Reset, U1 ATmega328P, Y1 8MHz

Commit message: Pushbutton PTHs now mechanical (DRC fun)
Connections:
- net 24VAC-1: now reaches CN1.1, D1.3
- net 24VAC-2: now reaches CN1.2, D1.4
Changed lines of the file:
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@@
     (effects (font (size 1.27 1.27)) (justify left bottom))
+  )
+  (label "24VAC-2" (at 26.67 41.275 270) (fields_autoplaced)
+    (effects (font (size 1.27 1.27)) (justify right bottom))
   )
   (label "D6" (at 169.545 135.89 180) (fields_autoplaced)
@@
     (effects (font (size 1.27 1.27)) (justify left bottom))
   )
+  (label "24VAC-1" (at 26.67 31.115 90) (fields_autoplaced)
+    (effects (font (size 1.27 1.27)) (justify left bottom))
+  )

Commit message: Adding a switch for Storage Target
Parts:
- removed TP5: GPIO17, TestPoint:TestPoint_THTPad_1.0x1.0mm_Drill0.5mm, symbol Connector:TestPoint
Connections:
- net GPIO17: now reaches J1.11 (Pin_11)
Other:
- sheet User Interface ports: added Storage Target; removed none
Changed lines of the file:
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@@
+    (stroke (width 0) (type default))
+  )
+  (wire (pts (xy 52.705 106.045) (xy 54.61 106.045))
     (stroke (width 0) (type default))
   )
@@
     (effects (font (size 1.27 1.27)) (justify right bottom))
   )
+  (label "GPIO17" (at 86.995 107.315 180) (fields_autoplaced)
+    (effects (font (size 1.27 1.27)) (justify right bottom))
+  )
   (label "A1" (at 169.545 102.87 180) (fields_autoplaced)
     (effects (font (size 1.27 1.27)) (justify right bottom))
@@
   (label "A0" (at 169.545 100.33 180) (fields_autoplaced)
     (effects (font (size 1.27 1.27)) (justify right bottom))
+  )
+  (label "GPIO17" (at 54.61 106.045 0) (fields_autoplaced)
+    (effects (font (size 1.27 1.27)) (justify left bottom))
   )
   (label "MISO" (at 113.03 107.315 0) (fields_autoplaced)
@@
     )
   )
-  (symbol (lib_id "Connector:TestPoint") (at 86.995 107.315 90) (unit 1)
-    (in_bom yes) (on_board yes) (dnp no)
-    (property "Reference" "TP5" (at 87.63 111.76 90)
-      (effects (font (size 1.27 1.27)) (justify left) hide)
-    )
-    (property "Value" "GPIO17" (at 81.915 107.315 90)
-      (effects (font (size 1.27 1.27)) (justify left))
-    )
-    (property "Footprint" "TestPoint:TestPoint_THTPad_1.0x1.0mm_Drill0.5mm" (at 86.995 102.235 0)
-      (effects (font (size 1.27 1.27)) hide)
-    )
-    (property "Datasheet" "~" (at 86.995 102.235 0)
-      (effects (font (size 1.27 1.27)) hide)
-    )
-    (property "LCSC" "" (at 86.995 107.315 0)
-      (effects (font (size 1.27 1.27)) hide)
-    )
-    (property "Inventory" "" (at 86.995 107.315 0)
-      (effects (font (size 1.27 1.27)) hide)
-    )
-    (pin "1")
-    (instances
-      (project "scan-controller-kicad"
-        (path "/ab6dbce1-4ecf-44ae-8f33-5f07e4f43ca9"
-          (reference "TP5") (unit 1)
-        )
-      )
-    )
-  )
   (symbol (lib_id "power:GNDD") (at 125.095 70.485 0) (unit 1)
     (in_bom yes) (on_board yes) (dnp no)
@@
       (effects (font (size 1.27 1.27)) (justify right))
     )
+    (pin "Storage Target" input (at 52.705 106.045 0)
+      (effects (font (size 1.27 1.27)) (justify right))
+    )

Commit message: Fixing BOM
Parts:
- J1: Inventory E -> (none); LCSC C35165 -> (none)
- J2, J3, J4, TP1, TP2, TP3, TP4, TP6, TP7, TP8, TP9: now left out of the parts list
- Q1: LCSC C5364308 -> C347503
Changed lines of the file:
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@@
   )
   (symbol (lib_id "Connector_Generic:Conn_01x06") (at 226.06 103.505 0) (unit 1)
-    (in_bom yes) (on_board yes) (dnp no)
+    (in_bom no) (on_board yes) (dnp no)
     (property "Reference" "J4" (at 228.092 103.7082 0)
       (effects (font (size 1.27 1.27)) (justify left))
@@
   )
   (symbol (lib_id "Connector:TestPoint") (at 48.26 23.495 0) (unit 1)
-    (in_bom yes) (on_board yes) (dnp no)
+    (in_bom no) (on_board yes) (dnp no)
     (property "Reference" "TP1" (at 46.99 15.24 0)
       (effects (font (size 1.27 1.27)) (justify left))
@@
   )
   (symbol (lib_id "Connector:AVR-ISP-6") (at 220.98 135.255 0) (mirror y) (unit 1)
-    (in_bom yes) (on_board yes) (dnp no)
+    (in_bom no) (on_board yes) (dnp no)
     (property "Reference" "J3" (at 229.362 132.8166 0)
       (effects (font (size 1.27 1.27)) (justify right))
@@
   )
   (symbol (lib_id "Connector:TestPoint") (at 85.725 132.715 90) (unit 1)
-    (in_bom yes) (on_board yes) (dnp no)
+    (in_bom no) (on_board yes) (dnp no)
     (property "Reference" "TP4" (at 85.09 133.985 90)
       (effects (font (size 1.27 1.27)))
@@
       (effects (font (size 1.27 1.27)) hide)
     )
-    (property "LCSC" "C35165" (at 100.965 117.475 0)
-      (effects (font (size 1.27 1.27)) hide)
-    )
-    (property "Inventory" "E" (at 100.965 117.475 0)
+    (property "LCSC" "" (at 100.965 117.475 0)
+      (effects (font (size 1.27 1.27)) hide)
+    )
+    (property "Inventory" "" (at 100.965 117.475 0)
       (effects (font (size 1.27 1.27)) hide)
     )
@@
   )
   (symbol (lib_id "Connector:TestPoint") (at 85.725 130.175 90) (unit 1)
-    (in_bom yes) (on_board yes) (dnp no)
+    (in_bom no) (on_board yes) (dnp no)
     (property "Reference" "TP3" (at 85.09 128.905 90)
       (effects (font (size 1.27 1.27)))
@@
   )
   (symbol (lib_id "Connector:TestPoint") (at 203.835 85.09 270) (mirror x) (unit 1)
-    (in_bom yes) (on_board yes) (dnp no)
+    (in_bom no) (on_board yes) (dnp no)
     (property "Reference" "TP9" (at 203.2 89.535 90)
       (effects (font (size 1.27 1.27)) (justify left))
@@
   )
   (symbol (lib_id "Connector:TestPoint") (at 86.995 109.855 90) (unit 1)
-    (in_bom yes) (on_board yes) (dnp no)
+    (in_bom no) (on_board yes) (dnp no)
     (property "Reference" "TP6" (at 87.63 114.3 90)
       (effects (font (size 1.27 1.27)) (justify left) hide)
@@
   )
   (symbol (lib_id "Connector:TestPoint") (at 168.91 138.43 90) (mirror x) (unit 1)
-    (in_bom yes) (on_board yes) (dnp no)
+    (in_bom no) (on_board yes) (dnp no)
     (property "Reference" "TP8" (at 167.005 140.335 90)
       (effects (font (size 1.27 1.27)) (justify left) hide)
@@
   )
   (symbol (lib_id "Connector:TestPoint") (at 167.005 82.55 90) (mirror x) (unit 1)
-    (in_bom yes) (on_board yes) (dnp no)
+    (in_bom no) (on_board yes) (dnp no)
     (property "Reference" "TP7" (at 165.1 84.455 90)
       (effects (font (size 1.27 1.27)) (justify left) hide)
@@
   )
   (symbol (lib_id "Connector:TestPoint") (at 54.61 41.275 180) (unit 1)
-    (in_bom yes) (on_board yes) (dnp no)
+    (in_bom no) (on_board yes) (dnp no)
     (property "Reference" "TP2" (at 55.88 49.53 0)
       (effects (font (size 1.27 1.27)) (justify left) hide)
@@
       (effects (font (size 1.27 1.27)) (justify left) hide)
     )
-    (property "LCSC" "C5364308" (at 130.175 59.055 0)
+    (property "LCSC" "C347503" (at 130.175 59.055 0)
       (effects (font (size 1.27 1.27)) hide)
     )
@@
   )
   (symbol (lib_id "Connector_Generic:Conn_01x02") (at 120.65 102.235 0) (unit 1)
-    (in_bom yes) (on_board yes) (dnp no)
+    (in_bom no) (on_board yes) (dnp no)
     (property "Reference" "J2" (at 120.015 107.95 0)
       (effects (font (size 1.27 1.27)) (justify left))

Commit message: Connect PGIO with SCL (instead of SDA) for power. Connect Atmega SDA to bus (was nc)
Other:
- note added: "D2 ist zu hell Kamerakabel-Schlitz? TP umbenennen oder entfernen"
Changed lines of the file:
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@@
     (stroke (width 0) (type default))
+  )
+  (text "D2 ist zu hell\nKamerakabel-Schlitz?\nTP umbenennen oder entfernen"
+    (at 222.885 27.305 0)
+    (effects (font (size 1.27 1.27)) (justify left bottom))
   )
   (label "GNDD" (at 57.15 42.545 0) (fields_autoplaced)

Commit message: Fixing I2C Conns. Power Button still broken
Connections:
- net SCL: now also J1.37 (Pin_37)
- net GPIO26 renamed SDA
- net SDA: no longer J1.37 (Pin_37)
Other:
- note added: "(Underscore placed to keep the Net called SCL)"
- note added: "D2 ist zu hell Kamerakabel-Schlitz? TP umbenennen oder entfernen I2c fixen Power switch fixen Add I2C TPs"
- note removed: "D2 ist zu hell Kamerakabel-Schlitz? TP umbenennen oder entfernen"
Changed lines of the file:
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@@
   (junction (at 138.43 43.815) (diameter 0) (color 0 0 0 0)
   )
+  (junction (at 89.535 99.695) (diameter 0) (color 0 0 0 0)
+  )
   (junction (at 92.075 94.615) (diameter 0) (color 0 0 0 0)
   )
   (junction (at 188.595 66.04) (diameter 0) (color 0 0 0 0)
-  )
-  (junction (at 89.535 97.155) (diameter 0) (color 0 0 0 0)
   )
   (junction (at 164.465 97.79) (diameter 0) (color 0 0 0 0)
@@
     (stroke (width 0) (type default))
   )
-  (wire (pts (xy 85.725 99.695) (xy 95.885 99.695))
+  (wire (pts (xy 85.725 99.695) (xy 89.535 99.695))
     (stroke (width 0) (type default))
   )
@@
     (stroke (width 0) (type default))
   )
-  (wire (pts (xy 89.535 97.155) (xy 95.885 97.155))
+  (wire (pts (xy 85.725 97.155) (xy 95.885 97.155))
     (stroke (width 0) (type default))
   )
@@
     (stroke (width 0) (type default))
   )
-  (wire (pts (xy 89.535 97.155) (xy 89.535 140.335))
+  (wire (pts (xy 89.535 99.695) (xy 89.535 140.335))
     (stroke (width 0) (type default))
   )
@@
     (stroke (width 0) (type default))
   )
+  (wire (pts (xy 89.535 99.695) (xy 95.885 99.695))
+    (stroke (width 0) (type default))
+  )
   (wire (pts (xy 34.29 38.735) (xy 48.26 38.735))
     (stroke (width 0) (type default))
@@
     (stroke (width 0) (type default))
   )
-  (wire (pts (xy 85.725 97.155) (xy 89.535 97.155))
-    (stroke (width 0) (type default))
-  )
   (wire (pts (xy 86.995 140.335) (xy 89.535 140.335))
     (stroke (width 0) (type default))
@@
     (stroke (width 0) (type default))
   )
-  (text "D2 ist zu hell\nKamerakabel-Schlitz?\nTP umbenennen oder entfernen"
+  (text "(Underscore placed to \nkeep the Net called SCL)" (at 71.755 144.145 0)
+    (effects (font (size 1 1)) (justify left bottom))
+  )
+  (text "D2 ist zu hell\nKamerakabel-Schlitz?\nTP umbenennen oder entfernen\nI2c fixen\nPower switch fixen\nAdd I2C TPs"
     (at 222.885 27.305 0)
     (effects (font (size 1.27 1.27)) (justify left bottom))
@@
     (effects (font (size 1.27 1.27)) (justify right bottom))
   )
-  (label "GPIO26" (at 54.61 75.565 0) (fields_autoplaced)
+  (label "_GPIO26" (at 54.61 75.565 0) (fields_autoplaced)
     (effects (font (size 1.27 1.27)) (justify left bottom))
   )
@@
     (effects (font (size 1.27 1.27)) (justify right bottom))
   )
-  (label "GPIO26" (at 86.995 140.335 180) (fields_autoplaced)
-    (effects (font (size 1.27 1.27)) (justify right bottom))
-  )
+  (label "_GPIO26" (at 86.995 140.335 180) (fields_autoplaced)
+    (effects (font (size 1.27 1.27)) (justify right bottom))
+  )

Commit message: Reduced Power LED Brightness (0.3 mA @ 2.2V, wow), FIxed Power Switch Footprint
Other:
- note added: "~(D2 ist zu hell) Kamerakabel-Schlitz? TP umbenennen oder entfernen ~(I2c fixen) ~(Power switch fixen) Add I2C TPs Target Schalter größer?"
- note removed: "D2 ist zu hell Kamerakabel-Schlitz? TP umbenennen oder entfernen I2c fixen Power switch fixen Add I2C TPs"
Changed lines of the file:
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@@
     (effects (font (size 1 1)) (justify left bottom))
   )
-  (text "D2 ist zu hell\nKamerakabel-Schlitz?\nTP umbenennen oder entfernen\nI2c fixen\nPower switch fixen\nAdd I2C TPs"
-    (at 222.885 27.305 0)
+  (text "~(D2 ist zu hell)\nKamerakabel-Schlitz?\nTP umbenennen oder entfernen\n~(I2c fixen)\n~(Power switch fixen)\nAdd I2C TPs\nTarget Schalter größer?"
+    (at 217.17 40.005 0)
     (effects (font (size 1.27 1.27)) (justify left bottom))
   )

Commit message: Flip U6, it broke the KSQ
Other:
- note added: "~(D2 ist zu hell) ~(U6 flippen) Kamerakabel-Schlitz? TP umbenennen oder entfernen ~(I2c fixen) ~(Power switch fixen) Add I2C TPs Target Schalter größer?"
- note removed: "~(D2 ist zu hell) Kamerakabel-Schlitz? TP umbenennen oder entfernen ~(I2c fixen) ~(Power switch fixen) Add I2C TPs Target Schalter größer?"
Changed lines of the file:
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@@
     (effects (font (size 1 1)) (justify left bottom))
   )
-  (text "~(D2 ist zu hell)\nKamerakabel-Schlitz?\nTP umbenennen oder entfernen\n~(I2c fixen)\n~(Power switch fixen)\nAdd I2C TPs\nTarget Schalter größer?"
+  (text "~(D2 ist zu hell)\n~(U6 flippen)\nKamerakabel-Schlitz?\nTP umbenennen oder entfernen\n~(I2c fixen)\n~(Power switch fixen)\nAdd I2C TPs\nTarget Schalter größer?"
     (at 217.17 40.005 0)
     (effects (font (size 1.27 1.27)) (justify left bottom))

Commit message: Updating Todos
Other:
- note added: "Kamerakabel-Schlitz? TP umbenennen oder entfernen Add I2C TPs Target Schalter größer? FTDI Masse kennzeichnen Exp/Current prüfen KSQ LEDs nötig?"
- note removed: "~(D2 ist zu hell) ~(U6 flippen) Kamerakabel-Schlitz? TP umbenennen oder entfernen ~(I2c fixen) ~(Power switch fixen) Add I2C TPs Target Schalter größer?"
Changed lines of the file:
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@@
     (effects (font (size 1 1)) (justify left bottom))
   )
-  (text "~(D2 ist zu hell)\n~(U6 flippen)\nKamerakabel-Schlitz?\nTP umbenennen oder entfernen\n~(I2c fixen)\n~(Power switch fixen)\nAdd I2C TPs\nTarget Schalter größer?"
+  (text "Kamerakabel-Schlitz?\nTP umbenennen oder entfernen\nAdd I2C TPs\nTarget Schalter größer?\nFTDI Masse kennzeichnen\nExp/Current prüfen\nKSQ LEDs nötig?"
     (at 217.17 40.005 0)
     (effects (font (size 1.27 1.27)) (justify left bottom))
