File: scan-controller-kicad/scan-controller-kicad.kicad_sch (KiCad schematic)
At the start: 33 parts, among them CN1 24V in, J1 Raspi GPIO, J2 Raspi UART, J3 ICSP, J4 FTDI, Q1 IRLML2502, Q2 IRLML6402, SW1 Reset, U1 ATmega328P, Y1 8MHz

Commit message: Add the missing BJP Transistor for the shaft eye
Other:
- note added: "eKamerakabel-Schlitz? TP umbenennen oder entfernen TPs mit Löchern (i2c zumindest) Add I2C TPs Target Schalter größer? FTDI Masse kennzeichnen Exp/Current prüfen KSQ LEDs nötig? Shaft LED als Einbauhilfe Eye-Connectoren spiegeln (GND!) Transistor am Shaft Eye ergänzen Taster durch SMD ersetzen"
- note removed: "Kamerakabel-Schlitz? TP umbenennen oder entfernen Add I2C TPs Target Schalter größer? FTDI Masse kennzeichnen Exp/Current prüfen KSQ LEDs nötig?"
Changed lines of the file:
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@@
     (effects (font (size 1 1)) (justify left bottom))
   )
-  (text "Kamerakabel-Schlitz?\nTP umbenennen oder entfernen\nAdd I2C TPs\nTarget Schalter größer?\nFTDI Masse kennzeichnen\nExp/Current prüfen\nKSQ LEDs nötig?"
+  (text "eKamerakabel-Schlitz?\nTP umbenennen oder entfernen\nTPs mit Löchern (i2c zumindest)\nAdd I2C TPs\nTarget Schalter größer?\nFTDI Masse kennzeichnen\nExp/Current prüfen\nKSQ LEDs nötig?\nShaft LED als Einbauhilfe\nEye-Connectoren spiegeln (GND!)\nTransistor am Shaft Eye ergänzen\nTaster durch SMD ersetzen"
     (at 217.17 40.005 0)
     (effects (font (size 1.27 1.27)) (justify left bottom))

Commit message: Freeing up D4 (328) as it isn't needed
Other:
- sheet Sensors ports: added Film End LED; removed Film End
- note added: "eKamerakabel-Schlitz? TP umbenennen oder entfernen https://forum.kicad.info/t/answer-how-to-avoid-annotate-adding-number-but-still-label-pcb/38283/17 TPs mit Löchern (i2c zumindest) Add I2C TPs Target Schalter größer? FTDI Masse kennzeichnen Exp/Current prüfen KSQ LEDs nötig? Shaft LED als Einbauhilfe Eye-Connectoren spiegeln (GND!) Transistor am Shaft Eye ergänzen Taster durch SMD ersetzen"
- note removed: "eKamerakabel-Schlitz? TP umbenennen oder entfernen TPs mit Löchern (i2c zumindest) Add I2C TPs Target Schalter größer? FTDI Masse kennzeichnen Exp/Current prüfen KSQ LEDs nötig? Shaft LED als Einbauhilfe Eye-Connectoren spiegeln (GND!) Transistor am Shaft Eye ergänzen Taster durch SMD ersetzen"
Changed lines of the file:
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@@
     (stroke (width 0) (type default))
   )
-  (wire (pts (xy 52.705 132.08) (xy 54.61 132.08))
+  (wire (pts (xy 52.705 131.445) (xy 54.61 131.445))
     (stroke (width 0) (type default))
   )
@@
     (effects (font (size 1 1)) (justify left bottom))
   )
-  (text "eKamerakabel-Schlitz?\nTP umbenennen oder entfernen\nTPs mit Löchern (i2c zumindest)\nAdd I2C TPs\nTarget Schalter größer?\nFTDI Masse kennzeichnen\nExp/Current prüfen\nKSQ LEDs nötig?\nShaft LED als Einbauhilfe\nEye-Connectoren spiegeln (GND!)\nTransistor am Shaft Eye ergänzen\nTaster durch SMD ersetzen"
-    (at 217.17 40.005 0)
+  (text "eKamerakabel-Schlitz?\nTP umbenennen oder entfernen\nhttps://forum.kicad.info/t/answer-how-to-avoid-annotate-adding-number-but-still-label-pcb/38283/17\nTPs mit Löchern (i2c zumindest)\nAdd I2C TPs\nTarget Schalter größer?\nFTDI Masse kennzeichnen\nExp/Current prüfen\nKSQ LEDs nötig?\nShaft LED als Einbauhilfe\nEye-Connectoren spiegeln (GND!)\nTransistor am Shaft Eye ergänzen\nTaster durch SMD ersetzen"
+    (at 59.69 189.865 0)
     (effects (font (size 1.27 1.27)) (justify left bottom))
   )
@@
     (effects (font (size 1.27 1.27)) (justify left bottom))
   )
-  (label "D4" (at 54.61 100.965 0) (fields_autoplaced)
-    (effects (font (size 1.27 1.27)) (justify left bottom))
-  )
   (label "SCL" (at 85.725 99.695 180) (fields_autoplaced)
     (effects (font (size 1.27 1.27)) (justify right bottom))
@@
     (effects (font (size 1.27 1.27)) (justify right bottom))
   )
+  (label "D3" (at 54.61 100.965 0) (fields_autoplaced)
+    (effects (font (size 1.27 1.27)) (justify left bottom))
+  )
   (label "~{RST}" (at 209.55 137.795 180) (fields_autoplaced)
     (effects (font (size 1.27 1.27)) (justify right bottom))
@@
     (effects (font (size 1.27 1.27)) (justify left bottom))
   )
-  (label "D3" (at 54.61 132.08 0) (fields_autoplaced)
+  (label "D3" (at 54.61 131.445 0) (fields_autoplaced)
     (effects (font (size 1.27 1.27)) (justify left bottom))
   )
@@
       (effects (font (size 1.27 1.27)) (justify right))
     )
-    (pin "Film End" input (at 52.705 132.08 0)
+    (pin "Film End LED" input (at 52.705 131.445 0)
       (effects (font (size 1.27 1.27)) (justify right))
     )

Commit message: Improved the TP Symbol/Footprint
Parts:
- TP3: footprint TestPoint:TestPoint_THTPad_1.0x1.0mm_Drill0.5mm -> Peacemans_Footprints:TestPoint_THTPad_1.5x1.5mm_Drill0.7mm_named; symbol Connector:TestPoint -> Peacemans_Teile:TestPoint_named; TP_Label (none) -> GPIO5; now in the parts list
- TP4: footprint TestPoint:TestPoint_THTPad_1.0x1.0mm_Drill0.5mm -> Peacemans_Footprints:TestPoint_THTPad_1.5x1.5mm_Drill0.7mm_named; symbol Connector:TestPoint -> Peacemans_Teile:TestPoint_named; TP_Label (none) -> GPIO6; now in the parts list
Changed lines of the file:
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@@
     )
   )
-  (symbol (lib_id "Connector:TestPoint") (at 85.725 132.715 90) (unit 1)
-    (in_bom no) (on_board yes) (dnp no)
+  (symbol (lib_id "Peacemans_Teile:TestPoint_named") (at 85.725 132.715 90) (unit 1)
+    (in_bom yes) (on_board yes) (dnp no)
     (property "Reference" "TP4" (at 85.09 133.985 90)
       (effects (font (size 1.27 1.27)))
@@
       (effects (font (size 1.27 1.27)))
     )
-    (property "Footprint" "TestPoint:TestPoint_THTPad_1.0x1.0mm_Drill0.5mm" (at 85.725 127.635 0)
+    (property "Footprint" "Peacemans_Footprints:TestPoint_THTPad_1.5x1.5mm_Drill0.7mm_named" (at 85.725 127.635 0)
       (effects (font (size 1.27 1.27)) hide)
     )
@@
       (effects (font (size 1.27 1.27)) hide)
     )
-    (property "LCSC" "" (at 85.725 132.715 0)
-      (effects (font (size 1.27 1.27)) hide)
-    )
-    (property "Inventory" "" (at 85.725 132.715 0)
-      (effects (font (size 1.27 1.27)) hide)
+    (property "TP_Label" "GPIO6" (at 81.28 135.255 90)
+      (effects (font (size 1.27 1.27)))
     )
     (pin "1")
@@
     )
   )
-  (symbol (lib_id "Connector:TestPoint") (at 85.725 130.175 90) (unit 1)
-    (in_bom no) (on_board yes) (dnp no)
+  (symbol (lib_id "Peacemans_Teile:TestPoint_named") (at 85.725 130.175 90) (unit 1)
+    (in_bom yes) (on_board yes) (dnp no)
     (property "Reference" "TP3" (at 85.09 128.905 90)
       (effects (font (size 1.27 1.27)))
@@
       (effects (font (size 1.27 1.27)))
     )
-    (property "Footprint" "TestPoint:TestPoint_THTPad_1.0x1.0mm_Drill0.5mm" (at 85.725 125.095 0)
+    (property "Footprint" "Peacemans_Footprints:TestPoint_THTPad_1.5x1.5mm_Drill0.7mm_named" (at 85.725 125.095 0)
       (effects (font (size 1.27 1.27)) hide)
     )
@@
       (effects (font (size 1.27 1.27)) hide)
     )
-    (pin "1")
+    (property "TP_Label" "GPIO5" (at 83.185 126.365 90)
+      (effects (font (size 1.27 1.27)))
+    )
+    (pin "1")

Commit message: TPs renamed (using https://forum.kicad.info/t/answer-how-to-avoid-annotate-adding-number-but-still-label-pcb/38283/17)
Parts:
- TP1: footprint TestPoint:TestPoint_THTPad_2.0x2.0mm_Drill1.0mm -> Peacemans_Footprints:TestPoint_THTPad_1.5x1.5mm_Drill0.7mm_named; symbol Connector:TestPoint -> Peacemans_Teile:TestPoint_named; TP_Label (none) -> 24VDC; now in the parts list
- TP2: footprint TestPoint:TestPoint_THTPad_2.0x2.0mm_Drill1.0mm -> Peacemans_Footprints:TestPoint_THTPad_1.5x1.5mm_Drill0.7mm_named; symbol Connector:TestPoint -> Peacemans_Teile:TestPoint_named; TP_Label (none) -> GND; now in the parts list
- TP6: footprint TestPoint:TestPoint_THTPad_1.0x1.0mm_Drill0.5mm -> Peacemans_Footprints:TestPoint_THTPad_1.5x1.5mm_Drill0.7mm_named; symbol Connector:TestPoint -> Peacemans_Teile:TestPoint_named; TP_Label (none) -> GPIO27; now in the parts list
- TP7: footprint TestPoint:TestPoint_THTPad_1.5x1.5mm_Drill0.7mm -> Peacemans_Footprints:TestPoint_THTPad_1.5x1.5mm_Drill0.7mm_named; symbol Connector:TestPoint -> Peacemans_Teile:TestPoint_named; TP_Label (none) -> D10; now in the parts list
- TP8: footprint TestPoint:TestPoint_THTPad_1.5x1.5mm_Drill0.7mm -> Peacemans_Footprints:TestPoint_THTPad_1.5x1.5mm_Drill0.7mm_named; symbol Connector:TestPoint -> Peacemans_Teile:TestPoint_named; TP_Label (none) -> D7; now in the parts list
- TP9: footprint TestPoint:TestPoint_THTPad_1.5x1.5mm_Drill0.7mm -> Peacemans_Footprints:TestPoint_THTPad_1.5x1.5mm_Drill0.7mm_named; symbol Connector:TestPoint -> Peacemans_Teile:TestPoint_named; TP_Label (none) -> A7; now in the parts list
Changed lines of the file:
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@@
     )
   )
-  (symbol (lib_id "Connector:TestPoint") (at 48.26 23.495 0) (unit 1)
-    (in_bom no) (on_board yes) (dnp no)
-    (property "Reference" "TP1" (at 46.99 15.24 0)
+  (symbol (lib_id "Peacemans_Teile:TestPoint_named") (at 48.26 23.495 0) (unit 1)
+    (in_bom yes) (on_board yes) (dnp no)
+    (property "Reference" "TP1" (at 46.355 16.51 0)
       (effects (font (size 1.27 1.27)) (justify left))
     )
     (property "Value" "24V" (at 46.99 17.78 0)
-      (effects (font (size 1.27 1.27)) (justify left))
-    )
-    (property "Footprint" "TestPoint:TestPoint_THTPad_2.0x2.0mm_Drill1.0mm" (at 53.34 23.495 0)
+      (effects (font (size 1.27 1.27)) (justify left) hide)
+    )
+    (property "Footprint" "Peacemans_Footprints:TestPoint_THTPad_1.5x1.5mm_Drill0.7mm_named" (at 53.34 23.495 0)
       (effects (font (size 1.27 1.27)) hide)
     )
@@
       (effects (font (size 1.27 1.27)) hide)
     )
-    (property "LCSC" "" (at 48.26 23.495 0)
-      (effects (font (size 1.27 1.27)) hide)
-    )
-    (property "Inventory" "" (at 48.26 23.495 0)
-      (effects (font (size 1.27 1.27)) hide)
+    (property "TP_Label" "24VDC" (at 48.26 18.415 0)
+      (effects (font (size 1.27 1.27)))
     )
     (pin "1")
@@
     )
     (property "Value" "GPIO6" (at 76.2 132.715 90)
-      (effects (font (size 1.27 1.27)))
+      (effects (font (size 1.27 1.27)) hide)
     )
     (property "Footprint" "Peacemans_Footprints:TestPoint_THTPad_1.5x1.5mm_Drill0.7mm_named" (at 85.725 127.635 0)
@@
       (effects (font (size 1.27 1.27)) hide)
     )
-    (property "TP_Label" "GPIO6" (at 81.28 135.255 90)
+    (property "TP_Label" "GPIO6" (at 78.105 132.715 90)
       (effects (font (size 1.27 1.27)))
     )
@@
     )
     (property "Value" "GPIO5" (at 76.2 130.175 90)
-      (effects (font (size 1.27 1.27)))
+      (effects (font (size 1.27 1.27)) hide)
     )
     (property "Footprint" "Peacemans_Footprints:TestPoint_THTPad_1.5x1.5mm_Drill0.7mm_named" (at 85.725 125.095 0)
@@
       (effects (font (size 1.27 1.27)) hide)
     )
-    (property "TP_Label" "GPIO5" (at 83.185 126.365 90)
+    (property "TP_Label" "GPIO5" (at 78.105 130.175 90)
       (effects (font (size 1.27 1.27)))
     )
@@
     )
   )
-  (symbol (lib_id "Connector:TestPoint") (at 203.835 85.09 270) (mirror x) (unit 1)
-    (in_bom no) (on_board yes) (dnp no)
+  (symbol (lib_id "Peacemans_Teile:TestPoint_named") (at 203.835 85.09 270) (mirror x) (unit 1)
+    (in_bom yes) (on_board yes) (dnp no)
     (property "Reference" "TP9" (at 203.2 89.535 90)
       (effects (font (size 1.27 1.27)) (justify left))
@@
       (effects (font (size 1.27 1.27)) (justify left))
     )
-    (property "Footprint" "TestPoint:TestPoint_THTPad_1.5x1.5mm_Drill0.7mm" (at 203.835 80.01 0)
+    (property "Footprint" "Peacemans_Footprints:TestPoint_THTPad_1.5x1.5mm_Drill0.7mm_named" (at 203.835 80.01 0)
       (effects (font (size 1.27 1.27)) hide)
     )
@@
       (effects (font (size 1.27 1.27)) hide)
     )
-    (property "LCSC" "" (at 203.835 85.09 0)
-      (effects (font (size 1.27 1.27)) hide)
-    )
-    (property "Inventory" "" (at 203.835 85.09 0)
-      (effects (font (size 1.27 1.27)) hide)
+    (property "TP_Label" "A7" (at 203.835 85.09 0)
+      (effects (font (size 1.27 1.27)))
     )
     (pin "1")
@@
     )
   )
-  (symbol (lib_id "Connector:TestPoint") (at 86.995 109.855 90) (unit 1)
-    (in_bom no) (on_board yes) (dnp no)
+  (symbol (lib_id "Peacemans_Teile:TestPoint_named") (at 86.995 109.855 90) (unit 1)
+    (in_bom yes) (on_board yes) (dnp no)
     (property "Reference" "TP6" (at 87.63 114.3 90)
       (effects (font (size 1.27 1.27)) (justify left) hide)
@@
       (effects (font (size 1.27 1.27)) (justify left))
     )
-    (property "Footprint" "TestPoint:TestPoint_THTPad_1.0x1.0mm_Drill0.5mm" (at 86.995 104.775 0)
+    (property "Footprint" "Peacemans_Footprints:TestPoint_THTPad_1.5x1.5mm_Drill0.7mm_named" (at 86.995 104.775 0)
       (effects (font (size 1.27 1.27)) hide)
     )
@@
       (effects (font (size 1.27 1.27)) hide)
     )
-    (property "LCSC" "" (at 86.995 109.855 0)
-      (effects (font (size 1.27 1.27)) hide)
-    )
-    (property "Inventory" "" (at 86.995 109.855 0)
-      (effects (font (size 1.27 1.27)) hide)
+    (property "TP_Label" "GPIO27" (at 86.995 109.855 0)
+      (effects (font (size 1.27 1.27)))
     )
     (pin "1")
@@
     )
   )
-  (symbol (lib_id "Connector:TestPoint") (at 168.91 138.43 90) (mirror x) (unit 1)
-    (in_bom no) (on_board yes) (dnp no)
+  (symbol (lib_id "Peacemans_Teile:TestPoint_named") (at 168.91 138.43 90) (mirror x) (unit 1)
+    (in_bom yes) (on_board yes) (dnp no)
     (property "Reference" "TP8" (at 167.005 140.335 90)
       (effects (font (size 1.27 1.27)) (justify left) hide)
@@
       (effects (font (size 1.27 1.27)) (justify left))
     )
-    (property "Footprint" "TestPoint:TestPoint_THTPad_1.5x1.5mm_Drill0.7mm" (at 168.91 143.51 0)
+    (property "Footprint" "Peacemans_Footprints:TestPoint_THTPad_1.5x1.5mm_Drill0.7mm_named" (at 168.91 143.51 0)
       (effects (font (size 1.27 1.27)) hide)
     )
@@
       (effects (font (size 1.27 1.27)) hide)
     )
-    (property "LCSC" "" (at 168.91 138.43 0)
-      (effects (font (size 1.27 1.27)) hide)
-    )
-    (property "Inventory" "" (at 168.91 138.43 0)
-      (effects (font (size 1.27 1.27)) hide)
+    (property "TP_Label" "D7" (at 168.91 138.43 0)
+      (effects (font (size 1.27 1.27)))
     )
     (pin "1")
@@
     )
   )
-  (symbol (lib_id "Connector:TestPoint") (at 167.005 82.55 90) (mirror x) (unit 1)
-    (in_bom no) (on_board yes) (dnp no)
+  (symbol (lib_id "Peacemans_Teile:TestPoint_named") (at 167.005 82.55 90) (mirror x) (unit 1)
+    (in_bom yes) (on_board yes) (dnp no)
     (property "Reference" "TP7" (at 165.1 84.455 90)
       (effects (font (size 1.27 1.27)) (justify left) hide)
@@
       (effects (font (size 1.27 1.27)) (justify left))
     )
-    (property "Footprint" "TestPoint:TestPoint_THTPad_1.5x1.5mm_Drill0.7mm" (at 167.005 87.63 0)
+    (property "Footprint" "Peacemans_Footprints:TestPoint_THTPad_1.5x1.5mm_Drill0.7mm_named" (at 167.005 87.63 0)
       (effects (font (size 1.27 1.27)) hide)
     )
@@
       (effects (font (size 1.27 1.27)) hide)
     )
-    (property "LCSC" "" (at 167.005 82.55 0)
-      (effects (font (size 1.27 1.27)) hide)
-    )
-    (property "Inventory" "" (at 167.005 82.55 0)
-      (effects (font (size 1.27 1.27)) hide)
+    (property "TP_Label" "D10" (at 167.005 82.55 0)
+      (effects (font (size 1.27 1.27)))
     )
     (pin "1")
@@
     )
   )
-  (symbol (lib_id "Connector:TestPoint") (at 54.61 41.275 180) (unit 1)
-    (in_bom no) (on_board yes) (dnp no)
+  (symbol (lib_id "Peacemans_Teile:TestPoint_named") (at 54.61 41.275 180) (unit 1)
+    (in_bom yes) (on_board yes) (dnp no)
     (property "Reference" "TP2" (at 55.88 49.53 0)
       (effects (font (size 1.27 1.27)) (justify left) hide)
@@
       (effects (font (size 1.27 1.27)) (justify left))
     )
-    (property "Footprint" "TestPoint:TestPoint_THTPad_2.0x2.0mm_Drill1.0mm" (at 49.53 41.275 0)
+    (property "Footprint" "Peacemans_Footprints:TestPoint_THTPad_1.5x1.5mm_Drill0.7mm_named" (at 49.53 41.275 0)
       (effects (font (size 1.27 1.27)) hide)
     )
@@
       (effects (font (size 1.27 1.27)) hide)
     )
-    (property "LCSC" "" (at 54.61 41.275 0)
-      (effects (font (size 1.27 1.27)) hide)
-    )
-    (property "Inventory" "" (at 54.61 41.275 0)
-      (effects (font (size 1.27 1.27)) hide)
-    )
-    (pin "1")
+    (property "TP_Label" "GND" (at 54.61 41.275 0)
+      (effects (font (size 1.27 1.27)))
+    )
+    (pin "1")
