File: scan-controller-kicad/scan-controller-kicad.kicad_sch (KiCad schematic)
At the start: 33 parts, among them CN1 24V in, J1 Raspi GPIO, J2 Raspi UART, J3 ICSP, J4 FTDI, Q1 IRLML2502, Q2 IRLML6402, SW1 Reset, U1 ATmega328P, Y1 8MHz

Commit message: Replacing D6 LED with 1N4148 Adding TPs for Lamp Current Fixing TP Labels and other Labels Add LED D9 that actually reflects Lamp status Add control LEDs for Eyes (makes mounting much easier) Add mini manual and tech specs on the back side
Parts:
- added TP12, TP5: TestPoint, Peacemans_Footprints:TestPoint_THTPad_1.5x1.5mm_Drill0.7mm_named, symbol Peacemans_Teile:TestPoint_named
Connections:
- net SCL: now also TP12.1
- net SDA: now also TP5.1
Other:
- sheet Sensors ports: added Film End; removed Film End LED
- note added: "eKamerakabel-Schlitz? Target Schalter größer? FTDI Masse kennzeichnen Exp/Current prüfen KSQ LEDs nötig? Shaft LED als Einbauhilfe Taster durch SMD ersetzen"
- note removed: "eKamerakabel-Schlitz? TP umbenennen oder entfernen https://forum.kicad.info/t/answer-how-to-avoid-annotate-adding-number-but-still-label-pcb/38283/17 TPs mit Löchern (i2c zumindest) Add I2C TPs Target Schalter größer? FTDI Masse kennzeichnen Exp/Current prüfen KSQ LEDs nötig? Shaft LED als Einbauhilfe Eye-Connectoren spiegeln (GND!) Transistor am Shaft Eye ergänzen Taster durch SMD ersetzen"
Changed lines of the file:
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@@
   (junction (at 110.49 109.855) (diameter 0) (color 0 0 0 0)
+  )
+  (junction (at 86.995 99.695) (diameter 0) (color 0 0 0 0)
+  )
+  (junction (at 86.995 97.155) (diameter 0) (color 0 0 0 0)
   )
   (junction (at 125.095 43.815) (diameter 0) (color 0 0 0 0)
@@
     (stroke (width 0) (type default))
   )
-  (wire (pts (xy 85.725 99.695) (xy 89.535 99.695))
+  (wire (pts (xy 85.725 99.695) (xy 86.995 99.695))
     (stroke (width 0) (type default))
   )
@@
     (stroke (width 0) (type default))
   )
+  (wire (pts (xy 52.705 130.81) (xy 54.61 130.81))
+    (stroke (width 0) (type default))
+  )
   (wire (pts (xy 110.49 145.415) (xy 93.98 145.415))
     (stroke (width 0) (type default))
@@
     (stroke (width 0) (type default))
   )
-  (wire (pts (xy 52.705 131.445) (xy 54.61 131.445))
-    (stroke (width 0) (type default))
-  )
-  (wire (pts (xy 85.725 97.155) (xy 95.885 97.155))
+  (wire (pts (xy 85.725 97.155) (xy 86.995 97.155))
     (stroke (width 0) (type default))
   )
@@
     (stroke (width 0) (type default))
   )
+  (wire (pts (xy 86.995 99.695) (xy 89.535 99.695))
+    (stroke (width 0) (type default))
+  )
   (wire (pts (xy 57.15 41.275) (xy 57.15 42.545))
     (stroke (width 0) (type default))
@@
   )
   (wire (pts (xy 173.355 92.71) (xy 164.465 92.71))
+    (stroke (width 0) (type default))
+  )
+  (wire (pts (xy 86.995 97.155) (xy 95.885 97.155))
     (stroke (width 0) (type default))
   )
@@
     (effects (font (size 1 1)) (justify left bottom))
   )
-  (text "eKamerakabel-Schlitz?\nTP umbenennen oder entfernen\nhttps://forum.kicad.info/t/answer-how-to-avoid-annotate-adding-number-but-still-label-pcb/38283/17\nTPs mit Löchern (i2c zumindest)\nAdd I2C TPs\nTarget Schalter größer?\nFTDI Masse kennzeichnen\nExp/Current prüfen\nKSQ LEDs nötig?\nShaft LED als Einbauhilfe\nEye-Connectoren spiegeln (GND!)\nTransistor am Shaft Eye ergänzen\nTaster durch SMD ersetzen"
+  (text "eKamerakabel-Schlitz?\nTarget Schalter größer?\nFTDI Masse kennzeichnen\nExp/Current prüfen\nKSQ LEDs nötig?\nShaft LED als Einbauhilfe\nTaster durch SMD ersetzen"
     (at 59.69 189.865 0)
     (effects (font (size 1.27 1.27)) (justify left bottom))
@@
     (effects (font (size 1.27 1.27)) (justify left bottom))
   )
-  (label "D3" (at 54.61 131.445 0) (fields_autoplaced)
+  (label "D3" (at 54.61 130.81 0) (fields_autoplaced)
     (effects (font (size 1.27 1.27)) (justify left bottom))
   )
@@
         (path "/ab6dbce1-4ecf-44ae-8f33-5f07e4f43ca9"
           (reference "#PWR04") (unit 1)
+        )
+      )
+    )
+  )
+  (symbol (lib_id "Peacemans_Teile:TestPoint_named") (at 86.995 99.695 180) (unit 1)
+    (in_bom yes) (on_board yes) (dnp no)
+    (property "Reference" "TP12" (at 86.995 106.553 0)
+      (effects (font (size 1.27 1.27)) hide)
+    )
+    (property "Value" "TestPoint" (at 86.995 104.775 0)
+      (effects (font (size 1.27 1.27)) hide)
+    )
+    (property "Footprint" "Peacemans_Footprints:TestPoint_THTPad_1.5x1.5mm_Drill0.7mm_named" (at 81.915 99.695 0)
+      (effects (font (size 1.27 1.27)) hide)
+    )
+    (property "Datasheet" "~" (at 81.915 99.695 0)
+      (effects (font (size 1.27 1.27)) hide)
+    )
+    (property "TP_Label" "SCL" (at 83.82 102.87 0)
+      (effects (font (size 1.27 1.27)))
+    )
+    (pin "1")
+    (instances
+      (project "scan-controller-kicad"
+        (path "/ab6dbce1-4ecf-44ae-8f33-5f07e4f43ca9"
+          (reference "TP12") (unit 1)
         )
       )
@@
   (symbol (lib_id "Peacemans_Teile:TestPoint_named") (at 203.835 85.09 270) (mirror x) (unit 1)
     (in_bom yes) (on_board yes) (dnp no)
-    (property "Reference" "TP9" (at 203.2 89.535 90)
+    (property "Reference" "TP9" (at 203.835 86.995 90)
       (effects (font (size 1.27 1.27)) (justify left))
     )
     (property "Value" "A7" (at 203.835 86.995 90)
-      (effects (font (size 1.27 1.27)) (justify left))
+      (effects (font (size 1.27 1.27)) (justify left) hide)
     )
     (property "Footprint" "Peacemans_Footprints:TestPoint_THTPad_1.5x1.5mm_Drill0.7mm_named" (at 203.835 80.01 0)
@@
       (effects (font (size 1.27 1.27)) hide)
     )
-    (property "TP_Label" "A7" (at 203.835 85.09 0)
+    (property "TP_Label" "A7" (at 209.55 85.09 90)
       (effects (font (size 1.27 1.27)))
     )
@@
     )
     (property "Value" "GPIO27" (at 81.915 109.855 90)
-      (effects (font (size 1.27 1.27)) (justify left))
+      (effects (font (size 1.27 1.27)) (justify left) hide)
     )
     (property "Footprint" "Peacemans_Footprints:TestPoint_THTPad_1.5x1.5mm_Drill0.7mm_named" (at 86.995 104.775 0)
@@
       (effects (font (size 1.27 1.27)) hide)
     )
-    (property "TP_Label" "GPIO27" (at 86.995 109.855 0)
+    (property "TP_Label" "GPIO27" (at 78.74 109.855 90)
       (effects (font (size 1.27 1.27)))
     )
@@
     )
     (property "Value" "D7" (at 169.545 137.16 90)
-      (effects (font (size 1.27 1.27)) (justify left))
+      (effects (font (size 1.27 1.27)) (justify left) hide)
     )
     (property "Footprint" "Peacemans_Footprints:TestPoint_THTPad_1.5x1.5mm_Drill0.7mm_named" (at 168.91 143.51 0)
@@
       (effects (font (size 1.27 1.27)) hide)
     )
-    (property "TP_Label" "D7" (at 168.91 138.43 0)
+    (property "TP_Label" "D7" (at 163.195 138.43 90)
       (effects (font (size 1.27 1.27)))
     )
@@
     )
     (property "Value" "D10" (at 169.545 81.28 90)
-      (effects (font (size 1.27 1.27)) (justify left))
+      (effects (font (size 1.27 1.27)) (justify left) hide)
     )
     (property "Footprint" "Peacemans_Footprints:TestPoint_THTPad_1.5x1.5mm_Drill0.7mm_named" (at 167.005 87.63 0)
@@
       (effects (font (size 1.27 1.27)) hide)
     )
-    (property "TP_Label" "D10" (at 167.005 82.55 0)
+    (property "TP_Label" "D10" (at 160.655 82.55 90)
       (effects (font (size 1.27 1.27)))
     )
@@
         (path "/ab6dbce1-4ecf-44ae-8f33-5f07e4f43ca9"
           (reference "J2") (unit 1)
+        )
+      )
+    )
+  )
+  (symbol (lib_id "Peacemans_Teile:TestPoint_named") (at 86.995 97.155 0) (unit 1)
+    (in_bom yes) (on_board yes) (dnp no)
+    (property "Reference" "TP5" (at 86.995 90.297 0)
+      (effects (font (size 1.27 1.27)) hide)
+    )
+    (property "Value" "TestPoint" (at 86.995 92.075 0)
+      (effects (font (size 1.27 1.27)) hide)
+    )
+    (property "Footprint" "Peacemans_Footprints:TestPoint_THTPad_1.5x1.5mm_Drill0.7mm_named" (at 92.075 97.155 0)
+      (effects (font (size 1.27 1.27)) hide)
+    )
+    (property "Datasheet" "~" (at 92.075 97.155 0)
+      (effects (font (size 1.27 1.27)) hide)
+    )
+    (property "TP_Label" "SDA" (at 84.455 92.71 0)
+      (effects (font (size 1.27 1.27)))
+    )
+    (pin "1")
+    (instances
+      (project "scan-controller-kicad"
+        (path "/ab6dbce1-4ecf-44ae-8f33-5f07e4f43ca9"
+          (reference "TP5") (unit 1)
         )
       )
@@
       (effects (font (size 1.27 1.27)) (justify right))
     )
-    (pin "Film End LED" input (at 52.705 131.445 0)
+    (pin "Film End" input (at 52.705 130.81 0)
       (effects (font (size 1.27 1.27)) (justify right))
     )

Commit message: Last Version with the second OpAmp stilll in use
Connections:
- net D4: no longer names the net of U1.2 (PD4)
- no-connect marks 14 -> 15
Other:
- sheet User Interface ports: added none; removed Film End LED
Changed lines of the file:
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@@
   (junction (at 48.26 23.495) (diameter 0) (color 0 0 0 0)
   )
+  (no_connect (at 169.545 130.81))
   (no_connect (at 95.885 120.015))
   (no_connect (at 95.885 122.555))
@@
     (stroke (width 0) (type default))
   )
-  (wire (pts (xy 52.705 100.965) (xy 54.61 100.965))
-    (stroke (width 0) (type default))
-  )
   (wire (pts (xy 169.545 95.25) (xy 169.545 97.79))
     (stroke (width 0) (type default))
@@
     (effects (font (size 1.27 1.27)) (justify left bottom))
   )
-  (label "D4" (at 169.545 130.81 180) (fields_autoplaced)
-    (effects (font (size 1.27 1.27)) (justify right bottom))
-  )
   (label "D6" (at 243.84 85.09 180) (fields_autoplaced)
     (effects (font (size 1.27 1.27)) (justify right bottom))
-  )
-  (label "D3" (at 54.61 100.965 0) (fields_autoplaced)
-    (effects (font (size 1.27 1.27)) (justify left bottom))
   )
   (label "~{RST}" (at 209.55 137.795 180) (fields_autoplaced)
@@
       (effects (font (size 1.27 1.27)) (justify right))
     )
-    (pin "Film End LED" input (at 52.705 100.965 0)
-      (effects (font (size 1.27 1.27)) (justify right))
-    )

Commit message: DRC happy!
Changed lines of the file:
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@@
   (symbol (lib_id "Connector_Generic:Conn_01x02") (at 120.65 102.235 0) (unit 1)
     (in_bom no) (on_board yes) (dnp no)
-    (property "Reference" "J2" (at 120.015 107.95 0)
+    (property "Reference" "J2" (at 122.555 105.41 0)
       (effects (font (size 1.27 1.27)) (justify left))
     )

Commit message: Saving before renumbering refs
Parts:
- TP1: TP_Label 24VDC -> VDCext
Changed lines of the file:
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@@
       (effects (font (size 1.27 1.27)) hide)
     )
-    (property "TP_Label" "24VDC" (at 48.26 18.415 0)
+    (property "TP_Label" "VDCext" (at 48.26 18.415 0)
       (effects (font (size 1.27 1.27)))
     )
