File: scan-controller-kicad/drivers.kicad_sch (KiCad schematic)
At the start: 40 parts, among them CN4 Lamp, CN5 Fan, CN6 Motor, Q1 IRF7470, Q5 SS8050, U5 DRV8871DDA, U6 78L05, U7 XL4015, U8 TL431, U9 LM358

Commit message: 31 nets to go
Parts:
- renumbered C18 to C17, C19 to C18, C20 to C19, C21 to C20, C22 to C21, C23 to C22, C24 to C23, C25 to C24

Commit message: Pushbutton PTHs now mechanical (DRC fun)
Connections:
- net Mot-A: now reaches CN6.1, U5.6 (OUT1)
- net Mot-B: now reaches CN6.2, U5.8 (OUT2)
Changed lines of the file:
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@@
 (kicad_sch (version 20230121) (generator eeschema)
   (paper "A4")
+  (junction (at 81.28 54.61) (diameter 0) (color 0 0 0 0)
+  )
   (junction (at 215.9 121.285) (diameter 0) (color 0 0 0 0)
   )
@@
   )
   (junction (at 201.93 92.71) (diameter 0) (color 0 0 0 0)
+  )
+  (junction (at 81.28 52.07) (diameter 0) (color 0 0 0 0)
   )
   (junction (at 169.545 121.285) (diameter 0) (color 0 0 0 0)
@@
     (stroke (width 0) (type default))
   )
+  (wire (pts (xy 81.28 52.07) (xy 90.17 52.07))
+    (stroke (width 0) (type default))
+  )
   (wire (pts (xy 165.735 119.38) (xy 165.735 121.285))
     (stroke (width 0) (type default))
@@
   )
   (wire (pts (xy 121.285 121.285) (xy 118.745 121.285))
+    (stroke (width 0) (type default))
+  )
+  (wire (pts (xy 81.28 54.61) (xy 90.17 54.61))
     (stroke (width 0) (type default))
   )
@@
     (effects (font (size 1.27 1.27)) (justify left bottom))
   )
+  (label "Mot-B" (at 90.17 54.61 0) (fields_autoplaced)
+    (effects (font (size 1.27 1.27)) (justify left bottom))
+  )
+  (label "Mot-A" (at 90.17 52.07 0) (fields_autoplaced)
+    (effects (font (size 1.27 1.27)) (justify left bottom))
+  )

Commit message: Labels, Keep-out, L moved away from camera cable
Connections:
- net 5V-RPi: now also CN5.3; no longer CN5.1
- net at D4.2 (A), Q5.3 (C): now also CN5.1; no longer CN5.3
Changed lines of the file:
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@@
     )
   )
-  (symbol (lib_id "easyeda2kicad:KF141R-2.54-3P") (at 58.42 90.805 0) (unit 1)
+  (symbol (lib_id "easyeda2kicad:KF141R-2.54-3P") (at 58.42 90.805 0) (mirror x) (unit 1)
     (in_bom yes) (on_board yes) (dnp no)
-    (property "Reference" "CN5" (at 57.15 84.455 0)
+    (property "Reference" "CN5" (at 57.15 97.155 0)
       (effects (font (size 1.27 1.27)) (justify left))
     )
-    (property "Value" "Fan" (at 57.785 97.155 0)
+    (property "Value" "Fan" (at 57.785 84.455 0)
       (effects (font (size 1.27 1.27)) (justify left))
     )
-    (property "Footprint" "easyeda2kicad:CONN-TH_3P-P2.54_KF141R-2.54-3P" (at 58.42 100.965 0)
+    (property "Footprint" "easyeda2kicad:CONN-TH_3P-P2.54_KF141R-2.54-3P" (at 58.42 80.645 0)
       (effects (font (size 1.27 1.27)) hide)
     )
-    (property "Datasheet" "https://lcsc.com/product-detail/New-Quadratic-Unclassified-Data_Cixi-Kefa-Elec-KF141R-2-54-3P_C475125.html" (at 58.42 103.505 0)
+    (property "Datasheet" "https://lcsc.com/product-detail/New-Quadratic-Unclassified-Data_Cixi-Kefa-Elec-KF141R-2-54-3P_C475125.html" (at 58.42 78.105 0)
       (effects (font (size 1.27 1.27)) hide)
     )
-    (property "LCSC Part" "" (at 58.42 106.045 0)
+    (property "LCSC Part" "" (at 58.42 75.565 0)
       (effects (font (size 1.27 1.27)) hide)
     )

Commit message: Fixing BOM
Parts:
- Q1: LCSC C386356 -> C693168
Changed lines of the file:
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@@
       (effects (font (size 1.27 1.27)) (justify left) hide)
     )
-    (property "LCSC" "C386356" (at 126.365 118.745 0)
+    (property "LCSC" "C693168" (at 126.365 118.745 0)
       (effects (font (size 1.27 1.27)) hide)
     )

Commit message: Flip U6, it broke the KSQ
Parts:
- U6: symbol Regulator_Linear:L7805 -> Regulator_Linear:L78L05_SOT89
Connections:
- net 24VDC: now also U6.3 (IN); no longer U6.1 (IN)
- net at C20.1, R33.1, R39.1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: now also U6.1 (OUT); no longer U6.3 (OUT)
Changed lines of the file:
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@@
     )
   )
-  (symbol (lib_id "Regulator_Linear:L7805") (at 149.86 107.95 0) (unit 1)
+  (symbol (lib_id "Regulator_Linear:L78L05_SOT89") (at 149.86 107.95 0) (unit 1)
     (in_bom yes) (on_board yes) (dnp no)
     (property "Reference" "U6" (at 149.86 101.6 0)
@@
       (effects (font (size 1.27 1.27)))
     )
-    (property "Footprint" "Package_TO_SOT_SMD:SOT-89-3" (at 150.495 111.76 0)
-      (effects (font (size 1.27 1.27) italic) (justify left) hide)
+    (property "Footprint" "Package_TO_SOT_SMD:SOT-89-3" (at 149.86 102.87 0)
+      (effects (font (size 1.27 1.27) italic) hide)
     )
-    (property "Datasheet" "https://datasheet.lcsc.com/lcsc/2304140030_UTC-Unisonic-Tech-78L05G-AB3-R_C71136.pdf" (at 149.86 109.22 0)
+    (property "Datasheet" "http://www.st.com/content/ccc/resource/technical/document/datasheet/15/55/e5/aa/23/5b/43/fd/CD00000446.pdf/files/CD00000446.pdf/jcr:content/translations/en.CD00000446.pdf" (at 149.86 109.22 0)
       (effects (font (size 1.27 1.27)) hide)
     )

Commit message: Fixing R35 (270 instead of 90k9)
Parts:
- R35: LCSC C104550 -> C137558
Changed lines of the file:
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@@
       (effects (font (size 1.27 1.27)) hide)
     )
-    (property "LCSC" "C104550" (at 207.01 95.885 0)
+    (property "LCSC" "C137558" (at 207.01 95.885 0)
       (effects (font (size 1.27 1.27)) hide)
     )

Commit message: Fixing Shunt Connection to enable Current Control
Connections:
- net Lamp-GND: no longer CN4.1
- net at R38.2, R40.1, U9.3 (+)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: now also CN4.1
Other:
- moved on the sheet: CN4
Changed lines of the file:
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@@
   (junction (at 81.28 54.61) (diameter 0) (color 0 0 0 0)
   )
-  (junction (at 215.9 121.285) (diameter 0) (color 0 0 0 0)
-  )
   (junction (at 201.93 110.49) (diameter 0) (color 0 0 0 0)
   )
@@
   (junction (at 207.01 80.01) (diameter 0) (color 0 0 0 0)
   )
+  (junction (at 234.315 121.285) (diameter 0) (color 0 0 0 0)
+  )
   (junction (at 207.01 89.535) (diameter 0) (color 0 0 0 0)
   )
@@
   (junction (at 138.43 107.95) (diameter 0) (color 0 0 0 0)
   )
-  (no_connect (at 226.695 82.55))
+  (no_connect (at 245.11 82.55))
   (no_connect (at 53.34 90.805))
   (wire (pts (xy 158.75 107.95) (xy 160.02 107.95))
     (stroke (width 0) (type default))
   )
-  (wire (pts (xy 209.55 80.01) (xy 226.695 80.01))
+  (wire (pts (xy 209.55 80.01) (xy 245.11 80.01))
     (stroke (width 0) (type default))
   )
@@
     (stroke (width 0) (type default))
   )
-  (wire (pts (xy 212.725 121.285) (xy 215.9 121.285))
+  (wire (pts (xy 212.725 121.285) (xy 217.805 121.285))
     (stroke (width 0) (type default))
   )
@@
     (stroke (width 0) (type default))
   )
-  (wire (pts (xy 215.9 121.285) (xy 215.9 85.09))
-    (stroke (width 0) (type default))
-  )
   (wire (pts (xy 186.69 107.95) (xy 184.785 107.95))
     (stroke (width 0) (type default))
@@
     (stroke (width 0) (type default))
   )
-  (wire (pts (xy 215.9 85.09) (xy 226.695 85.09))
-    (stroke (width 0) (type default))
-  )
   (wire (pts (xy 231.14 100.33) (xy 234.315 100.33))
     (stroke (width 0) (type default))
@@
     (stroke (width 0) (type default))
   )
-  (wire (pts (xy 215.9 121.285) (xy 217.805 121.285))
+  (wire (pts (xy 245.11 121.285) (xy 245.11 85.09))
     (stroke (width 0) (type default))
   )
@@
   )
   (wire (pts (xy 218.44 112.395) (xy 218.44 116.205))
+    (stroke (width 0) (type default))
+  )
+  (wire (pts (xy 234.315 121.285) (xy 245.11 121.285))
     (stroke (width 0) (type default))
   )
@@
     )
   )
-  (symbol (lib_id "easyeda2kicad:KF141R-2.54-3P") (at 231.775 82.55 0) (mirror x) (unit 1)
-    (in_bom yes) (on_board yes) (dnp no)
-    (property "Reference" "CN4" (at 230.505 88.9 0)
-      (effects (font (size 1.27 1.27)) (justify left))
-    )
-    (property "Value" "Lamp" (at 231.14 76.2 0)
-      (effects (font (size 1.27 1.27)) (justify left))
-    )
-    (property "Footprint" "easyeda2kicad:CONN-TH_3P-P2.54_KF141R-2.54-3P" (at 231.775 72.39 0)
-      (effects (font (size 1.27 1.27)) hide)
-    )
-    (property "Datasheet" "https://lcsc.com/product-detail/New-Quadratic-Unclassified-Data_Cixi-Kefa-Elec-KF141R-2-54-3P_C475125.html" (at 231.775 69.85 0)
-      (effects (font (size 1.27 1.27)) hide)
-    )
-    (property "LCSC Part" "" (at 231.775 67.31 0)
-      (effects (font (size 1.27 1.27)) hide)
-    )
-    (property "LCSC" "C475125" (at 231.775 82.55 0)
-      (effects (font (size 1.27 1.27)) hide)
-    )
-    (property "Inventory" "" (at 231.775 82.55 0)
-      (effects (font (size 1.27 1.27)) hide)
-    )
+  (symbol (lib_id "easyeda2kicad:KF141R-2.54-3P") (at 250.19 82.55 0) (mirror x) (unit 1)
+    (in_bom yes) (on_board yes) (dnp no)
+    (property "Reference" "CN4" (at 248.92 88.9 0)
+      (effects (font (size 1.27 1.27)) (justify left))
+    )
+    (property "Value" "Lamp" (at 249.555 76.2 0)
+      (effects (font (size 1.27 1.27)) (justify left))
+    )
+    (property "Footprint" "easyeda2kicad:CONN-TH_3P-P2.54_KF141R-2.54-3P" (at 250.19 72.39 0)
+      (effects (font (size 1.27 1.27)) hide)
+    )
+    (property "Datasheet" "https://lcsc.com/product-detail/New-Quadratic-Unclassified-Data_Cixi-Kefa-Elec-KF141R-2-54-3P_C475125.html" (at 250.19 69.85 0)
+      (effects (font (size 1.27 1.27)) hide)
+    )
+    (property "LCSC Part" "" (at 250.19 67.31 0)
+      (effects (font (size 1.27 1.27)) hide)
+    )
+    (property "LCSC" "C475125" (at 250.19 82.55 0)
+      (effects (font (size 1.27 1.27)) hide)
+    )
+    (property "Inventory" "" (at 250.19 82.55 0)
+      (effects (font (size 1.27 1.27)) hide)
+    )
