File: scan-controller-kicad/drivers.kicad_sch (KiCad schematic)
At the start: 40 parts, among them CN4 Lamp, CN5 Fan, CN6 Motor, Q1 IRF7470, Q5 SS8050, U5 DRV8871DDA, U6 78L05, U7 XL4015, U8 TL431, U9 LM358

Commit message: Freeing up D4 (328) as it isn't needed
Parts:
- renumbered C7 to C15, C8 to C16, CN5 to CN4, CN6 to CN5, CN4 to CN6, Q5 to Q6, Q1 to Q7, R15 to R29, R19 to R30, R3 to R31, R2 to R32
Changed lines of the file:
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@@
   (symbol (lib_id "Device:R_Small") (at 126.365 103.505 180) (unit 1)
     (in_bom yes) (on_board yes) (dnp no)
-    (property "Reference" "R2" (at 129.54 105.41 0)
+    (property "Reference" "R32" (at 129.54 105.41 0)
       (effects (font (size 1.27 1.27)))
     )
@@
     (instances
       (project "scan-controller-kicad"
-        (path "/ab6dbce1-4ecf-44ae-8f33-5f07e4f43ca9"
-          (reference "R2") (unit 1)
-        )
         (path "/ab6dbce1-4ecf-44ae-8f33-5f07e4f43ca9/f199f7c1-4da9-41da-ae5e-c136f90f6de6"
           (reference "R32") (unit 1)
@@
   (symbol (lib_id "Device:R_Small") (at 78.74 62.23 0) (unit 1)
     (in_bom yes) (on_board yes) (dnp no)
-    (property "Reference" "R19" (at 80.01 60.96 0)
+    (property "Reference" "R30" (at 80.01 60.96 0)
       (effects (font (size 1.27 1.27)) (justify left))
     )
@@
     (instances
       (project "scan-controller-kicad"
-        (path "/ab6dbce1-4ecf-44ae-8f33-5f07e4f43ca9"
-          (reference "R19") (unit 1)
-        )
         (path "/ab6dbce1-4ecf-44ae-8f33-5f07e4f43ca9/f199f7c1-4da9-41da-ae5e-c136f90f6de6"
           (reference "R30") (unit 1)
@@
   (symbol (lib_id "power:GNDD") (at 118.745 124.46 0) (unit 1)
     (in_bom yes) (on_board yes) (dnp no)
-    (property "Reference" "#PWR05" (at 118.745 130.81 0)
+    (property "Reference" "#PWR032" (at 118.745 130.81 0)
       (effects (font (size 1.27 1.27)) hide)
     )
@@
     (instances
       (project "scan-controller-kicad"
-        (path "/ab6dbce1-4ecf-44ae-8f33-5f07e4f43ca9"
-          (reference "#PWR05") (unit 1)
-        )
         (path "/ab6dbce1-4ecf-44ae-8f33-5f07e4f43ca9/f199f7c1-4da9-41da-ae5e-c136f90f6de6"
           (reference "#PWR032") (unit 1)
@@
   (symbol (lib_id "easyeda2kicad:KF141R-2.54-3P") (at 58.42 90.805 0) (mirror x) (unit 1)
     (in_bom yes) (on_board yes) (dnp no)
-    (property "Reference" "CN5" (at 57.15 97.155 0)
+    (property "Reference" "CN4" (at 57.15 97.155 0)
       (effects (font (size 1.27 1.27)) (justify left))
     )
@@
     (instances
       (project "scan-controller-kicad"
-        (path "/ab6dbce1-4ecf-44ae-8f33-5f07e4f43ca9"
-          (reference "CN5") (unit 1)
-        )
         (path "/ab6dbce1-4ecf-44ae-8f33-5f07e4f43ca9/f199f7c1-4da9-41da-ae5e-c136f90f6de6"
           (reference "CN4") (unit 1)
@@
   (symbol (lib_id "Device:R_Small") (at 122.555 113.665 270) (unit 1)
     (in_bom yes) (on_board yes) (dnp no)
-    (property "Reference" "R3" (at 120.65 115.57 90)
+    (property "Reference" "R31" (at 120.65 115.57 90)
       (effects (font (size 1.27 1.27)) (justify left))
     )
@@
     (instances
       (project "scan-controller-kicad"
-        (path "/ab6dbce1-4ecf-44ae-8f33-5f07e4f43ca9"
-          (reference "R3") (unit 1)
-        )
         (path "/ab6dbce1-4ecf-44ae-8f33-5f07e4f43ca9/f199f7c1-4da9-41da-ae5e-c136f90f6de6"
           (reference "R31") (unit 1)
@@
   (symbol (lib_id "power:GNDD") (at 49.53 106.045 0) (unit 1)
     (in_bom yes) (on_board yes) (dnp no)
-    (property "Reference" "#PWR022" (at 49.53 112.395 0)
+    (property "Reference" "#PWR028" (at 49.53 112.395 0)
       (effects (font (size 1.27 1.27)) hide)
     )
@@
     (instances
       (project "scan-controller-kicad"
-        (path "/ab6dbce1-4ecf-44ae-8f33-5f07e4f43ca9"
-          (reference "#PWR022") (unit 1)
-        )
         (path "/ab6dbce1-4ecf-44ae-8f33-5f07e4f43ca9/f199f7c1-4da9-41da-ae5e-c136f90f6de6"
           (reference "#PWR028") (unit 1)
@@
   (symbol (lib_id "Device:R_Small") (at 38.1 99.695 270) (unit 1)
     (in_bom yes) (on_board yes) (dnp no)
-    (property "Reference" "R15" (at 38.1 97.155 90)
+    (property "Reference" "R29" (at 38.1 97.155 90)
       (effects (font (size 1.27 1.27)))
     )
@@
     (instances
       (project "scan-controller-kicad"
-        (path "/ab6dbce1-4ecf-44ae-8f33-5f07e4f43ca9"
-          (reference "R15") (unit 1)
-        )
         (path "/ab6dbce1-4ecf-44ae-8f33-5f07e4f43ca9/f199f7c1-4da9-41da-ae5e-c136f90f6de6"
           (reference "R29") (unit 1)
@@
     (instances
       (project "scan-controller-kicad"
-        (path "/ab6dbce1-4ecf-44ae-8f33-5f07e4f43ca9"
-          (reference "U5") (unit 1)
-        )
         (path "/ab6dbce1-4ecf-44ae-8f33-5f07e4f43ca9/f199f7c1-4da9-41da-ae5e-c136f90f6de6"
           (reference "U5") (unit 1)
@@
   (symbol (lib_id "Transistor_BJT:BC847") (at 46.99 99.695 0) (unit 1)
     (in_bom yes) (on_board yes) (dnp no)
-    (property "Reference" "Q5" (at 51.8414 98.5266 0)
+    (property "Reference" "Q6" (at 51.8414 98.5266 0)
       (effects (font (size 1.27 1.27)) (justify left))
     )
@@
     (instances
       (project "scan-controller-kicad"
-        (path "/ab6dbce1-4ecf-44ae-8f33-5f07e4f43ca9"
-          (reference "Q5") (unit 1)
-        )
         (path "/ab6dbce1-4ecf-44ae-8f33-5f07e4f43ca9/f199f7c1-4da9-41da-ae5e-c136f90f6de6"
           (reference "Q6") (unit 1)
@@
   (symbol (lib_id "Device:C_Polarized_Small") (at 53.975 38.1 0) (unit 1)
     (in_bom yes) (on_board yes) (dnp no)
-    (property "Reference" "C7" (at 49.53 36.195 0)
+    (property "Reference" "C15" (at 49.53 36.195 0)
       (effects (font (size 1.27 1.27)) (justify left))
     )
@@
     (instances
       (project "scan-controller-kicad"
-        (path "/ab6dbce1-4ecf-44ae-8f33-5f07e4f43ca9"
-          (reference "C7") (unit 1)
-        )
         (path "/ab6dbce1-4ecf-44ae-8f33-5f07e4f43ca9/f199f7c1-4da9-41da-ae5e-c136f90f6de6"
           (reference "C15") (unit 1)
@@
   (symbol (lib_id "Device:C_Small") (at 60.96 38.1 0) (unit 1)
     (in_bom yes) (on_board yes) (dnp no)
-    (property "Reference" "C8" (at 62.23 36.195 0)
+    (property "Reference" "C16" (at 62.23 36.195 0)
       (effects (font (size 1.27 1.27)) (justify left))
     )
@@
     (instances
       (project "scan-controller-kicad"
-        (path "/ab6dbce1-4ecf-44ae-8f33-5f07e4f43ca9"
-          (reference "C8") (unit 1)
-        )
         (path "/ab6dbce1-4ecf-44ae-8f33-5f07e4f43ca9/f199f7c1-4da9-41da-ae5e-c136f90f6de6"
           (reference "C16") (unit 1)
@@
   (symbol (lib_id "easyeda2kicad:KF141R-2.54-3P") (at 250.19 82.55 0) (mirror x) (unit 1)
     (in_bom yes) (on_board yes) (dnp no)
-    (property "Reference" "CN4" (at 248.92 88.9 0)
+    (property "Reference" "CN6" (at 248.92 88.9 0)
       (effects (font (size 1.27 1.27)) (justify left))
     )
@@
     (instances
       (project "scan-controller-kicad"
-        (path "/ab6dbce1-4ecf-44ae-8f33-5f07e4f43ca9"
-          (reference "CN4") (unit 1)
-        )
         (path "/ab6dbce1-4ecf-44ae-8f33-5f07e4f43ca9/f199f7c1-4da9-41da-ae5e-c136f90f6de6"
           (reference "CN6") (unit 1)
@@
   (symbol (lib_id "power:GNDD") (at 60.96 43.18 0) (unit 1)
     (in_bom yes) (on_board yes) (dnp no)
-    (property "Reference" "#PWR025" (at 60.96 49.53 0)
+    (property "Reference" "#PWR030" (at 60.96 49.53 0)
       (effects (font (size 1.27 1.27)) hide)
     )
@@
     (instances
       (project "scan-controller-kicad"
-        (path "/ab6dbce1-4ecf-44ae-8f33-5f07e4f43ca9"
-          (reference "#PWR025") (unit 1)
-        )
         (path "/ab6dbce1-4ecf-44ae-8f33-5f07e4f43ca9/f199f7c1-4da9-41da-ae5e-c136f90f6de6"
           (reference "#PWR030") (unit 1)
@@
     (instances
       (project "scan-controller-kicad"
-        (path "/ab6dbce1-4ecf-44ae-8f33-5f07e4f43ca9"
-          (reference "D4") (unit 1)
-        )
         (path "/ab6dbce1-4ecf-44ae-8f33-5f07e4f43ca9/f199f7c1-4da9-41da-ae5e-c136f90f6de6"
           (reference "D4") (unit 1)
@@
   (symbol (lib_id "Transistor_FET:IRF7403") (at 126.365 118.745 270) (unit 1)
     (in_bom yes) (on_board yes) (dnp no) (fields_autoplaced)
-    (property "Reference" "Q1" (at 127.635 124.46 0)
+    (property "Reference" "Q7" (at 127.635 124.46 0)
       (effects (font (size 1.27 1.27)) (justify left))
     )
@@
     (instances
       (project "scan-controller-kicad"
-        (path "/ab6dbce1-4ecf-44ae-8f33-5f07e4f43ca9"
-          (reference "Q1") (unit 1)
-        )
         (path "/ab6dbce1-4ecf-44ae-8f33-5f07e4f43ca9/f199f7c1-4da9-41da-ae5e-c136f90f6de6"
           (reference "Q7") (unit 1)
@@
   (symbol (lib_id "power:GNDD") (at 53.975 43.18 0) (unit 1)
     (in_bom yes) (on_board yes) (dnp no)
-    (property "Reference" "#PWR023" (at 53.975 49.53 0)
+    (property "Reference" "#PWR029" (at 53.975 49.53 0)
       (effects (font (size 1.27 1.27)) hide)
     )
@@
     (instances
       (project "scan-controller-kicad"
-        (path "/ab6dbce1-4ecf-44ae-8f33-5f07e4f43ca9"
-          (reference "#PWR023") (unit 1)
-        )
         (path "/ab6dbce1-4ecf-44ae-8f33-5f07e4f43ca9/f199f7c1-4da9-41da-ae5e-c136f90f6de6"
           (reference "#PWR029") (unit 1)
@@
   (symbol (lib_id "easyeda2kicad:KF142R-5.08-2P") (at 86.36 53.34 0) (unit 1)
     (in_bom yes) (on_board yes) (dnp no)
-    (property "Reference" "CN6" (at 86.995 48.26 0)
+    (property "Reference" "CN5" (at 86.995 48.26 0)
       (effects (font (size 1.27 1.27)))
     )
@@
     (instances
       (project "scan-controller-kicad"
-        (path "/ab6dbce1-4ecf-44ae-8f33-5f07e4f43ca9"
-          (reference "CN6") (unit 1)
-        )
         (path "/ab6dbce1-4ecf-44ae-8f33-5f07e4f43ca9/f199f7c1-4da9-41da-ae5e-c136f90f6de6"
           (reference "CN5") (unit 1)
@@
   (symbol (lib_id "power:GNDD") (at 68.58 66.04 0) (unit 1)
     (in_bom yes) (on_board yes) (dnp no)
-    (property "Reference" "#PWR030" (at 68.58 72.39 0)
+    (property "Reference" "#PWR031" (at 68.58 72.39 0)
       (effects (font (size 1.27 1.27)) hide)
     )
@@
     (instances
       (project "scan-controller-kicad"
-        (path "/ab6dbce1-4ecf-44ae-8f33-5f07e4f43ca9"
-          (reference "#PWR030") (unit 1)
-        )
         (path "/ab6dbce1-4ecf-44ae-8f33-5f07e4f43ca9/f199f7c1-4da9-41da-ae5e-c136f90f6de6"
           (reference "#PWR031") (unit 1)

Commit message: Replacing D6 LED with 1N4148 Adding TPs for Lamp Current Fixing TP Labels and other Labels Add LED D9 that actually reflects Lamp status Add control LEDs for Eyes (makes mounting much easier) Add mini manual and tech specs on the back side
Parts:
- added D9: Lamp (wh), LED_SMD:LED_0805_2012Metric, symbol Device:LED_Small
- added R43: 2K2, Resistor_SMD:R_0805_2012Metric, symbol Device:R_Small
- added TP13, TP14, TP15: TestPoint, Peacemans_Footprints:TestPoint_THTPad_1.5x1.5mm_Drill0.7mm_named, symbol Peacemans_Teile:TestPoint_named
- D6: value LED (wh) -> 1N4148W; footprint LED_SMD:LED_0805_2012Metric -> Diode_SMD:D_SOD-123; symbol Device:LED_Small -> Diode:1N4448W; Inventory B -> (none); LCSC C34499 -> C81598
Connections:
- net GNDD: now also D9.1 (K)
- net Lamp: now also R43.1
- net at C22.1, C23.1, CN6.3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: now also TP14.1
- net at CN6.1, R38.2, R40.1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: now also TP15.1
- net at CN6.2: now also TP13.1
- new net: D9.2 (A), R43.2
- no-connect marks 2 -> 1
Other:
- moved on the sheet: D8, R40

Commit message: Last Version with the second OpAmp stilll in use
Other:
- note added: "Current"
- note added: "Voltage"
Changed lines of the file:
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@@
     (stroke (width 0) (type default))
+  )
+  (text "Current" (at 172.085 120.65 0)
+    (effects (font (size 1.27 1.27)) (justify left bottom))
+  )
+  (text "Voltage" (at 209.55 89.535 0)
+    (effects (font (size 1.27 1.27)) (justify left bottom))
   )
   (label "Lamp-GND" (at 133.985 124.46 0) (fields_autoplaced)

Commit message: Lamp Driver final, but now off grid :-?
Parts:
- removed D7, D8: LED (ye), LED_SMD:LED_0805_2012Metric, symbol Device:LED_Small
- removed R36: 90K9, Resistor_SMD:R_0805_2012Metric, symbol Device:R_Small
- removed R37: 10K, Resistor_SMD:R_0805_2012Metric, symbol Device:R_Small
- removed R39, R40: 1K, Resistor_SMD:R_0805_2012Metric, symbol Device:R_Small
- removed U9: LM358, Package_SO:SOIC-8_3.9x4.9mm_P1.27mm, symbol Amplifier_Operational:LM358
- added U10: LM358, Package_SO:SOIC-8_3.9x4.9mm_P1.27mm, symbol Amplifier_Operational:LM358
Connections:
- net Lamp-GND: now also U10.4 (V-)
- net at C20.1, R33.1, U6.1 (OUT): now also U10.8 (V+)
- net at C24.2, RV4.2: now also U10.2 (-), U10.5 (+)
- net at C24.1, D6.2 (A): now also U10.1
- net at CN6.1, R38.2, TP15.1: now also U10.3 (+)
- new net: U10.6 (-), U10.7
Other:
- moved on the sheet: C15, C16, C17, C18, C19, C20, C21, C22, C23, C24, CN5, CN6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

Commit message: Fixing the Lamp Driver Grid
Other:
- moved on the sheet: C15, C16, CN5, R30, U5

Commit message: Added Mounting Holes back in
Parts:
- added TP16: TestPoint, Peacemans_Footprints:TestPoint_THTPad_1.5x1.5mm_Drill0.7mm_named, symbol Peacemans_Teile:TestPoint_named
Connections:
- net Lamp-GND: now also TP16.1
Changed lines of the file:
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@@
+    )
+  )
+  (symbol (lib_id "Peacemans_Teile:TestPoint_named") (at 176.53 97.155 180) (unit 1)
+    (in_bom yes) (on_board yes) (dnp no)
+    (property "Reference" "TP16" (at 176.53 104.013 0)
+      (effects (font (size 1.27 1.27)) hide)
+    )
+    (property "Value" "TestPoint" (at 176.53 102.235 0)
+      (effects (font (size 1.27 1.27)) hide)
+    )
+    (property "Footprint" "Peacemans_Footprints:TestPoint_THTPad_1.5x1.5mm_Drill0.7mm_named" (at 171.45 97.155 0)
+      (effects (font (size 1.27 1.27)) hide)
+    )
+    (property "Datasheet" "~" (at 171.45 97.155 0)
+      (effects (font (size 1.27 1.27)) hide)
+    )
+    (property "TP_Label" "Motor GND" (at 176.53 102.87 0)
+      (effects (font (size 1.27 1.27)))
+    )
+    (pin "1")
+    (instances
+      (project "scan-controller-kicad"
+        (path "/ab6dbce1-4ecf-44ae-8f33-5f07e4f43ca9/f199f7c1-4da9-41da-ae5e-c136f90f6de6"
+          (reference "TP16") (unit 1)
+        )
+      )
     )
   )

Commit message: Reannotated
Parts:
- U8: renamed from U10; footprint (none) -> Package_SO:SOIC-8_3.9x4.9mm_P1.27mm
- renumbered C17 to C1, C21 to C12, C19 to C14, C23 to C15, C24 to C16, C15 to C17, C16 to C18, C22 to C19, C18 to C2, C20 to C3, CN5 to CN2, CN4 to CN3, CN6 to CN4, D5 to D4, D6 to D5, D9 to D6, D4 to D8, Q7 to Q1, Q6 to Q8, R33 to R10, R35 to R16, R34 to R17, R38 to R18, R30 to R19, R43 to R26, R29 to R38, R32 to R8, R31 to R9, RV4 to RV1, RV5 to RV3, TP15 to TP14, TP14 to TP15, TP13 to TP16, TP16 to TP9, U6 to U3, U5 to U4, U8 to U6, U10 to U8
