File: scan-controller-kicad/userinterface.kicad_sch (KiCad schematic)
At the start: 26 parts, among them SW1 Power, SW10 Rec, SW2 Lamp, SW3 Zoom, SW4 <<, SW5 <, SW7 Stop, SW8 >, SW9 >>

Commit message: It's getting neat and readable
Parts:
- added D5: Film End, LED_SMD:LED_0805_2012Metric, symbol Device:LED_Small
- added R20: 300R, Resistor_SMD:R_0805_2012Metric, symbol Device:R_Small
Connections:
- net GNDD: now also D5.1 (K)
- new net: D5.2 (A), R20.2
- new net Film End LED: R20.1
Changed lines of the file:
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@@
+    (stroke (width 0) (type default))
+  )
+  (wire (pts (xy 219.075 64.135) (xy 219.075 67.945))
     (stroke (width 0) (type default))
   )
@@
     (stroke (width 0) (type default))
   )
+  (wire (pts (xy 219.075 73.025) (xy 219.075 74.93))
+    (stroke (width 0) (type default))
+  )
   (wire (pts (xy 200.025 128.27) (xy 200.025 130.81))
     (stroke (width 0) (type default))
@@
     (stroke (width 0) (type default))
   )
+  (wire (pts (xy 219.075 80.01) (xy 219.075 81.915))
+    (stroke (width 0) (type default))
+  )
   (wire (pts (xy 111.125 124.46) (xy 111.125 125.73))
     (stroke (width 0) (type default))
@@
   )
   (wire (pts (xy 172.72 78.105) (xy 161.29 78.105))
+    (stroke (width 0) (type default))
+  )
+  (wire (pts (xy 213.995 64.135) (xy 219.075 64.135))
     (stroke (width 0) (type default))
   )
@@
     (effects (font (size 1.27 1.27)) (justify left))
   )
+  (hierarchical_label "Film End LED" (shape input) (at 213.995 64.135 180) (fields_autoplaced)
+    (effects (font (size 1.27 1.27)) (justify right))
+  )
   (hierarchical_label "Keys 1" (shape input) (at 130.81 65.405 0) (fields_autoplaced)
     (effects (font (size 1.27 1.27)) (justify left))
@@
     )
   )
+  (symbol (lib_id "Device:R_Small") (at 219.075 70.485 0) (unit 1)
+    (in_bom yes) (on_board yes) (dnp no)
+    (property "Reference" "R20" (at 215.9 72.39 90)
+      (effects (font (size 1.27 1.27)) (justify left))
+    )
+    (property "Value" "300R" (at 221.615 71.755 90)
+      (effects (font (size 1.27 1.27)) (justify left))
+    )
+    (property "Footprint" "Resistor_SMD:R_0805_2012Metric" (at 219.075 70.485 0)
+      (effects (font (size 1.27 1.27)) hide)
+    )
+    (property "Datasheet" "~" (at 219.075 70.485 0)
+      (effects (font (size 1.27 1.27)) hide)
+    )
+    (property "LCSC" "C17617" (at 219.075 70.485 0)
+      (effects (font (size 1.27 1.27)) hide)
+    )
+    (pin "1")
+    (pin "2")
+    (instances
+      (project "scan-controller-kicad"
+        (path "/ab6dbce1-4ecf-44ae-8f33-5f07e4f43ca9"
+          (reference "R20") (unit 1)
+        )
+        (path "/ab6dbce1-4ecf-44ae-8f33-5f07e4f43ca9/486b6b54-3904-49a9-9b52-9c586c7b0887"
+          (reference "R20") (unit 1)
+        )
+      )
+    )
+  )
   (symbol (lib_id "power:GNDD") (at 110.49 95.885 0) (unit 1)
     (in_bom yes) (on_board yes) (dnp no)
@@
     )
   )
+  (symbol (lib_id "power:GNDD") (at 219.075 81.915 0) (unit 1)
+    (in_bom yes) (on_board yes) (dnp no)
+    (property "Reference" "#PWR036" (at 219.075 88.265 0)
+      (effects (font (size 1.27 1.27)) hide)
+    )
+    (property "Value" "GNDD" (at 219.075 85.725 0)
+      (effects (font (size 1.27 1.27)))
+    )
+    (property "Footprint" "" (at 219.075 81.915 0)
+      (effects (font (size 1.27 1.27)) hide)
+    )
+    (property "Datasheet" "" (at 219.075 81.915 0)
+      (effects (font (size 1.27 1.27)) hide)
+    )
+    (pin "1")
+    (instances
+      (project "scan-controller-kicad"
+        (path "/ab6dbce1-4ecf-44ae-8f33-5f07e4f43ca9"
+          (reference "#PWR036") (unit 1)
+        )
+        (path "/ab6dbce1-4ecf-44ae-8f33-5f07e4f43ca9/486b6b54-3904-49a9-9b52-9c586c7b0887"
+          (reference "#PWR05") (unit 1)
+        )
+      )
+    )
+  )
   (symbol (lib_id "Device:R_Small") (at 177.8 67.945 270) (unit 1)
     (in_bom yes) (on_board yes) (dnp no)
@@
         )
       )
+    )
+  )
+  (symbol (lib_id "Device:LED_Small") (at 219.075 77.47 90) (unit 1)
+    (in_bom yes) (on_board yes) (dnp no)
+    (property "Reference" "D5" (at 215.9 77.47 0)
+      (effects (font (size 1.27 1.27)))
+    )
+    (property "Value" "Film End" (at 221.615 78.105 0)
+      (effects (font (size 1.27 1.27)))
+    )
+    (property "Footprint" "LED_SMD:LED_0805_2012Metric" (at 219.075 77.47 90)
+      (effects (font (size 1.27 1.27)) hide)
+    )
+    (property "Datasheet" "https://datasheet.lcsc.com/lcsc/2304140030_Foshan-NationStar-Optoelectronics-NCD0805R1_C84256.pdf" (at 219.075 77.47 90)
+      (effects (font (size 1.27 1.27)) hide)
+    )
+    (property "LCSC" " C84256" (at 219.075 77.47 0)
+      (effects (font (size 1.27 1.27)) hide)
+    )
+    (pin "1")
+    (pin "2")
+    (instances
+      (project "scan-controller-kicad"
+        (path "/ab6dbce1-4ecf-44ae-8f33-5f07e4f43ca9"
+          (reference "D5") (unit 1)
+        )
+        (path "/ab6dbce1-4ecf-44ae-8f33-5f07e4f43ca9/486b6b54-3904-49a9-9b52-9c586c7b0887"
+          (reference "D5") (unit 1)
+        )
+      )

Commit message: Adding missing components Mfnrs and footprints
Parts:
- D5: LCSC C84256 -> C84256
- D6: LCSC C2297 -> C2297
- SW1, SW10, SW2, SW3, SW4, SW5, SW7, SW8, SW9: LCSC (none) -> C93156; LCSC Part C93156 -> (none)

Commit message: BOM progress
Parts:
- D5: value Film End -> Film End (re); Inventory (none) -> B
- D6: value Power -> Power (gr); Inventory (none) -> B
- R20, R21, R22, R23, R24, R25, R26, R28, R29, R30, R31, R32: Inventory (none) -> B
Changed lines of the file:
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@@
+      (effects (font (size 1.27 1.27)) hide)
+    )
+    (property "Inventory" "" (at 118.11 65.405 0)
       (effects (font (size 1.27 1.27)) hide)
     )
@@
       (effects (font (size 1.27 1.27)) hide)
     )
+    (property "Inventory" "" (at 200.025 125.73 0)
+      (effects (font (size 1.27 1.27)) hide)
+    )
     (pin "1")
     (pin "2")
@@
       (effects (font (size 1.27 1.27)) hide)
     )
+    (property "Inventory" "" (at 118.11 88.265 0)
+      (effects (font (size 1.27 1.27)) hide)
+    )
     (pin "1")
     (pin "2")
@@
       (effects (font (size 1.27 1.27)) hide)
     )
+    (property "Inventory" "B" (at 219.075 70.485 0)
+      (effects (font (size 1.27 1.27)) hide)
+    )
     (pin "1")
     (pin "2")
@@
       (effects (font (size 1.27 1.27)) hide)
     )
+    (property "Inventory" "B" (at 111.125 137.16 0)
+      (effects (font (size 1.27 1.27)) hide)
+    )
     (pin "1")
     (pin "2")
@@
       (effects (font (size 1.27 1.27)) hide)
     )
+    (property "Inventory" "" (at 172.72 73.025 0)
+      (effects (font (size 1.27 1.27)) hide)
+    )
     (pin "1")
     (pin "2")
@@
       (effects (font (size 1.27 1.27)) hide)
     )
+    (property "Inventory" "B" (at 111.125 114.3 0)
+      (effects (font (size 1.27 1.27)) hide)
+    )
     (pin "1")
     (pin "2")
@@
       (effects (font (size 1.27 1.27)) hide)
     )
+    (property "Inventory" "" (at 161.29 73.025 0)
+      (effects (font (size 1.27 1.27)) hide)
+    )
     (pin "1")
     (pin "2")
@@
     )
     (property "LCSC" "C93156" (at 120.65 39.37 0)
+      (effects (font (size 1.27 1.27)) hide)
+    )
+    (property "Inventory" "" (at 120.65 39.37 0)
       (effects (font (size 1.27 1.27)) hide)
     )
@@
       (effects (font (size 1.27 1.27)) hide)
     )
+    (property "Inventory" "" (at 163.195 112.395 0)
+      (effects (font (size 1.27 1.27)) hide)
+    )
     (pin "1")
     (pin "2")
@@
       (effects (font (size 1.27 1.27)) hide)
     )
+    (property "Inventory" "B" (at 110.49 76.835 0)
+      (effects (font (size 1.27 1.27)) hide)
+    )
     (pin "1")
     (pin "2")
@@
       (effects (font (size 1.27 1.27)) hide)
     )
+    (property "Inventory" "" (at 118.745 118.11 0)
+      (effects (font (size 1.27 1.27)) hide)
+    )
     (pin "1")
     (pin "2")
@@
       (effects (font (size 1.27 1.27)) hide)
     )
+    (property "Inventory" "B" (at 110.49 69.215 0)
+      (effects (font (size 1.27 1.27)) hide)
+    )
     (pin "1")
     (pin "2")
@@
       (effects (font (size 1.27 1.27)) hide)
     )
+    (property "Inventory" "" (at 118.745 133.35 0)
+      (effects (font (size 1.27 1.27)) hide)
+    )
     (pin "1")
     (pin "2")
@@
       (effects (font (size 1.27 1.27)))
     )
-    (property "Value" "Power" (at 187.96 75.565 90)
+    (property "Value" "Power (gr)" (at 187.96 75.565 90)
       (effects (font (size 1.27 1.27)))
     )
@@
       (effects (font (size 1.27 1.27)) hide)
     )
+    (property "Inventory" "B" (at 184.15 73.025 0)
+      (effects (font (size 1.27 1.27)) hide)
+    )
     (pin "1")
     (pin "2")
@@
       (effects (font (size 1.27 1.27)) hide)
     )
+    (property "Inventory" "B" (at 111.125 129.54 0)
+      (effects (font (size 1.27 1.27)) hide)
+    )
     (pin "1")
     (pin "2")
@@
       (effects (font (size 1.27 1.27)) hide)
     )
+    (property "Inventory" "" (at 118.11 80.645 0)
+      (effects (font (size 1.27 1.27)) hide)
+    )
     (pin "1")
     (pin "2")
@@
       (effects (font (size 1.27 1.27)) hide)
     )
+    (property "Inventory" "" (at 118.745 125.73 0)
+      (effects (font (size 1.27 1.27)) hide)
+    )
     (pin "1")
     (pin "2")
@@
       (effects (font (size 1.27 1.27)) hide)
     )
+    (property "Inventory" "B" (at 126.365 137.16 0)
+      (effects (font (size 1.27 1.27)) hide)
+    )
     (pin "1")
     (pin "2")
@@
       (effects (font (size 1.27 1.27)) hide)
     )
+    (property "Inventory" "B" (at 110.49 92.075 0)
+      (effects (font (size 1.27 1.27)) hide)
+    )
     (pin "1")
     (pin "2")
@@
       (effects (font (size 1.27 1.27)) hide)
     )
+    (property "Inventory" "B" (at 110.49 84.455 0)
+      (effects (font (size 1.27 1.27)) hide)
+    )
     (pin "1")
     (pin "2")
@@
     )
     (property "LCSC" "C17713" (at 111.125 121.92 0)
+      (effects (font (size 1.27 1.27)) hide)
+    )
+    (property "Inventory" "B" (at 111.125 121.92 0)
       (effects (font (size 1.27 1.27)) hide)
     )
@@
       (effects (font (size 1.27 1.27)) hide)
     )
+    (property "Inventory" "" (at 180.975 119.38 0)
+      (effects (font (size 1.27 1.27)) hide)
+    )
     (pin "1")
     (pin "2")
@@
       (effects (font (size 1.27 1.27)) hide)
     )
+    (property "Inventory" "" (at 118.745 110.49 0)
+      (effects (font (size 1.27 1.27)) hide)
+    )
     (pin "1")
     (pin "2")
@@
       (effects (font (size 1.27 1.27)) hide)
     )
+    (property "Inventory" "B" (at 177.8 67.945 0)
+      (effects (font (size 1.27 1.27)) hide)
+    )
     (pin "1")
     (pin "2")
@@
       (effects (font (size 1.27 1.27)))
     )
-    (property "Value" "Film End" (at 221.615 78.105 0)
+    (property "Value" "Film End (re)" (at 221.615 78.105 0)
       (effects (font (size 1.27 1.27)))
     )
@@
       (effects (font (size 1.27 1.27)) hide)
     )
+    (property "Inventory" "B" (at 219.075 77.47 0)
+      (effects (font (size 1.27 1.27)) hide)
+    )
     (pin "1")
     (pin "2")
@@
       (effects (font (size 1.27 1.27)) hide)
     )
+    (property "Inventory" "" (at 118.11 73.025 0)
+      (effects (font (size 1.27 1.27)) hide)
+    )
     (pin "1")
     (pin "2")
@@
       (effects (font (size 1.27 1.27)) hide)
     )
+    (property "Inventory" "B" (at 125.73 92.075 0)
+      (effects (font (size 1.27 1.27)) hide)
+    )

Commit message: BOM complete!
Parts:
- C11: footprint Capacitor_SMD:CP_Elec_5x5.4 -> Capacitor_SMD:C_0805_2012Metric; symbol Device:C_Polarized_Small -> Device:C_Small; Inventory (none) -> B; LCSC C335978 -> C15850
- C13: Inventory (none) -> B
- RV1, RV2: footprint easyeda2kicad:RES-ADJ-SMD_RDC506002A -> easyeda2kicad:RES-ADJ-TH_RK09K1130AJ3; Inventory (none) -> E; LCSC C115341 -> C470295
- RV3: footprint easyeda2kicad:RES-ADJ-SMD_RDC506002A -> easyeda2kicad:RES-ADJ-TH_3P-L10.0-W10.0-P2.50-L; Inventory (none) -> E; LCSC C115341 -> C118954
- SW2: Inventory (none) -> E
Changed lines of the file:
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@@
       (effects (font (size 1.27 1.27)) hide)
     )
-    (property "Inventory" "" (at 118.11 65.405 0)
+    (property "Inventory" "E" (at 118.11 65.405 0)
       (effects (font (size 1.27 1.27)) hide)
     )
@@
       (effects (font (size 1.27 1.27)) (justify right))
     )
-    (property "Footprint" "easyeda2kicad:RES-ADJ-SMD_RDC506002A" (at 200.025 125.73 0)
-      (effects (font (size 1.27 1.27)) hide)
-    )
-    (property "Datasheet" "~" (at 200.025 125.73 0)
-      (effects (font (size 1.27 1.27)) hide)
-    )
-    (property "LCSC" "C115341" (at 200.025 125.73 0)
-      (effects (font (size 1.27 1.27)) hide)
-    )
-    (property "Inventory" "" (at 200.025 125.73 0)
+    (property "Footprint" "easyeda2kicad:RES-ADJ-TH_3P-L10.0-W10.0-P2.50-L" (at 200.025 125.73 0)
+      (effects (font (size 1.27 1.27)) hide)
+    )
+    (property "Datasheet" "https://datasheet.lcsc.com/lcsc/1811071811_BOCHEN-Chengdu-Guosheng-Tech-3296W-1-103_C118954.pdf" (at 200.025 125.73 0)
+      (effects (font (size 1.27 1.27)) hide)
+    )
+    (property "LCSC" "C118954" (at 200.025 125.73 0)
+      (effects (font (size 1.27 1.27)) hide)
+    )
+    (property "Inventory" "E" (at 200.025 125.73 0)
       (effects (font (size 1.27 1.27)) hide)
     )
@@
       (effects (font (size 1.27 1.27)) hide)
     )
-    (property "Inventory" "" (at 172.72 73.025 0)
+    (property "Inventory" "B" (at 172.72 73.025 0)
       (effects (font (size 1.27 1.27)) hide)
     )
@@
     )
   )
-  (symbol (lib_id "Device:C_Polarized_Small") (at 161.29 73.025 0) (unit 1)
+  (symbol (lib_id "Device:C_Small") (at 161.29 73.025 0) (unit 1)
     (in_bom yes) (on_board yes) (dnp no)
     (property "Reference" "C11" (at 157.48 75.565 0)
@@
       (effects (font (size 1.27 1.27)) (justify left))
     )
-    (property "Footprint" "Capacitor_SMD:CP_Elec_5x5.4" (at 161.29 73.025 0)
-      (effects (font (size 1.27 1.27)) hide)
-    )
-    (property "Datasheet" "~" (at 161.29 73.025 0)
-      (effects (font (size 1.27 1.27)) hide)
-    )
-    (property "LCSC" "C335978" (at 161.29 73.025 0)
-      (effects (font (size 1.27 1.27)) hide)
-    )
-    (property "Inventory" "" (at 161.29 73.025 0)
+    (property "Footprint" "Capacitor_SMD:C_0805_2012Metric" (at 161.29 73.025 0)
+      (effects (font (size 1.27 1.27)) hide)
+    )
+    (property "Datasheet" "https://datasheet.lcsc.com/lcsc/2304140030_Samsung-Electro-Mechanics-CL21A106KAYNNNE_C15850.pdf" (at 161.29 73.025 0)
+      (effects (font (size 1.27 1.27)) hide)
+    )
+    (property "LCSC" "C15850" (at 161.29 73.025 0)
+      (effects (font (size 1.27 1.27)) hide)
+    )
+    (property "Inventory" "B" (at 161.29 73.025 0)
       (effects (font (size 1.27 1.27)) hide)
     )
@@
       (effects (font (size 1.27 1.27)) (justify right))
     )
-    (property "Footprint" "easyeda2kicad:RES-ADJ-SMD_RDC506002A" (at 163.195 112.395 0)
-      (effects (font (size 1.27 1.27)) hide)
-    )
-    (property "Datasheet" "~" (at 163.195 112.395 0)
-      (effects (font (size 1.27 1.27)) hide)
-    )
-    (property "LCSC" "C115341" (at 163.195 112.395 0)
-      (effects (font (size 1.27 1.27)) hide)
-    )
-    (property "Inventory" "" (at 163.195 112.395 0)
+    (property "Footprint" "easyeda2kicad:RES-ADJ-TH_RK09K1130AJ3" (at 163.195 112.395 0)
+      (effects (font (size 1.27 1.27)) hide)
+    )
+    (property "Datasheet" "https://datasheet.lcsc.com/lcsc/2304140030_ALPSALPINE-RK09K1130AP5_C470295.pdf" (at 163.195 112.395 0)
+      (effects (font (size 1.27 1.27)) hide)
+    )
+    (property "LCSC" "C470295" (at 163.195 112.395 0)
+      (effects (font (size 1.27 1.27)) hide)
+    )
+    (property "Inventory" "E" (at 163.195 112.395 0)
       (effects (font (size 1.27 1.27)) hide)
     )
@@
       (effects (font (size 1.27 1.27)) (justify right))
     )
-    (property "Footprint" "easyeda2kicad:RES-ADJ-SMD_RDC506002A" (at 180.975 119.38 0)
-      (effects (font (size 1.27 1.27)) hide)
-    )
-    (property "Datasheet" "~" (at 180.975 119.38 0)
-      (effects (font (size 1.27 1.27)) hide)
-    )
-    (property "LCSC" "C115341" (at 180.975 119.38 0)
-      (effects (font (size 1.27 1.27)) hide)
-    )
-    (property "Inventory" "" (at 180.975 119.38 0)
-      (effects (font (size 1.27 1.27)) hide)
-    )
+    (property "Footprint" "easyeda2kicad:RES-ADJ-TH_RK09K1130AJ3" (at 180.975 119.38 0)
+      (effects (font (size 1.27 1.27)) hide)
+    )
+    (property "Datasheet" "https://datasheet.lcsc.com/lcsc/2304140030_ALPSALPINE-RK09K1130AP5_C470295.pdf" (at 180.975 119.38 0)
+      (effects (font (size 1.27 1.27)) hide)
+    )
+    (property "LCSC" "C470295" (at 180.975 119.38 0)
+      (effects (font (size 1.27 1.27)) hide)
+    )
+    (property "Inventory" "E" (at 180.975 119.38 0)
+      (effects (font (size 1.27 1.27)) hide)
+    )
