File: scan-controller-kicad/userinterface.kicad_sch (KiCad schematic)
At the start: 27 parts, among them SW1 Power, SW10 Rec, SW2 Lamp, SW3 Zoom, SW4 <<, SW5 <, SW7 Stop, SW8 >, SW9 >>

Commit message: Changes shape to hold the cehapo 5.0" Display as cover
Parts:
- RV1, RV2: footprint easyeda2kicad:RES-ADJ-TH_RK09K1130AJ3 -> easyeda2kicad:RES-TH_RK09K1110A0J; LCSC C470295 -> C209767
- SW1: footprint easyeda2kicad:KEY-TH_4P-L12.0-W12.0-P5.0-LS12.5-EH-small -> easyeda2kicad:KEY-TH_4P-L7.3-W10.2-P4.50-LS7.0; Inventory (none) -> E; LCSC C93156 -> C231320
Changed lines of the file:
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@@
       (effects (font (size 1.27 1.27)))
     )
-    (property "Footprint" "easyeda2kicad:KEY-TH_4P-L12.0-W12.0-P5.0-LS12.5-EH-small" (at 120.65 49.53 0)
+    (property "Footprint" "easyeda2kicad:KEY-TH_4P-L7.3-W10.2-P4.50-LS7.0" (at 120.65 49.53 0)
       (effects (font (size 1.27 1.27)) hide)
     )
@@
       (effects (font (size 1.27 1.27)) hide)
     )
-    (property "LCSC" "C93156" (at 120.65 39.37 0)
-      (effects (font (size 1.27 1.27)) hide)
-    )
-    (property "Inventory" "" (at 120.65 39.37 0)
+    (property "LCSC" "C231320" (at 120.65 39.37 0)
+      (effects (font (size 1.27 1.27)) hide)
+    )
+    (property "Inventory" "E" (at 120.65 39.37 0)
       (effects (font (size 1.27 1.27)) hide)
     )
@@
       (effects (font (size 1.27 1.27)) (justify right))
     )
-    (property "Footprint" "easyeda2kicad:RES-ADJ-TH_RK09K1130AJ3" (at 163.195 112.395 0)
+    (property "Footprint" "easyeda2kicad:RES-TH_RK09K1110A0J" (at 163.195 112.395 0)
       (effects (font (size 1.27 1.27)) hide)
     )
@@
       (effects (font (size 1.27 1.27)) hide)
     )
-    (property "LCSC" "C470295" (at 163.195 112.395 0)
+    (property "LCSC" "C209767" (at 163.195 112.395 0)
       (effects (font (size 1.27 1.27)) hide)
     )
@@
       (effects (font (size 1.27 1.27)) (justify right))
     )
-    (property "Footprint" "easyeda2kicad:RES-ADJ-TH_RK09K1130AJ3" (at 180.975 119.38 0)
+    (property "Footprint" "easyeda2kicad:RES-TH_RK09K1110A0J" (at 180.975 119.38 0)
       (effects (font (size 1.27 1.27)) hide)
     )
@@
       (effects (font (size 1.27 1.27)) hide)
     )
-    (property "LCSC" "C470295" (at 180.975 119.38 0)
-      (effects (font (size 1.27 1.27)) hide)
-    )
+    (property "LCSC" "C209767" (at 180.975 119.38 0)
+      (effects (font (size 1.27 1.27)) hide)
+    )

Commit message: Adding a switch for Storage Target
Parts:
- added J2: Target, Connector_PinHeader_2.54mm:PinHeader_1x03_P2.54mm_Vertical, symbol Connector_Generic:Conn_01x03
- added R20 (x2): 47K, Resistor_SMD:R_0805_2012Metric, symbol Device:R_Small
- added SW11: Target, easyeda2kicad:SW-SMD_MK-12C02-G025, symbol Switch:SW_SPDT
Connections:
- net 3.3V-uC: now also J2.1 (Pin_1), R20.1
- net GNDD: now also J2.3 (Pin_3), R20.2
- new net: R20.2, SW11.1 (A)
- new net: R20.1, SW11.3 (C)
- new net Storage Target: J2.2 (Pin_2), SW11.2 (B)

Commit message: Fixing BOM
Parts:
- J2: now left out of the parts list
- SW11: footprint easyeda2kicad:SW-SMD_MK-12C02-G025 -> easyeda2kicad:SW-SMD_3P-P1.50_L2.7-W6.6; LCSC C778186 -> C319020
Changed lines of the file:
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@@
       (effects (font (size 1.27 1.27)))
     )
-    (property "Footprint" "easyeda2kicad:SW-SMD_MK-12C02-G025" (at 173.99 40.64 0)
-      (effects (font (size 1.27 1.27)) hide)
-    )
-    (property "Datasheet" "https://datasheet.lcsc.com/lcsc/2304140030_G-Switch-MK-12C02-G025_C778186.pdf" (at 173.99 40.64 0)
-      (effects (font (size 1.27 1.27)) hide)
-    )
-    (property "LCSC" "C778186" (at 173.99 40.64 0)
+    (property "Footprint" "easyeda2kicad:SW-SMD_3P-P1.50_L2.7-W6.6" (at 173.99 40.64 0)
+      (effects (font (size 1.27 1.27)) hide)
+    )
+    (property "Datasheet" "https://datasheet.lcsc.com/lcsc/2110151630_XKB-Connectivity-SK-3296S-01-L1_C319020.pdf" (at 173.99 40.64 0)
+      (effects (font (size 1.27 1.27)) hide)
+    )
+    (property "LCSC" "C319020" (at 173.99 40.64 0)
       (effects (font (size 1.27 1.27)) hide)
     )
@@
   )
   (symbol (lib_id "Connector_Generic:Conn_01x03") (at 187.325 48.895 0) (unit 1)
-    (in_bom yes) (on_board yes) (dnp no)
+    (in_bom no) (on_board yes) (dnp no)
     (property "Reference" "J2" (at 186.055 43.815 0)
       (effects (font (size 1.27 1.27)) (justify left))

Commit message: Reduced Power LED Brightness (0.3 mA @ 2.2V, wow), FIxed Power Switch Footprint
Parts:
- R21: value 220R -> 3K3
- SW1: symbol easyeda2kicad:B3F-5000_sm -> easyeda2kicad:B3F-3152; LCSC Part (none) -> C231320
Connections:
- net GNDD: now also SW1.1; no longer SW1.3, SW1.4
- net Power: no longer SW1.1
Changed lines of the file:
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@@
     (effects (font (size 1.27 1.27)) (justify left))
   )
-  (hierarchical_label "Power" (shape input) (at 124.46 39.37 0) (fields_autoplaced)
+  (hierarchical_label "Power" (shape input) (at 132.08 39.37 0) (fields_autoplaced)
     (effects (font (size 1.27 1.27)) (justify left))
   )
@@
     )
   )
-  (symbol (lib_id "easyeda2kicad:B3F-5000_sm") (at 120.65 39.37 0) (unit 1)
-    (in_bom yes) (on_board yes) (dnp no)
-    (property "Reference" "SW1" (at 124.46 37.465 0)
-      (effects (font (size 1.27 1.27)) hide)
-    )
-    (property "Value" "Power" (at 120.65 41.91 0)
-      (effects (font (size 1.27 1.27)))
-    )
-    (property "Footprint" "easyeda2kicad:KEY-TH_4P-L7.3-W10.2-P4.50-LS7.0" (at 120.65 49.53 0)
-      (effects (font (size 1.27 1.27)) hide)
-    )
-    (property "Datasheet" "https://lcsc.com/product-detail/Others_Omron-Electronics_B3F-5000_Omron-Electronics-B3F-5000_C93156.html" (at 120.65 52.07 0)
-      (effects (font (size 1.27 1.27)) hide)
-    )
-    (property "LCSC Part" "" (at 120.65 54.61 0)
-      (effects (font (size 1.27 1.27)) hide)
-    )
-    (property "LCSC" "C231320" (at 120.65 39.37 0)
-      (effects (font (size 1.27 1.27)) hide)
-    )
-    (property "Inventory" "E" (at 120.65 39.37 0)
+  (symbol (lib_id "easyeda2kicad:B3F-3152") (at 124.46 41.91 0) (unit 1)
+    (in_bom yes) (on_board yes) (dnp no)
+    (property "Reference" "SW1" (at 128.27 40.005 0)
+      (effects (font (size 1.27 1.27)) hide)
+    )
+    (property "Value" "Power" (at 124.46 44.45 0)
+      (effects (font (size 1.27 1.27)))
+    )
+    (property "Footprint" "easyeda2kicad:KEY-TH_4P-L7.3-W10.2-P4.50-LS7.0" (at 124.46 49.53 0)
+      (effects (font (size 1.27 1.27)) hide)
+    )
+    (property "Datasheet" "https://lcsc.com/product-detail/Others_Omron-Electronics_B3F-3152_Omron-Electronics-B3F-3152_C231320.html" (at 124.46 52.07 0)
+      (effects (font (size 1.27 1.27)) hide)
+    )
+    (property "LCSC Part" "C231320" (at 124.46 54.61 0)
+      (effects (font (size 1.27 1.27)) hide)
+    )
+    (property "LCSC" "C231320" (at 124.46 41.91 0)
+      (effects (font (size 1.27 1.27)) hide)
+    )
+    (property "Inventory" "E" (at 124.46 41.91 0)
       (effects (font (size 1.27 1.27)) hide)
     )
@@
       (effects (font (size 1.27 1.27)) (justify left))
     )
-    (property "Value" "220R" (at 175.26 65.405 90)
-      (effects (font (size 1.27 1.27)) (justify left))
-    )
+    (property "Value" "3K3" (at 175.26 65.405 90)
+      (effects (font (size 1.27 1.27)) (justify left))
+    )

Commit message: Freeing up D4 (328) as it isn't needed
Parts:
- renumbered C13 to C11, D6 to D2, D5 to D3, J2 to J7, R25 to R10, R28 to R11, R29 to R12, R30 to R13, R31 to R14, R26 to R15, R32 to R16, R21 to R17, R20 to R18, R20 to R41, R20 to R42, R22 to R7, R23 to R8, R24 to R9, SW1 to SW10, SW7 to SW6, SW8 to SW7, SW9 to SW8, SW10 to SW9
Connections:
- net 3.3V-uC: now also J7.3 (Pin_3); no longer J7.1 (Pin_1)
- net GNDD: now also J7.1 (Pin_1); no longer J7.3 (Pin_3)

Commit message: Replacing D6 LED with 1N4148 Adding TPs for Lamp Current Fixing TP Labels and other Labels Add LED D9 that actually reflects Lamp status Add control LEDs for Eyes (makes mounting much easier) Add mini manual and tech specs on the back side
Parts:
- removed D3: Film End (re), LED_SMD:LED_0805_2012Metric, symbol Device:LED_Small
- removed R18: 300R, Resistor_SMD:R_0805_2012Metric, symbol Device:R_Small
- R17: LCSC C17557 -> C26010
Changed lines of the file:
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@@
-    (stroke (width 0) (type default))
-  )
-  (wire (pts (xy 219.075 64.135) (xy 219.075 67.945))
     (stroke (width 0) (type default))
   )
@@
     (stroke (width 0) (type default))
   )
-  (wire (pts (xy 219.075 73.025) (xy 219.075 74.93))
-    (stroke (width 0) (type default))
-  )
   (wire (pts (xy 200.025 128.27) (xy 200.025 130.81))
     (stroke (width 0) (type default))
@@
     (stroke (width 0) (type default))
   )
-  (wire (pts (xy 219.075 80.01) (xy 219.075 81.915))
-    (stroke (width 0) (type default))
-  )
   (wire (pts (xy 111.125 124.46) (xy 111.125 125.73))
     (stroke (width 0) (type default))
@@
   )
   (wire (pts (xy 125.73 80.645) (xy 125.73 88.265))
-    (stroke (width 0) (type default))
-  )
-  (wire (pts (xy 213.995 64.135) (xy 219.075 64.135))
     (stroke (width 0) (type default))
   )
@@
     (effects (font (size 1.27 1.27)) (justify left))
   )
-  (hierarchical_label "Film End LED" (shape input) (at 213.995 64.135 180) (fields_autoplaced)
-    (effects (font (size 1.27 1.27)) (justify right))
-  )
   (hierarchical_label "Keys 1" (shape input) (at 130.81 65.405 0) (fields_autoplaced)
     (effects (font (size 1.27 1.27)) (justify left))
@@
         (path "/ab6dbce1-4ecf-44ae-8f33-5f07e4f43ca9/486b6b54-3904-49a9-9b52-9c586c7b0887"
           (reference "SW5") (unit 1)
-        )
-      )
-    )
-  )
-  (symbol (lib_id "Device:R_Small") (at 219.075 70.485 0) (unit 1)
-    (in_bom yes) (on_board yes) (dnp no)
-    (property "Reference" "R18" (at 215.9 72.39 90)
-      (effects (font (size 1.27 1.27)) (justify left))
-    )
-    (property "Value" "300R" (at 221.615 71.755 90)
-      (effects (font (size 1.27 1.27)) (justify left))
-    )
-    (property "Footprint" "Resistor_SMD:R_0805_2012Metric" (at 219.075 70.485 0)
-      (effects (font (size 1.27 1.27)) hide)
-    )
-    (property "Datasheet" "~" (at 219.075 70.485 0)
-      (effects (font (size 1.27 1.27)) hide)
-    )
-    (property "LCSC" "C17617" (at 219.075 70.485 0)
-      (effects (font (size 1.27 1.27)) hide)
-    )
-    (property "Inventory" "B" (at 219.075 70.485 0)
-      (effects (font (size 1.27 1.27)) hide)
-    )
-    (pin "1")
-    (pin "2")
-    (instances
-      (project "scan-controller-kicad"
-        (path "/ab6dbce1-4ecf-44ae-8f33-5f07e4f43ca9/486b6b54-3904-49a9-9b52-9c586c7b0887"
-          (reference "R18") (unit 1)
         )
       )
@@
     )
   )
-  (symbol (lib_id "power:GNDD") (at 219.075 81.915 0) (unit 1)
-    (in_bom yes) (on_board yes) (dnp no)
-    (property "Reference" "#PWR020" (at 219.075 88.265 0)
-      (effects (font (size 1.27 1.27)) hide)
-    )
-    (property "Value" "GNDD" (at 219.075 85.725 0)
-      (effects (font (size 1.27 1.27)))
-    )
-    (property "Footprint" "" (at 219.075 81.915 0)
-      (effects (font (size 1.27 1.27)) hide)
-    )
-    (property "Datasheet" "" (at 219.075 81.915 0)
-      (effects (font (size 1.27 1.27)) hide)
-    )
-    (pin "1")
-    (instances
-      (project "scan-controller-kicad"
-        (path "/ab6dbce1-4ecf-44ae-8f33-5f07e4f43ca9/486b6b54-3904-49a9-9b52-9c586c7b0887"
-          (reference "#PWR020") (unit 1)
-        )
-      )
-    )
-  )
   (symbol (lib_id "Device:R_Small") (at 177.8 67.945 270) (unit 1)
     (in_bom yes) (on_board yes) (dnp no)
@@
       (effects (font (size 1.27 1.27)) hide)
     )
-    (property "LCSC" "C17557" (at 177.8 67.945 0)
+    (property "LCSC" "C26010" (at 177.8 67.945 0)
       (effects (font (size 1.27 1.27)) hide)
     )
@@
         )
       )
-    )
-  )
-  (symbol (lib_id "Device:LED_Small") (at 219.075 77.47 90) (unit 1)
-    (in_bom yes) (on_board yes) (dnp no)
-    (property "Reference" "D3" (at 215.9 77.47 0)
-      (effects (font (size 1.27 1.27)))
-    )
-    (property "Value" "Film End (re)" (at 227.33 78.105 90)
-      (effects (font (size 1.27 1.27)))
-    )
-    (property "Footprint" "LED_SMD:LED_0805_2012Metric" (at 219.075 77.47 90)
-      (effects (font (size 1.27 1.27)) hide)
-    )
-    (property "Datasheet" "https://datasheet.lcsc.com/lcsc/2304140030_Foshan-NationStar-Optoelectronics-NCD0805R1_C84256.pdf" (at 219.075 77.47 90)
-      (effects (font (size 1.27 1.27)) hide)
-    )
-    (property "LCSC" "C84256" (at 219.075 77.47 0)
-      (effects (font (size 1.27 1.27)) hide)
-    )
-    (property "Inventory" "B" (at 219.075 77.47 0)
-      (effects (font (size 1.27 1.27)) hide)
-    )
-    (pin "1")
-    (pin "2")
-    (instances
-      (project "scan-controller-kicad"
-        (path "/ab6dbce1-4ecf-44ae-8f33-5f07e4f43ca9/486b6b54-3904-49a9-9b52-9c586c7b0887"
-          (reference "D3") (unit 1)
-        )
-      )

Commit message: Reannotated
Parts:
- renumbered C11 to C13, D2 to D1, J7 to J4, R16 to R13, R42 to R2, R7 to R21, R15 to R23, R8 to R25, R9 to R28, R11 to R32, R10 to R35, R13 to R37, R12 to R39, R41 to R4, R14 to R40, R17 to R7, RV3 to RV2, RV2 to RV4, RV1 to RV5, SW10 to SW1, SW8 to SW10, SW9 to SW11, SW11 to SW2, SW2 to SW4, SW4 to SW5, SW3 to SW6, SW6 to SW7, SW5 to SW8, SW7 to SW9

Commit message: Updated the Power Switch
Parts:
- SW1: footprint easyeda2kicad:KEY-TH_4P-L7.3-W10.2-P4.50-LS7.0 -> easyeda2kicad:KEY-TH_1825027-8; LCSC C231320 -> C266196
Changed lines of the file:
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@@
       (effects (font (size 1.27 1.27)))
     )
-    (property "Footprint" "easyeda2kicad:KEY-TH_4P-L7.3-W10.2-P4.50-LS7.0" (at 124.46 49.53 0)
+    (property "Footprint" "easyeda2kicad:KEY-TH_1825027-8" (at 124.46 49.53 0)
       (effects (font (size 1.27 1.27)) hide)
     )
@@
       (effects (font (size 1.27 1.27)) hide)
     )
-    (property "LCSC" "C231320" (at 124.46 41.91 0)
+    (property "LCSC" "C266196" (at 124.46 41.91 0)
       (effects (font (size 1.27 1.27)) hide)
     )
@@
       (effects (font (size 1.27 1.27)) hide)
     )
+    (property "Sim.Device" "C231320" (at 124.46 41.91 0)
+      (effects (font (size 1.27 1.27)) hide)
+    )
