File: scan-controller-kicad/userinterface.kicad_sch (KiCad schematic)
At the start: 29 parts, among them J4 Target, SW1 Power, SW10 >>, SW11 Rec, SW2 Target, SW4 Lamp, SW5 <<, SW6 Zoom, SW7 Stop, SW8 <, SW9 >

Commit message: Preparing for bootstrap-ability
Other:
- moved on the sheet: C13, D1, J4, R13, R2, R21, R23, R25, R28, R32, R35, R37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
