File: scan-controller-kicad/scan-controller-kicad.kicad_pcb (KiCad board)
At the start: 2 copper layers, 132.1 x 101.6 mm, 130 parts, among them CN1 24V in, CN2 Shaft Eye, CN3 Film End Eye, CN4 Fan, CN5 Motor, CN6 Lamp, J1 Raspi GPIO, J2 Raspi UART, J3 ICSP, J4 FTDI, J5 Shaft Eye, J6 Film End Eye, Q1 IRLML2502, Q2 IRLML6402, Q3 DMMT5401, Q4 DMG2305UX, Q5 SS8050, Q6 SS8050, Q7 IRF7470, SW1 Reset, SW10 Power, SW2 Lamp, SW3 Zoom, SW4 <<, SW5 <, SW6 Stop, SW7 >, SW8 >>, SW9 Rec, U1 ATmega328P, U2 74LVC14, U3 QRE1113, U4 QRE1113, U5 DRV8871DDA, U6 78L05, U7 XL4015, U8 TL431, U9 LM358, Y1 8MHz

Commit message: Backzp before upgrading to Kicad Nightly due to DRC errors
Parts:
- moved TP8 0.51 mm to (142.2, 106.9)
- moved REF** 0.25 mm to (111.4, 71.6)
- moved C23 0.16 mm to (207.5, 106.6)
- moved CN2 0.16 mm to (223.4, 128.2)
- moved CN6 0.16 mm to (223.4, 97.7)
- moved R14 0.16 mm to (221.9, 133.5)
- moved R6 0.16 mm to (188.1, 118.3)
- moved SW3 0.16 mm to (149.7, 142.2)
- moved SW6 0.16 mm to (187.8, 142.2)
- moved SW8 0.16 mm to (213.2, 142.2)
- moved TP4 0.16 mm to (170.8, 130.7)
- moved C1 0.16 mm to (195.4, 74.2)
- moved C18 0.16 mm to (179.6, 74.2)
- moved C2 0.16 mm to (210.9, 124.1)
- moved C20 0.16 mm to (168.5, 88.6)
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Routing:
- net Net-(U5-OUT2): track 72.4 -> 14.6 mm
- net Net-(U5-OUT1): track 65.1 -> 15.0 mm
- net 3.3V-uC: track 87.8 -> 71.2 mm
- net /GPIO26: track 148.4 -> 143.3 mm
- net Net-(D6-K): vias 6 -> 5
- net /SCL: vias 7 -> 6

Commit message: Pushbutton PTHs now mechanical (DRC fun)
Parts:
- removed REF** (x2): MountingHole_2.2mm_M2_ISO7380_Pad_TopBottom, MountingHole:MountingHole_2.2mm_M2_ISO7380_Pad_TopBottom
- moved R6 1.11 mm to (186.9, 118.3)
- moved R1 1.09 mm to (182.9, 118.3)
- moved R18 0.64 mm to (230.4, 133.5)
- moved R14 0.37 mm to (221.5, 133.5)
Connections:
- net Net-(CN1-Pad1) renamed /24VAC-1
- net Net-(CN1-Pad2) renamed /24VAC-2
- net Net-(U5-OUT1) renamed /Drivers/Mot-A
- net Net-(U5-OUT2) renamed /Drivers/Mot-B
Routing:
- net Net-(Q3B-C2): track 15.7 -> 17.1 mm
- net /uC-Power: track 27.0 -> 25.9 mm
- net Net-(R13-Pad2): track 16.1 -> 17.1 mm, vias 0 -> 1
- net Net-(J5-Pin_2): track 7.72 -> 8.61 mm
- net Net-(D3-A): track 1.96 -> 2.60 mm

Commit message: Fixes all Footprint DRC Errors
Parts:
- moved D1 1.32 mm to (209.4, 71.0)
- moved CN1 1.19 mm to (223.4, 71.1)
- moved CN6 0.81 mm to (223.4, 96.9)
- moved CN5 0.78 mm to (223.4, 84.1)
- moved U5 0.68 mm to (210.0, 84.3)
- moved CN4 0.55 mm to (223.4, 107.3)
- moved CN3 0.30 mm to (223.4, 117.7)
Routing:
- net /24VAC-1: track 48.0 -> 0.00 mm
- net /24VAC-2: track 47.9 -> 0.00 mm
- net 24VDC: track 148.5 -> 127.6 mm
- net /Drivers/Mot-A: track 15.0 -> 0.00 mm
- net /Drivers/Mot-B: track 14.6 -> 0.00 mm
- net 5V-RPi: track 50.1 -> 45.1 mm
- net GND: track 84.3 -> 86.2 mm
- net Net-(U6-OUT): track 49.3 -> 47.6 mm
- net Net-(U5-ILIM): track 2.56 -> 3.25 mm
- net Net-(Q1-G): track 12.9 -> 12.5 mm, vias 0 -> 2
- added copper zone on F.Cu, net /24VAC-1
- added copper zone on F.Cu, net /24VAC-2
- added copper zone on F.Cu, net /Drivers/Mot-A
- added copper zone on F.Cu, net /Drivers/Mot-B
- added copper zone on F.Cu, net 24VDC

Commit message: DRC Happy!
Parts:
- moved R33 0.33 mm to (172.3, 88.9)
- moved J2 0.33 mm to (198.8, 130.0)
Routing:
- net Net-(D5-K): track 28.0 -> 28.7 mm

Commit message: smaller eyes
Parts:
- R19, R20, R21, R22: footprint Resistor_SMD:R_0805_2012Metric -> Resistor_SMD:R_0402_1005Metric
- moved R22 1.85 mm to (112.4, 61.5), turned to 90 degrees
- moved R21 1.75 mm to (112.3, 73.2), turned to 90 degrees
- moved R20 1.69 mm to (112.4, 58.3), turned to -90 degrees
- moved R19 1.64 mm to (112.3, 70.0), turned to -90 degrees
Routing:
- net GND: track 86.2 -> 76.7 mm
- net 3.3V-uC: track 71.2 -> 72.2 mm
- net Net-(J6-Pin_2): track 7.97 -> 8.81 mm, vias 0 -> 1
- net Net-(J5-Pin_2): track 8.61 -> 8.79 mm, vias 0 -> 1

Commit message: Mount Holes 2/6
Parts:
- added REF**: MountingHole_2.2mm_M2_ISO7380_Pad_TopBottom, MountingHole:MountingHole_2.2mm_M2_ISO7380_Pad_TopBottom, F.Cu at (111.3, 59.9)
- added REF**: MountingHole_2.2mm_M2_ISO7380_Pad_TopBottom, MountingHole:MountingHole_2.2mm_M2_ISO7380_Pad_TopBottom, F.Cu at (111.3, 71.6)
- moved R21 1.14 mm to (112.8, 74.2), turned to 0 degrees
- moved R22 1.09 mm to (112.8, 62.5), turned to 0 degrees
- moved R19 1.02 mm to (112.8, 69.1), turned to 0 degrees
- moved R20 0.97 mm to (112.8, 57.4), turned to 0 degrees
Routing:
- net Net-(U3-A): track 2.64 -> 1.20 mm
- net Net-(U4-A): track 2.57 -> 1.21 mm
- net Net-(J6-Pin_2): track 8.81 -> 10.2 mm, vias 1 -> 2
- net Net-(J5-Pin_2): track 8.79 -> 10.1 mm, vias 1 -> 2
Other:
- outline, holes or cut-outs redrawn

Commit message: Round corners!
Parts:
- removed the REF** at (111.3, 59.9)
- removed the REF** at (111.3, 71.6)
- added REF**: MountingHole_2.2mm_M2_ISO7380_Pad_TopBottom, MountingHole:MountingHole_2.2mm_M2_ISO7380_Pad_TopBottom, F.Cu at (112.0, 85.9)
- added REF**: MountingHole_3.2mm_M3_Pad_Via, MountingHole:MountingHole_3.2mm_M3_Pad_Via, F.Cu at (127.0, 151.9)
- added REF**: Eye_Mousebites, Peacemans_Footprints:Eye_Mousebites, F.Cu at (121.2, 74.2)
- added REF**: MountingHole_3.2mm_M3_Pad_Via, MountingHole:MountingHole_3.2mm_M3_Pad_Via, F.Cu at (235.5, 151.8)
- added REF**: MountingHole_3.2mm_M3_Pad_Via, MountingHole:MountingHole_3.2mm_M3_Pad_Via, F.Cu at (235.5, 62.0)
- added REF**: MountingHole_3.2mm_M3_Pad_Via, MountingHole:MountingHole_3.2mm_M3_Pad_Via, F.Cu at (127.0, 62.0)
- added REF**: Eye_Mousebites, Peacemans_Footprints:Eye_Mousebites, F.Cu at (121.2, 85.9)
- added REF**: MountingHole_2.2mm_M2_ISO7380_Pad_TopBottom, MountingHole:MountingHole_2.2mm_M2_ISO7380_Pad_TopBottom, F.Cu at (112.0, 74.2)
- moved R21 14.8 mm to (113.5, 88.9)
- moved R22 14.8 mm to (113.5, 77.2)
- moved J5 14.2 mm to (119.5, 83.3)
- moved U3 14.2 mm to (115.7, 85.9)
- moved U4 14.2 mm to (115.7, 74.2)
- moved J6 14.2 mm to (119.5, 71.7)
- moved R19 13.7 mm to (113.5, 82.8)
- moved R20 13.7 mm to (113.5, 71.1)
Connections:
- J5 pad 1: 3.3V-uC -> /Sensors/3.3V-Eye2
- J5 pad 3: GND -> GND2
- J6 pad 1: 3.3V-uC -> /Sensors/3.3V-Eye1
- J6 pad 3: GND -> GND1
- R19 pad 1: 3.3V-uC -> /Sensors/3.3V-Eye2
- R20 pad 1: 3.3V-uC -> /Sensors/3.3V-Eye1
- R21 pad 1: 3.3V-uC -> /Sensors/3.3V-Eye2
- R22 pad 1: 3.3V-uC -> /Sensors/3.3V-Eye1
- U3 pad 2: GND -> GND2
- U3 pad 4: GND -> GND2
- U4 pad 2: GND -> GND1
- U4 pad 4: GND -> GND1
Routing:
- net 3.3V-uC: track 72.1 -> 68.0 mm, vias 13 -> 9
- net /Sensors/3.3V-Eye2: track 0.00 -> 2.77 mm, vias 0 -> 2
- net /Sensors/3.3V-Eye1: track 0.00 -> 2.76 mm, vias 0 -> 2
- net Net-(J6-Pin_2): track 10.2 -> 8.21 mm, vias 2 -> 1
- net Net-(J5-Pin_2): track 10.1 -> 8.21 mm, vias 2 -> 1
- added copper zone on B.Cu, net /Sensors/3.3V-Eye1
- added copper zone on B.Cu, net /Sensors/3.3V-Eye2
- added copper zone on F.Cu, net GND1
- added copper zone on F.Cu, net GND2
Other:
- board size 132.1 x 101.6 mm -> 131.3 x 101.6 mm
