File: scan-controller-kicad/scan-controller-kicad.kicad_pcb (KiCad board)
At the start: 2 copper layers, 122.2 x 113 mm, 136 parts, among them CN1 24V in, CN2 Shaft Eye, CN3 Film End Eye, CN4 Fan, CN5 Motor, CN6 Lamp, J1 Raspi GPIO, J2 Raspi UART, J3 ICSP, J4 FTDI, J5 Shaft Eye, J6 Film End Eye, Q1 IRLML2502, Q2 IRLML6402, Q3 DMMT5401, Q4 DMG2305UX, Q5 SS8050, Q6 SS8050, Q7 IRF7470, SW1 Reset, SW10 Power, SW2 Lamp, SW3 Zoom, SW4 <<, SW5 <, SW6 Stop, SW7 >, SW8 >>, SW9 Rec, U1 ATmega328P, U2 74LVC14, U3 QRE1113, U4 QRE1113, U5 DRV8871DDA, U6 78L05, U7 XL4015, U8 TL431, U9 LM358, Y1 8MHz

Commit message: More labels & cleanup
Other:
- board text added: "ICSP"
- board text added: "ICSP? Use other side!"
- board text added: "Power"
- board text added: "Raspberry Pi 4 goes here"
- board text added: "Run Speed"
- board text added: "Step Speed"
Changed lines of the file:
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@@
     (tags "mounting hole 2.2mm m2 iso7380")
     (attr exclude_from_pos_files exclude_from_bom)
-    (fp_text reference "REF**" (at 0 -2.75 90) (layer "F.SilkS")
+    (fp_text reference "REF**" (at 0 -2.75 90) (layer "F.SilkS") hide
         (effects (font (size 1 1) (thickness 0.15)))
     )
@@
     (property "ki_keywords" "connector")
     (attr through_hole)
-    (fp_text reference "J6" (at 0 -2.33 90) (layer "F.SilkS")
+    (fp_text reference "J6" (at 0 -2.33 90) (layer "F.SilkS") hide
         (effects (font (size 1 1) (thickness 0.15)))
     )
@@
     (property "ki_keywords" "connector")
     (attr through_hole)
-    (fp_text reference "J4" (at 2.8 12.04 90) (layer "F.SilkS")
+    (fp_text reference "J4" (at 2.8 12.04 90) (layer "F.SilkS") hide
         (effects (font (size 1 1) (thickness 0.15)))
     )
@@
     (tags "mounting hole 3.2mm m3")
     (attr exclude_from_pos_files exclude_from_bom)
-    (fp_text reference "REF**" (at 0 -4.2) (layer "F.SilkS")
+    (fp_text reference "REF**" (at 0 -4.2) (layer "F.SilkS") hide
         (effects (font (size 1 1) (thickness 0.15)))
     )
@@
     (property "ki_keywords" "AVR ISP Connector")
     (attr through_hole)
-    (fp_text reference "J3" (at 1.355237 7.677593 -180) (layer "F.SilkS")
+    (fp_text reference "J3" (at 1.355237 7.677593 180) (layer "F.SilkS") hide
         (effects (font (size 1 1) (thickness 0.15)))
     )
@@
     (property "ki_keywords" "resistor variable")
     (attr through_hole)
-    (fp_text reference "RV3" (at -2.57 2.962) (layer "F.SilkS")
+    (fp_text reference "RV3" (at -2.57 2.962) (layer "F.SilkS") hide
         (effects (font (size 1 1) (thickness 0.15)))
     )
@@
     (property "ki_keywords" "resistor variable")
     (attr through_hole)
-    (fp_text reference "RV1" (at 0 -5.65 180) (layer "F.SilkS")
+    (fp_text reference "RV1" (at 0 -5.65 180) (layer "F.SilkS") hide
         (effects (font (size 1 1) (thickness 0.15)))
     )
@@
     (property "ki_keywords" "R resistor")
     (attr smd)
-    (fp_text reference "R19" (at 0 -1.17 90) (layer "F.SilkS")
+    (fp_text reference "R19" (at 0 -1.17 90) (layer "F.SilkS") hide
         (effects (font (size 1 1) (thickness 0.15)))
     )
@@
     (property "ki_keywords" "LED diode light-emitting-diode")
     (attr smd)
-    (fp_text reference "D2" (at 2.833093 -0.207237 -270) (layer "F.SilkS")
+    (fp_text reference "D2" (at 2.606 0.052 -180) (layer "F.SilkS")
         (effects (font (size 1 1) (thickness 0.15)))
     )
@@
     (property "ki_keywords" "R resistor")
     (attr smd)
-    (fp_text reference "R22" (at 0 -1.17 90) (layer "F.SilkS")
+    (fp_text reference "R22" (at 0 -1.17 90) (layer "F.SilkS") hide
         (effects (font (size 1 1) (thickness 0.15)))
     )
@@
     (at 221.002 55.646)
     (attr through_hole)
-    (fp_text reference "REF**" (at 0 2.25) (layer "F.SilkS")
+    (fp_text reference "REF**" (at 0 2.25) (layer "F.SilkS") hide
         (effects (font (size 1 1) (thickness 0.15)))
     )
@@
     (property "ki_keywords" "Reflective Optical Sensor Opto reflex coupler")
     (attr through_hole)
-    (fp_text reference "U4" (at 0.0254 2.4892) (layer "F.SilkS")
+    (fp_text reference "U4" (at 0.0254 2.4892) (layer "F.SilkS") hide
         (effects (font (size 1 1) (thickness 0.15)))
     )
@@
     (property "Sheetname" "User Interface")
     (attr through_hole)
-    (fp_text reference "SW10" (at 0 -5.27) (layer "F.SilkS")
+    (fp_text reference "SW10" (at 0 -0.898) (layer "F.SilkS")
         (effects (font (size 1 1) (thickness 0.15)))
     )
@@
     (tags "mounting hole 3.2mm m3")
     (attr exclude_from_pos_files exclude_from_bom)
-    (fp_text reference "REFe" (at 0 -4.2) (layer "F.SilkS")
+    (fp_text reference "REFe" (at 0 -4.2) (layer "F.SilkS") hide
         (effects (font (size 1 1) (thickness 0.15)))
     )
@@
     (tags "mounting hole 3.2mm m3")
     (attr exclude_from_pos_files exclude_from_bom)
-    (fp_text reference "REFee" (at 0.254 -0.508) (layer "F.SilkS")
+    (fp_text reference "REFee" (at 0.254 -0.508) (layer "F.SilkS") hide
         (effects (font (size 1 1) (thickness 0.15)))
     )
@@
     (tags "mounting hole 3.2mm m3")
     (attr exclude_from_pos_files exclude_from_bom)
-    (fp_text reference "REF**" (at 0 -4.2) (layer "F.SilkS")
+    (fp_text reference "REF**" (at 0 -4.2) (layer "F.SilkS") hide
         (effects (font (size 1 1) (thickness 0.15)))
     )
@@
     (at 209.27 55.646)
     (attr through_hole)
-    (fp_text reference "REF**" (at 0 2.25) (layer "F.SilkS")
+    (fp_text reference "REF**" (at 0 2.25) (layer "F.SilkS") hide
         (effects (font (size 1 1) (thickness 0.15)))
     )
@@
     (property "ki_keywords" "quartz ceramic resonator oscillator")
     (attr smd)
-    (fp_text reference "Y1" (at 0 -2.8 90) (layer "F.SilkS")
+    (fp_text reference "Y1" (at 0 -2.975407 -180) (layer "F.SilkS")
         (effects (font (size 1 1) (thickness 0.15)))
     )
@@
     (tags "mounting hole 2.2mm m2 iso7380")
     (attr exclude_from_pos_files exclude_from_bom)
-    (fp_text reference "REF**" (at 0 -2.75 90) (layer "F.SilkS")
+    (fp_text reference "REF**" (at 0 -2.75 90) (layer "F.SilkS") hide
         (effects (font (size 1 1) (thickness 0.15)))
     )
@@
     (property "ki_keywords" "R resistor")
     (attr smd)
-    (fp_text reference "R21" (at 0 -1.17 90) (layer "F.SilkS")
+    (fp_text reference "R21" (at 0 -1.17 90) (layer "F.SilkS") hide
         (effects (font (size 1 1) (thickness 0.15)))
     )
@@
     (property "ki_keywords" "R resistor")
     (attr smd)
-    (fp_text reference "R17" (at 0 -1.65 -270) (layer "F.SilkS")
+    (fp_text reference "R17" (at 2.594 0.052 -180) (layer "F.SilkS")
         (effects (font (size 1 1) (thickness 0.15)))
     )
@@
     (property "ki_keywords" "resistor variable")
     (attr through_hole)
-    (fp_text reference "RV2" (at 0 -5.65 180) (layer "F.SilkS")
+    (fp_text reference "RV2" (at 0 0.126 180) (layer "F.SilkS") hide
         (effects (font (size 1 1) (thickness 0.15)))
     )
@@
     (property "ki_keywords" "Reflective Optical Sensor Opto reflex coupler")
     (attr through_hole)
-    (fp_text reference "U3" (at 0.0254 2.4892) (layer "F.SilkS")
+    (fp_text reference "U3" (at 0.0254 2.4892) (layer "F.SilkS") hide
         (effects (font (size 1 1) (thickness 0.15)))
     )
@@
     (property "ki_keywords" "connector")
     (attr through_hole)
-    (fp_text reference "J5" (at 0 -2.33 90) (layer "F.SilkS")
+    (fp_text reference "J5" (at 0 -2.33 90) (layer "F.SilkS") hide
         (effects (font (size 1 1) (thickness 0.15)))
     )
@@
     (property "ki_keywords" "R resistor")
     (attr smd)
-    (fp_text reference "R20" (at 0 -1.17 90) (layer "F.SilkS")
+    (fp_text reference "R20" (at 0 -1.17 90) (layer "F.SilkS") hide
         (effects (font (size 1 1) (thickness 0.15)))
     )
@@
     (property "ki_keywords" "resistor variable")
     (attr through_hole)
-    (fp_text reference "RV4" (at -2.384 3.062) (layer "F.SilkS")
+    (fp_text reference "RV4" (at -2.384 3.062) (layer "F.SilkS") hide
         (effects (font (size 1 1) (thickness 0.15)))
     )
@@
   (gr_line locked (start 129.75132 76.25132) (end 129.77132 126.22868)
     (stroke (width 0.15) (type default)) (layer "B.SilkS"))
+  (gr_rect (start 144.018 107.696) (end 151.892 113.284)
+    (stroke (width 0.15) (type default)) (fill none) (layer "B.SilkS"))
   (gr_line locked (start 214.75 126.25) (end 214.75 76.25)
     (stroke (width 0.15) (type default)) (layer "B.SilkS"))
@@
   (gr_line (start 233.3 55.9) (end 225.066 55.9)
     (stroke (width 0.1) (type default)) (layer "Edge.Cuts"))
+  (gr_text "ICSP? Use other side!" (at 151.892 106.934) (layer "B.SilkS")
+    (effects (font (size 1 1) (thickness 0.15)) (justify left bottom mirror))
+  )
+  (gr_text "Raspberry Pi 4 goes here" (at 192.024 102.362) (layer "B.SilkS")
+    (effects (font (size 2 2) (thickness 0.2)) (justify left bottom mirror))
+  )
   (gr_text "- +" (at 235.204 110.744 90) (layer "F.SilkS" knockout)
     (effects (font (size 2.5 2.5) (thickness 0.3)) (justify left bottom))
@@
     (effects (font (size 2.5 2.5) (thickness 0.3)) (justify left bottom))
   )
+  (gr_text "ICSP" (at 139.954 112.522) (layer "F.SilkS")
+    (effects (font (size 1 1) (thickness 0.15)) (justify left bottom))
+  )
+  (gr_text "Power" (at 132.842 64.77) (layer "F.SilkS" knockout)
+    (effects (font (size 1.5 1.5) (thickness 0.2)) (justify left bottom))
+  )
   (gr_text "24V in" (at 238.76 76.454 90) (layer "F.SilkS")
     (effects (font (size 2 2) (thickness 0.3)) (justify left bottom))
@@
     (effects (font (size 2 2) (thickness 0.3)) (justify left bottom))
   )
+  (gr_text "Run Speed" (at 143.764 71.882) (layer "F.SilkS" knockout)
+    (effects (font (size 1.5 1.5) (thickness 0.2)) (justify left bottom))
+  )
   (gr_text "End" (at 238.76 120.142 90) (layer "F.SilkS")
     (effects (font (size 2 2) (thickness 0.3)) (justify left bottom))
@@
     (effects (font (size 2 2) (thickness 0.3)) (justify left bottom))
   )
+  (gr_text "Step Speed" (at 159.258 71.882) (layer "F.SilkS" knockout)
+    (effects (font (size 1.5 1.5) (thickness 0.2)) (justify left bottom))
+  )
   (gr_text_box "Filmkorn-Scanner\nby filmkorn.org 2023 • Rev. A"

Commit message: Looks like we have a Rev. A
Other:
- board text added: "Current"
- board text added: "Exposure"
- board text added: "Voltage"
Changed lines of the file:
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@@
   (gr_line (start 233.3 55.9) (end 225.066 55.9)
     (stroke (width 0.1) (type default)) (layer "Edge.Cuts"))
-  (gr_text "ICSP? Use other side!" (at 151.892 106.934) (layer "B.SilkS")
+  (gr_text "ICSP? Use other side!" (at 152.146 105.664) (layer "B.SilkS")
     (effects (font (size 1 1) (thickness 0.15)) (justify left bottom mirror))
   )
@@
     (effects (font (size 2.5 2.5) (thickness 0.3)) (justify left bottom))
   )
+  (gr_text "Voltage" (at 199.898 58.928) (layer "F.SilkS" knockout)
+    (effects (font (size 1 1) (thickness 0.15)) (justify bottom))
+  )
   (gr_text "ICSP" (at 139.954 112.522) (layer "F.SilkS")
     (effects (font (size 1 1) (thickness 0.15)) (justify left bottom))
+  )
+  (gr_text "Current" (at 189.484 58.928) (layer "F.SilkS" knockout)
+    (effects (font (size 1 1) (thickness 0.15)) (justify bottom))
   )
   (gr_text "Power" (at 132.842 64.77) (layer "F.SilkS" knockout)
@@
     (effects (font (size 2.5 2.5) (thickness 0.3)) (justify left bottom))
   )
+  (gr_text "Exposure" (at 179.07 58.928) (layer "F.SilkS" knockout)
+    (effects (font (size 1 1) (thickness 0.15)) (justify bottom))
+  )
   (gr_text "Shaft" (at 238.76 132.08 90) (layer "F.SilkS")
