File: scan-controller-kicad/scan-controller-kicad.kicad_pcb (KiCad board)
At the start: 2 copper layers, 122.2 x 113 mm, 139 parts, among them CN1 24V in, CN2 Shaft Eye, CN3 Film End Eye, CN4 Fan, CN5 Motor, CN6 Lamp, J1 Raspi GPIO, J2 Raspi UART, J3 ICSP, J4 FTDI, J5 Shaft Eye, J6 Film End Eye, J7 Target, Q1 IRLML2502, Q2 IRLML6402, Q3 DMMT5401, Q4 DMG2305UX, Q5 SS8050, Q6 SS8050, Q7 IRF7470, SW1 Reset, SW10 Power, SW11 Target, SW2 Lamp, SW3 Zoom, SW4 <<, SW5 <, SW6 Stop, SW7 >, SW8 >>, SW9 Rec, U1 ATmega328P, U2 74LVC14, U3 QRE1113, U4 QRE1113, U5 DRV8871DDA, U6 78L05, U7 XL4015, U8 TL431, U9 LM358, Y1 8MHz

Commit message: Connect PGIO with SCL (instead of SDA) for power. Connect Atmega SDA to bus (was nc)
Routing:
- net /GPIO26: track 142.3 -> 149.5 mm
Other:
- board text added: "FTDI"
Changed lines of the file:
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@@
     (pad_to_mask_clearance 0)
     (aux_axis_origin 224.028 107.188)
+    (grid_origin 176.276 55.626)
     (pcbplotparams
       (layerselection 0x00010fc_ffffffff)
@@
     (effects (font (size 1.8 1.8) (thickness 0.3)) (justify bottom))
   )
+  (gr_text "FTDI" (at 120.904 62.23 -90) (layer "F.SilkS")
+    (effects (font (size 1.5 1.5) (thickness 0.3) bold) (justify left bottom))
+  )
   (gr_text "ICSP" (at 139.954 112.522) (layer "F.SilkS")
     (effects (font (size 1 1) (thickness 0.15)) (justify left bottom))
@@
       (effects (font (size 2 2) (thickness 0.2)) (justify left top mirror))
   )
-  (gr_text_box "Filmkorn-Scanner\nby filmkorn.org 2023 • Rev. A"
+  (gr_text_box "Filmkorn-Scanner\nby filmkorn.org 2023 • Rev. B"
     (start 129.45 79) (end 120.15 131.3) (angle 270) (layer "F.Mask")
       (effects (font (size 2 2) (thickness 0.2)) (justify left top))
@@
   (segment (start 163.359356 121.666) (end 160.645593 124.379763) (width 0.25) (layer "F.Cu") (net 54))
   (segment (start 141.986 89.408) (end 143.002 90.424) (width 0.25) (layer "F.Cu") (net 54))
-  (segment (start 153.599701 88.575701) (end 156.7 91.676) (width 0.25) (layer "F.Cu") (net 54))
+  (segment (start 150.622 89.408) (end 149.766788 89.408) (width 0.25) (layer "F.Cu") (net 54))
   (segment (start 156.073593 125.649763) (end 159.375593 125.649763) (width 0.25) (layer "F.Cu") (net 54))
   (segment (start 159.375593 125.649763) (end 160.645593 124.379763) (width 0.25) (layer "F.Cu") (net 54))
   (segment (start 203.317593 124.379763) (end 200.34983 121.412) (width 0.25) (layer "F.Cu") (net 54))
+  (segment (start 149.766788 89.408) (end 149.075593 90.099195) (width 0.25) (layer "F.Cu") (net 54))
   (segment (start 180.806415 121.666) (end 163.359356 121.666) (width 0.25) (layer "F.Cu") (net 54))
   (segment (start 203.825593 124.379763) (end 203.317593 124.379763) (width 0.25) (layer "F.Cu") (net 54))
-  (segment (start 156.7 91.676) (end 156.7 93) (width 0.25) (layer "F.Cu") (net 54))
+  (segment (start 151.384 90.17) (end 151.384 90.678) (width 0.25) (layer "F.Cu") (net 54))
   (segment (start 192.019119 120.569763) (end 181.902652 120.569763) (width 0.25) (layer "F.Cu") (net 54))
+  (segment (start 153.706 93) (end 156.7 93) (width 0.25) (layer "F.Cu") (net 54))
+  (segment (start 151.384 90.17) (end 150.622 89.408) (width 0.25) (layer "F.Cu") (net 54))
   (segment (start 200.34983 121.412) (end 192.861356 121.412) (width 0.25) (layer "F.Cu") (net 54))
   (segment (start 181.902652 120.569763) (end 180.806415 121.666) (width 0.25) (layer "F.Cu") (net 54))
   (segment (start 140.208 89.408) (end 141.986 89.408) (width 0.25) (layer "F.Cu") (net 54))
   (segment (start 157.596091 109.901763) (end 158.830093 108.667761) (width 0.25) (layer "F.Cu") (net 54))
+  (segment (start 151.384 90.678) (end 153.706 93) (width 0.25) (layer "F.Cu") (net 54))
   (segment (start 134.062 58.03) (end 134.062 83.262) (width 0.25) (layer "F.Cu") (net 54))
+  (segment (start 149.075593 90.099195) (end 149.075593 95.786763) (width 0.25) (layer "F.Cu") (net 54))
   (via (at 143.002 90.424) (size 0.8) (drill 0.4) (layers "F.Cu" "B.Cu") (net 54))
   (via (at 158.830093 108.667761) (size 0.8) (drill 0.4) (layers "F.Cu" "B.Cu") (net 54))
-  (via (at 153.599701 88.575701) (size 0.8) (drill 0.4) (layers "F.Cu" "B.Cu") (net 54))
+  (via (at 151.384 90.17) (size 0.8) (drill 0.4) (layers "F.Cu" "B.Cu") (net 54))
   (via (at 156.073593 125.649763) (size 0.8) (drill 0.4) (layers "F.Cu" "B.Cu") (net 54))
   (via (at 155.174549 112.349951) (size 0.8) (drill 0.4) (layers "F.Cu" "B.Cu") (net 54))
   (via (at 156.7 93) (size 0.8) (drill 0.4) (layers "F.Cu" "B.Cu") (net 54))
+  (segment (start 143.751 89.675) (end 143.002 90.424) (width 0.25) (layer "B.Cu") (net 54))
   (segment (start 156.625763 106.925763) (end 157.368371 106.925763) (width 0.25) (layer "B.Cu") (net 54))
-  (segment (start 143.751 89.675) (end 152.500402 89.675) (width 0.25) (layer "B.Cu") (net 54))
   (segment (start 156.1 106.4) (end 156.625763 106.925763) (width 0.25) (layer "B.Cu") (net 54))
   (segment (start 155.725593 125.301763) (end 156.073593 125.649763) (width 0.25) (layer "B.Cu") (net 54))
   (segment (start 155.725593 112.900995) (end 155.725593 125.301763) (width 0.25) (layer "B.Cu") (net 54))
-  (segment (start 143.002 90.424) (end 143.751 89.675) (width 0.25) (layer "B.Cu") (net 54))
   (segment (start 158.830093 108.387485) (end 158.830093 108.667761) (width 0.25) (layer "B.Cu") (net 54))
   (segment (start 156.1 96.159356) (end 156.1 106.4) (width 0.25) (layer "B.Cu") (net 54))
   (segment (start 155.174549 112.349951) (end 155.725593 112.900995) (width 0.25) (layer "B.Cu") (net 54))
+  (segment (start 150.889 89.675) (end 143.751 89.675) (width 0.25) (layer "B.Cu") (net 54))
   (segment (start 157.368371 106.925763) (end 158.830093 108.387485) (width 0.25) (layer "B.Cu") (net 54))
   (segment (start 156.7 95.559356) (end 156.1 96.159356) (width 0.25) (layer "B.Cu") (net 54))
-  (segment (start 152.500402 89.675) (end 153.599701 88.575701) (width 0.25) (layer "B.Cu") (net 54))
+  (segment (start 151.384 90.17) (end 150.889 89.675) (width 0.25) (layer "B.Cu") (net 54))
   (segment (start 156.7 93) (end 156.7 95.559356) (width 0.25) (layer "B.Cu") (net 54))
   (segment (start 220.843593 107.315) (end 225.923593 107.315) (width 0.25) (layer "F.Cu") (net 56))

Commit message: Fixing I2C Conns. Power Button still broken
Connections:
- J1 pad 3: /GPIO26 -> /SDA
- J1 pad 37: /GPIO26 -> /SCL
- SW10 pad 2: /GPIO26 -> /SCL
- U1 pad 27: /GPIO26 -> /SDA
Routing:
- net /GPIO26: track 149.5 -> 0.00 mm, vias 6 -> 0
- net /SDA: track 0.00 -> 89.5 mm, vias 0 -> 6
- net /SCL: track 84.1 -> 140.1 mm
- net GND: track 89.1 -> 86.0 mm
- net Net-(CN2-Pad2): track 95.3 -> 94.6 mm
- net Net-(Q5-B): track 88.8 -> 88.1 mm

Commit message: Flip U6, it broke the KSQ
Parts:
- R17: value 220R -> 3K3
- turned U6 to -90 degrees
Connections:
- C20 pad 1: Net-(U6-OUT) -> Net-(U6-IN)
- R33 pad 1: Net-(U6-OUT) -> Net-(U6-IN)
- R39 pad 1: Net-(U6-OUT) -> Net-(U6-IN)
- SW10 pad 1: unconnected-(SW10-Pad1) -> GND
- SW10 pad 4: GND -> unconnected-(SW10-Pad4)
- U6 pad 1: 24VDC -> Net-(U6-IN)
- U6 pad 3: Net-(U6-OUT) -> 24VDC
- U9 pad 8: Net-(U6-OUT) -> Net-(U6-IN)
Routing:
- net Net-(U6-IN): track 0.00 -> 61.1 mm, vias 0 -> 4
- net Net-(U6-OUT): track 55.1 -> 0.00 mm, vias 4 -> 0
- net /Drivers/Lamp-GND: track 40.8 -> 38.9 mm
- net 24VDC: track 123.3 -> 124.3 mm

Commit message: Fixing Shunt Connection to enable Current Control
Connections:
- CN6 pad 1: /Drivers/Lamp-GND -> Net-(U9A-+)
Routing:
- net Net-(U9A-+): track 16.4 -> 50.2 mm
Changed lines of the file:
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@@
     (pad_to_mask_clearance 0)
     (aux_axis_origin 224.028 107.188)
-    (grid_origin 176.276 55.626)
     (pcbplotparams
       (layerselection 0x00010fc_ffffffff)
@@
     (tags "resistor")
     (property "Inventory" "E")
-    (property "LCSC" "C104550")
+    (property "LCSC" "C137558")
     (property "Sheetfile" "drivers.kicad_sch")
     (property "Sheetname" "Drivers")
@@
     (property "ki_keywords" "Voltage Regulator 100mA Positive")
     (attr smd)
-    (fp_text reference "U6" (at 0.008407 3.406237 90) (layer "F.SilkS")
+    (fp_text reference "U6" (at 3.128237 1.387593 -180) (layer "F.SilkS")
         (effects (font (size 1 1) (thickness 0.15)))
     )
@@
       (stroke (width 0.06) (type solid)) (fill none) (layer "F.Fab"))
     (pad "1" thru_hole circle (at -2.54 -2.54 270) (size 2.1 2.1) (drill 1.399997) (layers "*.Cu" "*.Mask")
-      (net 12 "/Drivers/Lamp-GND") (pinfunction "1") (pintype "passive"))
+      (net 111 "Net-(U9A-+)") (pinfunction "1") (pintype "passive"))
     (pad "1" thru_hole rect (at -2.54 2.54 270) (size 2.1 2.1) (drill 1.399997) (layers "*.Cu" "*.Mask")
-      (net 12 "/Drivers/Lamp-GND") (pinfunction "1") (pintype "passive"))
+      (net 111 "Net-(U9A-+)") (pinfunction "1") (pintype "passive"))
     (pad "2" thru_hole circle (at 0 -2.54 270) (size 2.1 2.1) (drill 1.399997) (layers "*.Cu" "*.Mask")
       (net 35 "unconnected-(CN6-Pad2)") (pinfunction "2") (pintype "passive+no_connect"))
@@
   (segment (start 203.063593 80.564763) (end 203.063593 90.724763) (width 1.8) (layer "F.Cu") (net 1))
   (segment (start 169.281593 85.344) (end 169.281593 82.042) (width 1.8) (layer "F.Cu") (net 1))
-  (segment (start 171.591593 82.043763) (end 169.283356 82.043763) (width 1) (layer "F.Cu") (net 1))
   (segment (start 205.073 63.927) (end 207.3 61.7) (width 1.8) (layer "F.Cu") (net 1))
   (segment (start 179.568593 68.414763) (end 191.168593 80.014763) (width 1.8) (layer "F.Cu") (net 1))
   (segment (start 169.283356 82.043763) (end 169.281593 82.042) (width 1) (layer "F.Cu") (net 1))
+  (segment (start 171.591593 82.043763) (end 169.283356 82.043763) (width 1) (layer "F.Cu") (net 1))
   (segment (start 177.965237 68.414763) (end 179.568593 68.414763) (width 1.8) (layer "F.Cu") (net 1))
   (segment (start 202.428593 81.199763) (end 203.063593 80.564763) (width 1.8) (layer "F.Cu") (net 1))
@@
   (segment (start 205.54683 68.443) (end 205.073 68.443) (width 1.8) (layer "F.Cu") (net 1))
   (segment (start 209.366593 91.406763) (end 211.48263 93.5228) (width 1.8) (layer "F.Cu") (net 1))
-  (segment (start 169.431356 85.493763) (end 169.281593 85.344) (width 1) (layer "F.Cu") (net 1))
   (segment (start 169.281593 91.418407) (end 169.281593 85.344) (width 1.8) (layer "F.Cu") (net 1))
   (segment (start 164.987593 95.712407) (end 169.281593 91.418407) (width 1.8) (layer "F.Cu") (net 1))
@@
   (segment (start 184.371093 103.510263) (end 185.726593 102.154763) (width 0.25) (layer "F.Cu") (net 110))
   (segment (start 185.726593 100.884763) (end 180.776593 100.884763) (width 0.25) (layer "F.Cu") (net 111))
-  (segment (start 190.871593 102.789763) (end 190.871593 101.351263) (width 0.25) (layer "F.Cu") (net 111))
-  (segment (start 190.871593 101.351263) (end 190.363593 100.843263) (width 0.25) (layer "F.Cu") (net 111))
-  (segment (start 193.515093 102.893263) (end 193.411593 102.789763) (width 0.25) (layer "F.Cu") (net 111))
-  (segment (start 193.515093 104.821763) (end 193.515093 102.893263) (width 0.25) (layer "F.Cu") (net 111))
+  (segment (start 190.871593 101.351263) (end 190.363593 100.843263) (width 0.8) (layer "F.Cu") (net 111))
+  (segment (start 190.871593 102.789763) (end 190.871593 101.351263) (width 0.8) (layer "F.Cu") (net 111))
+  (segment (start 193.515093 104.821763) (end 193.515093 102.893263) (width 0.8) (layer "F.Cu") (net 111))
   (segment (start 190.363593 100.843263) (end 185.768093 100.843263) (width 0.25) (layer "F.Cu") (net 111))
   (segment (start 185.768093 100.843263) (end 185.726593 100.884763) (width 0.25) (layer "F.Cu") (net 111))
   (via (at 190.871593 102.789763) (size 0.8) (drill 0.4) (layers "F.Cu" "B.Cu") (net 111))
-  (via (at 193.411593 102.789763) (size 0.8) (drill 0.4) (layers "F.Cu" "B.Cu") (net 111))
-  (segment (start 193.411593 102.789763) (end 190.871593 102.789763) (width 0.25) (layer "B.Cu") (net 111))
+  (via (at 193.515093 102.893263) (size 0.8) (drill 0.4) (layers "F.Cu" "B.Cu") (net 111))
+  (segment (start 193.618593 102.789763) (end 217.49483 102.789763) (width 0.8) (layer "B.Cu") (net 111))
+  (segment (start 193.411593 102.789763) (end 190.871593 102.789763) (width 0.8) (layer "B.Cu") (net 111))
+  (segment (start 217.49483 102.789763) (end 220.843593 99.441) (width 0.8) (layer "B.Cu") (net 111))
+  (segment (start 193.515093 102.893263) (end 193.618593 102.789763) (width 0.8) (layer "B.Cu") (net 111))
+  (segment (start 193.515093 102.893263) (end 193.411593 102.789763) (width 0.8) (layer "B.Cu") (net 111))
+  (segment (start 220.843593 99.441) (end 225.923593 99.441) (width 0.8) (layer "B.Cu") (net 111))
   (segment (start 149.102956 104.314126) (end 149.075593 104.286763) (width 0.25) (layer "F.Cu") (net 114))
   (segment (start 149.102956 106.188067) (end 149.102956 104.314126) (width 0.25) (layer "F.Cu") (net 114))

Commit message: Add the missing BJP Transistor for the shaft eye
Parts:
- added Q8: SS8050, Package_TO_SOT_SMD:SOT-23, F.Cu at (135.3, 118.9)
Routing:
- net Net-(Q8-B): track 94.6 -> 103.5 mm, vias 1 -> 3
- net Net-(Q8-C): track 9.39 -> 13.8 mm

Commit message: Flipping J5/6 to have GND on Pin 1; Invert the Shaft Eye's ISR
Connections:
- J5 pad 1: /Sensors/3.3V-Eye2 -> GND2
- J5 pad 3: GND2 -> /Sensors/3.3V-Eye2
- J6 pad 1: /Sensors/3.3V-Eye1 -> GND1
- J6 pad 3: GND1 -> /Sensors/3.3V-Eye1
Changed lines of the file:
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@@
       (stroke (width 0.1) (type solid)) (layer "F.Fab"))
     (pad "1" thru_hole rect (at 0 0 270) (size 1.7 1.7) (drill 1) (layers "*.Cu" "*.Mask")
-      (net 122 "/Sensors/3.3V-Eye1") (pinfunction "Pin_1") (pintype "passive"))
+      (net 120 "GND1") (pinfunction "Pin_1") (pintype "passive"))
     (pad "2" thru_hole oval (at 0 2.54 270) (size 1.7 1.7) (drill 1) (layers "*.Cu" "*.Mask")
       (net 77 "Net-(J6-Pin_2)") (pinfunction "Pin_2") (pintype "passive"))
     (pad "3" thru_hole oval (at 0 5.08 270) (size 1.7 1.7) (drill 1) (layers "*.Cu" "*.Mask")
-      (net 120 "GND1") (pinfunction "Pin_3") (pintype "passive"))
+      (net 122 "/Sensors/3.3V-Eye1") (pinfunction "Pin_3") (pintype "passive"))
     (model "${KICAD6_3DMODEL_DIR}/Connector_PinHeader_2.54mm.3dshapes/PinHeader_1x03_P2.54mm_Vertical.wrl" hide
       (offset (xyz 0 0 0))
@@
       (stroke (width 0.1) (type solid)) (layer "F.Fab"))
     (pad "1" thru_hole rect (at 0 0 270) (size 1.7 1.7) (drill 1) (layers "*.Cu" "*.Mask")
-      (net 123 "/Sensors/3.3V-Eye2") (pinfunction "Pin_1") (pintype "passive"))
+      (net 121 "GND2") (pinfunction "Pin_1") (pintype "passive"))
     (pad "2" thru_hole oval (at 0 2.54 270) (size 1.7 1.7) (drill 1) (layers "*.Cu" "*.Mask")
       (net 76 "Net-(J5-Pin_2)") (pinfunction "Pin_2") (pintype "passive"))
     (pad "3" thru_hole oval (at 0 5.08 270) (size 1.7 1.7) (drill 1) (layers "*.Cu" "*.Mask")
-      (net 121 "GND2") (pinfunction "Pin_3") (pintype "passive"))
+      (net 123 "/Sensors/3.3V-Eye2") (pinfunction "Pin_3") (pintype "passive"))
     (model "${KICAD6_3DMODEL_DIR}/Connector_PinHeader_2.54mm.3dshapes/PinHeader_1x03_P2.54mm_Vertical.wrl" hide
       (offset (xyz 0 0 0))
