File: scan-controller-kicad/sensors.kicad_sch (KiCad schematic)
At the start: 23 parts, among them CN2 Shaft Eye, CN3 Film End Eye, J1 Shaft Eye, J2 Film End Eye, Q2 BC848, U1 74LVC14, U2 QRE1113, U3 QRE1113

Commit message: Adding missing components Mfnrs and footprints
Parts:
- CN2, CN3: LCSC (none) -> C475125; LCSC Part C475125 -> (none)
- R1, R5: LCSC (none) -> C17408
- U1: LCSC C6065 -> C6065
- U2, U3: LCSC (none) -> C232862

Commit message: BOM progress
Parts:
- R1, R10, R12, R13, R4, R5, R6, R7, R8, R9: Inventory (none) -> B
Changed lines of the file:
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@@
+      (effects (font (size 1.27 1.27)) hide)
+    )
+    (property "Inventory" "" (at 50.8 97.79 0)
       (effects (font (size 1.27 1.27)) hide)
     )
@@
       (effects (font (size 1.27 1.27)) hide)
     )
+    (property "Inventory" "B" (at 157.48 69.85 0)
+      (effects (font (size 1.27 1.27)) hide)
+    )
     (pin "1")
     (pin "2")
@@
       (effects (font (size 1.27 1.27)) hide)
     )
+    (property "Inventory" "" (at 183.515 125.73 0)
+      (effects (font (size 1.27 1.27)) hide)
+    )
     (pin "1")
     (pin "2")
@@
       (effects (font (size 1.27 1.27)) hide)
     )
+    (property "Inventory" "" (at 118.11 120.015 0)
+      (effects (font (size 1.27 1.27)) hide)
+    )
     (pin "1")
     (pin "2")
@@
       (effects (font (size 1.27 1.27)) hide)
     )
+    (property "Inventory" "" (at 182.88 78.74 0)
+      (effects (font (size 1.27 1.27)) hide)
+    )
     (pin "1")
     (pin "2")
@@
     )
     (property "LCSC" "C6065" (at 167.64 73.66 0)
+      (effects (font (size 1.27 1.27)) hide)
+    )
+    (property "Inventory" "" (at 167.64 73.66 0)
       (effects (font (size 1.27 1.27)) hide)
     )
@@
       (effects (font (size 1.27 1.27)) hide)
     )
+    (property "Inventory" "B" (at 158.115 115.57 0)
+      (effects (font (size 1.27 1.27)) hide)
+    )
     (pin "1")
     (pin "2")
@@
       (effects (font (size 1.27 1.27)) hide)
     )
+    (property "Inventory" "B" (at 107.315 69.215 0)
+      (effects (font (size 1.27 1.27)) hide)
+    )
     (pin "1")
     (pin "2")
@@
     )
     (property "LCSC" "C6065" (at 168.275 119.38 0)
+      (effects (font (size 1.27 1.27)) hide)
+    )
+    (property "Inventory" "" (at 168.275 119.38 0)
       (effects (font (size 1.27 1.27)) hide)
     )
@@
       (effects (font (size 1.27 1.27)) hide)
     )
+    (property "Inventory" "" (at 100.33 122.555 0)
+      (effects (font (size 1.27 1.27)) hide)
+    )
     (pin "1")
     (pin "2")
@@
       (effects (font (size 1.27 1.27)) hide)
     )
+    (property "Inventory" "" (at 200.025 121.92 0)
+      (effects (font (size 1.27 1.27)) hide)
+    )
     (pin "1")
     (instances
@@
     )
     (property "LCSC" "C232862" (at 99.695 76.835 0)
+      (effects (font (size 1.27 1.27)) hide)
+    )
+    (property "Inventory" "" (at 99.695 76.835 0)
       (effects (font (size 1.27 1.27)) hide)
     )
@@
       (effects (font (size 1.27 1.27)) hide)
     )
+    (property "Inventory" "B" (at 152.4 73.66 0)
+      (effects (font (size 1.27 1.27)) hide)
+    )
     (pin "1")
     (pin "2")
@@
       (effects (font (size 1.27 1.27)) hide)
     )
+    (property "Inventory" "" (at 140.97 73.66 0)
+      (effects (font (size 1.27 1.27)) hide)
+    )
     (pin "1")
     (pin "2")
@@
       (effects (font (size 1.27 1.27)) hide)
     )
+    (property "Inventory" "B" (at 179.705 119.38 0)
+      (effects (font (size 1.27 1.27)) hide)
+    )
     (pin "1")
     (pin "2")
@@
     )
     (property "LCSC" "C17408" (at 92.71 114.935 0)
+      (effects (font (size 1.27 1.27)) hide)
+    )
+    (property "Inventory" "B" (at 92.71 114.935 0)
       (effects (font (size 1.27 1.27)) hide)
     )
@@
       (effects (font (size 1.27 1.27)) hide)
     )
+    (property "Inventory" "" (at 155.575 125.73 0)
+      (effects (font (size 1.27 1.27)) hide)
+    )
     (pin "1")
     (pin "2")
@@
       (effects (font (size 1.27 1.27)) hide)
     )
+    (property "Inventory" "" (at 141.605 119.38 0)
+      (effects (font (size 1.27 1.27)) hide)
+    )
     (pin "1")
     (pin "2")
@@
       (effects (font (size 1.27 1.27)) hide)
     )
+    (property "Inventory" "B" (at 153.035 119.38 0)
+      (effects (font (size 1.27 1.27)) hide)
+    )
     (pin "1")
     (pin "2")
@@
       (effects (font (size 1.27 1.27)) hide)
     )
+    (property "Inventory" "" (at 59.69 83.82 0)
+      (effects (font (size 1.27 1.27)) hide)
+    )
     (pin "1")
     (pin "2")
@@
     )
     (property "LCSC" "C6065" (at 191.77 73.66 0)
+      (effects (font (size 1.27 1.27)) hide)
+    )
+    (property "Inventory" "" (at 191.77 73.66 0)
       (effects (font (size 1.27 1.27)) hide)
     )
@@
       (effects (font (size 1.27 1.27)) hide)
     )
+    (property "Inventory" "B" (at 179.07 73.66 0)
+      (effects (font (size 1.27 1.27)) hide)
+    )
     (pin "1")
     (pin "2")
@@
       (effects (font (size 1.27 1.27)) hide)
     )
+    (property "Inventory" "B" (at 107.95 114.935 0)
+      (effects (font (size 1.27 1.27)) hide)
+    )
     (pin "1")
     (pin "2")
@@
       (effects (font (size 1.27 1.27)) hide)
     )
+    (property "Inventory" "B" (at 92.075 69.215 0)
+      (effects (font (size 1.27 1.27)) hide)
+    )
     (pin "1")
     (pin "2")
@@
       (effects (font (size 1.27 1.27)) hide)
     )
+    (property "Inventory" "" (at 199.39 76.2 0)
+      (effects (font (size 1.27 1.27)) hide)
+    )
     (pin "1")
     (instances
@@
       (effects (font (size 1.27 1.27)) hide)
     )
+    (property "Inventory" "" (at 117.475 74.295 0)
+      (effects (font (size 1.27 1.27)) hide)
+    )
     (pin "1")
     (pin "2")
@@
       (effects (font (size 1.27 1.27)) hide)
     )
+    (property "Inventory" "" (at 192.405 119.38 0)
+      (effects (font (size 1.27 1.27)) hide)
+    )

Commit message: BOM complete!
Parts:
- C1: footprint LED_SMD:LED_0805_2012Metric -> Capacitor_SMD:C_0805_2012Metric; Inventory (none) -> B
- C4, C5: Inventory (none) -> B
- Q2: value BC848 -> SS8050; Inventory (none) -> B; LCSC C181142 -> C2150
- U1, U2, U3: Inventory (none) -> E
Changed lines of the file:
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@@
       (effects (font (size 1.27 1.27)) hide)
     )
-    (property "Inventory" "" (at 50.8 97.79 0)
+    (property "Inventory" "E" (at 50.8 97.79 0)
       (effects (font (size 1.27 1.27)) hide)
     )
@@
       (effects (font (size 1.27 1.27)) hide)
     )
-    (property "Inventory" "" (at 183.515 125.73 0)
+    (property "Inventory" "B" (at 183.515 125.73 0)
       (effects (font (size 1.27 1.27)) hide)
     )
@@
       (effects (font (size 1.27 1.27)) hide)
     )
-    (property "Inventory" "" (at 182.88 78.74 0)
+    (property "Inventory" "B" (at 182.88 78.74 0)
       (effects (font (size 1.27 1.27)) hide)
     )
@@
       (effects (font (size 1.27 1.27)) hide)
     )
-    (property "Inventory" "" (at 167.64 73.66 0)
+    (property "Inventory" "E" (at 167.64 73.66 0)
       (effects (font (size 1.27 1.27)) hide)
     )
@@
       (effects (font (size 1.27 1.27)) hide)
     )
-    (property "Inventory" "" (at 168.275 119.38 0)
+    (property "Inventory" "E" (at 168.275 119.38 0)
       (effects (font (size 1.27 1.27)) hide)
     )
@@
       (effects (font (size 1.27 1.27)) hide)
     )
-    (property "Inventory" "" (at 100.33 122.555 0)
+    (property "Inventory" "E" (at 100.33 122.555 0)
       (effects (font (size 1.27 1.27)) hide)
     )
@@
       (effects (font (size 1.27 1.27)) hide)
     )
-    (property "Inventory" "" (at 99.695 76.835 0)
+    (property "Inventory" "E" (at 99.695 76.835 0)
       (effects (font (size 1.27 1.27)) hide)
     )
@@
       (effects (font (size 1.27 1.27)) (justify left))
     )
-    (property "Value" "BC848" (at 160.4264 126.873 0)
+    (property "Value" "SS8050" (at 160.4264 126.873 0)
       (effects (font (size 1.27 1.27)) (justify left))
     )
@@
       (effects (font (size 1.27 1.27) italic) (justify left) hide)
     )
-    (property "Datasheet" "https://www.mouser.de/datasheet/2/308/BC846ALT1-D-1293035.pdf" (at 155.575 125.73 0)
+    (property "Datasheet" "https://datasheet.lcsc.com/lcsc/2303221100_Jiangsu-Changjing-Electronics-Technology-Co---Ltd--SS8050_C2150.pdf" (at 155.575 125.73 0)
       (effects (font (size 1.27 1.27)) (justify left) hide)
     )
-    (property "LCSC" "C181142" (at 155.575 125.73 0)
-      (effects (font (size 1.27 1.27)) hide)
-    )
-    (property "Inventory" "" (at 155.575 125.73 0)
+    (property "LCSC" "C2150" (at 155.575 125.73 0)
+      (effects (font (size 1.27 1.27)) hide)
+    )
+    (property "Inventory" "B" (at 155.575 125.73 0)
       (effects (font (size 1.27 1.27)) hide)
     )
@@
       (effects (font (size 1.27 1.27)) (justify left))
     )
-    (property "Footprint" "LED_SMD:LED_0805_2012Metric" (at 59.69 83.82 0)
+    (property "Footprint" "Capacitor_SMD:C_0805_2012Metric" (at 59.69 83.82 0)
       (effects (font (size 1.27 1.27)) hide)
     )
@@
       (effects (font (size 1.27 1.27)) hide)
     )
-    (property "Inventory" "" (at 59.69 83.82 0)
+    (property "Inventory" "B" (at 59.69 83.82 0)
       (effects (font (size 1.27 1.27)) hide)
     )
@@
       (effects (font (size 1.27 1.27)) hide)
     )
-    (property "Inventory" "" (at 191.77 73.66 0)
+    (property "Inventory" "E" (at 191.77 73.66 0)
       (effects (font (size 1.27 1.27)) hide)
     )
@@
       (effects (font (size 1.27 1.27)) hide)
     )
-    (property "Inventory" "" (at 192.405 119.38 0)
-      (effects (font (size 1.27 1.27)) hide)
-    )
+    (property "Inventory" "E" (at 192.405 119.38 0)
+      (effects (font (size 1.27 1.27)) hide)
+    )

Commit message: 31 nets to go
Parts:
- TP7, TP8: footprint TestPoint:TestPoint_THTPad_D2.0mm_Drill1.0mm -> TestPoint:TestPoint_Pad_1.5x1.5mm
Changed lines of the file:
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@@
         )
         (path "/ab6dbce1-4ecf-44ae-8f33-5f07e4f43ca9/32afee9c-f78c-4810-b9e6-48288995c3da"
-          (reference "C15") (unit 1)
+          (reference "C14") (unit 1)
         )
       )
@@
         )
         (path "/ab6dbce1-4ecf-44ae-8f33-5f07e4f43ca9/32afee9c-f78c-4810-b9e6-48288995c3da"
-          (reference "C14") (unit 1)
+          (reference "C13") (unit 1)
         )
       )
@@
       (effects (font (size 1.27 1.27)) (justify left))
     )
-    (property "Footprint" "TestPoint:TestPoint_THTPad_D2.0mm_Drill1.0mm" (at 194.945 121.92 0)
+    (property "Footprint" "TestPoint:TestPoint_Pad_1.5x1.5mm" (at 194.945 121.92 0)
       (effects (font (size 1.27 1.27)) hide)
     )
@@
         )
         (path "/ab6dbce1-4ecf-44ae-8f33-5f07e4f43ca9/32afee9c-f78c-4810-b9e6-48288995c3da"
-          (reference "C13") (unit 1)
+          (reference "C12") (unit 1)
         )
       )
@@
       (effects (font (size 1.27 1.27)) (justify left))
     )
-    (property "Footprint" "TestPoint:TestPoint_THTPad_D2.0mm_Drill1.0mm" (at 194.31 76.2 0)
-      (effects (font (size 1.27 1.27)) hide)
-    )
+    (property "Footprint" "TestPoint:TestPoint_Pad_1.5x1.5mm" (at 194.31 76.2 0)
+      (effects (font (size 1.27 1.27)) hide)
+    )

Commit message: smaller eyes
Parts:
- R1, R5: footprint Resistor_SMD:R_0805_2012Metric -> Resistor_SMD:R_0402_1005Metric; LCSC C17408 -> C25076
- R10, R4: footprint Resistor_SMD:R_0805_2012Metric -> Resistor_SMD:R_0402_1005Metric; LCSC C17713 -> C25792
Changed lines of the file:
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@@
       (effects (font (size 1.27 1.27)) (justify left))
     )
-    (property "Footprint" "Resistor_SMD:R_0805_2012Metric" (at 107.315 69.215 0)
+    (property "Footprint" "Resistor_SMD:R_0402_1005Metric" (at 107.315 69.215 0)
       (effects (font (size 1.27 1.27)) hide)
     )
@@
       (effects (font (size 1.27 1.27)) hide)
     )
-    (property "LCSC" "C17713" (at 107.315 69.215 0)
+    (property "LCSC" "C25792" (at 107.315 69.215 0)
       (effects (font (size 1.27 1.27)) hide)
     )
@@
       (effects (font (size 1.27 1.27)) (justify left))
     )
-    (property "Footprint" "Resistor_SMD:R_0805_2012Metric" (at 92.71 114.935 0)
+    (property "Footprint" "Resistor_SMD:R_0402_1005Metric" (at 92.71 114.935 0)
       (effects (font (size 1.27 1.27)) hide)
     )
@@
       (effects (font (size 1.27 1.27)) hide)
     )
-    (property "LCSC" "C17408" (at 92.71 114.935 0)
+    (property "LCSC" "C25076" (at 92.71 114.935 0)
       (effects (font (size 1.27 1.27)) hide)
     )
@@
       (effects (font (size 1.27 1.27)) (justify left))
     )
-    (property "Footprint" "Resistor_SMD:R_0805_2012Metric" (at 107.95 114.935 0)
+    (property "Footprint" "Resistor_SMD:R_0402_1005Metric" (at 107.95 114.935 0)
       (effects (font (size 1.27 1.27)) hide)
     )
@@
       (effects (font (size 1.27 1.27)) hide)
     )
-    (property "LCSC" "C17713" (at 107.95 114.935 0)
+    (property "LCSC" "C25792" (at 107.95 114.935 0)
       (effects (font (size 1.27 1.27)) hide)
     )
@@
       (effects (font (size 1.27 1.27)) (justify left))
     )
-    (property "Footprint" "Resistor_SMD:R_0805_2012Metric" (at 92.075 69.215 0)
+    (property "Footprint" "Resistor_SMD:R_0402_1005Metric" (at 92.075 69.215 0)
       (effects (font (size 1.27 1.27)) hide)
     )
@@
       (effects (font (size 1.27 1.27)) hide)
     )
-    (property "LCSC" "C17408" (at 92.075 69.215 0)
-      (effects (font (size 1.27 1.27)) hide)
-    )
+    (property "LCSC" "C25076" (at 92.075 69.215 0)
+      (effects (font (size 1.27 1.27)) hide)
+    )

Commit message: Round corners!
Connections:
- net 3.3V-uC: no longer J1.1 (Pin_1), J2.1 (Pin_1), R1.1, R10.1, R4.1, R5.1
- net GNDD: no longer J1.3 (Pin_3), J2.3 (Pin_3), U2.2 (K), U2.4, U3.2 (K), U3.4
- new net 3.3V-Eye1: J2.1 (Pin_1), R10.1, R5.1
- new net 3.3V-Eye2: J1.1 (Pin_1), R1.1, R4.1
- new net GND1: J2.3 (Pin_3), U3.2 (K), U3.4
- new net GND2: J1.3 (Pin_3), U2.2 (K), U2.4
Other:
- moved on the sheet: J1, J2, R1, R10, R4, R5, U2, U3
