File: scan-controller-kicad/sensors.kicad_sch (KiCad schematic)
At the start: 23 parts, among them CN2 Shaft Eye, CN3 Film End Eye, J1 Shaft Eye, J2 Film End Eye, Q2 SS8050, U1 74LVC14, U2 QRE1113, U3 QRE1113

Commit message: Labels, Keep-out, L moved away from camera cable
Connections:
- net 3.3V-uC: now also CN2.3, CN3.3; no longer CN2.1, CN3.1
- net GNDD: now also CN2.1, CN3.1; no longer CN2.3, CN3.3
Other:
- moved on the sheet: CN2, CN3
Changed lines of the file:
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@@
     )
   )
-  (symbol (lib_id "easyeda2kicad:KF141R-2.54-3P") (at 140.97 73.66 0) (mirror y) (unit 1)
-    (in_bom yes) (on_board yes) (dnp no)
-    (property "Reference" "CN2" (at 142.875 67.31 0)
-      (effects (font (size 1.27 1.27)) (justify left))
-    )
-    (property "Value" "Shaft Eye" (at 142.875 64.77 0)
-      (effects (font (size 1.27 1.27)) (justify left))
-    )
-    (property "Footprint" "easyeda2kicad:CONN-TH_3P-P2.54_KF141R-2.54-3P" (at 140.97 83.82 0)
-      (effects (font (size 1.27 1.27)) hide)
-    )
-    (property "Datasheet" "https://lcsc.com/product-detail/New-Quadratic-Unclassified-Data_Cixi-Kefa-Elec-KF141R-2-54-3P_C475125.html" (at 140.97 86.36 0)
-      (effects (font (size 1.27 1.27)) hide)
-    )
-    (property "LCSC Part" "" (at 140.97 88.9 0)
+  (symbol (lib_id "easyeda2kicad:KF141R-2.54-3P") (at 140.97 73.66 180) (unit 1)
+    (in_bom yes) (on_board yes) (dnp no)
+    (property "Reference" "CN2" (at 142.875 80.01 0)
+      (effects (font (size 1.27 1.27)) (justify left))
+    )
+    (property "Value" "Shaft Eye" (at 142.875 82.55 0)
+      (effects (font (size 1.27 1.27)) (justify left))
+    )
+    (property "Footprint" "easyeda2kicad:CONN-TH_3P-P2.54_KF141R-2.54-3P" (at 140.97 63.5 0)
+      (effects (font (size 1.27 1.27)) hide)
+    )
+    (property "Datasheet" "https://lcsc.com/product-detail/New-Quadratic-Unclassified-Data_Cixi-Kefa-Elec-KF141R-2-54-3P_C475125.html" (at 140.97 60.96 0)
+      (effects (font (size 1.27 1.27)) hide)
+    )
+    (property "LCSC Part" "" (at 140.97 58.42 0)
       (effects (font (size 1.27 1.27)) hide)
     )
@@
     )
   )
-  (symbol (lib_id "easyeda2kicad:KF141R-2.54-3P") (at 141.605 119.38 0) (mirror y) (unit 1)
-    (in_bom yes) (on_board yes) (dnp no)
-    (property "Reference" "CN3" (at 142.875 113.03 0)
-      (effects (font (size 1.27 1.27)) (justify left))
-    )
-    (property "Value" "Film End Eye" (at 144.145 110.49 0)
-      (effects (font (size 1.27 1.27)) (justify left))
-    )
-    (property "Footprint" "easyeda2kicad:CONN-TH_3P-P2.54_KF141R-2.54-3P" (at 141.605 129.54 0)
-      (effects (font (size 1.27 1.27)) hide)
-    )
-    (property "Datasheet" "https://lcsc.com/product-detail/New-Quadratic-Unclassified-Data_Cixi-Kefa-Elec-KF141R-2-54-3P_C475125.html" (at 141.605 132.08 0)
-      (effects (font (size 1.27 1.27)) hide)
-    )
-    (property "LCSC Part" "" (at 141.605 134.62 0)
-      (effects (font (size 1.27 1.27)) hide)
-    )
+  (symbol (lib_id "easyeda2kicad:KF141R-2.54-3P") (at 141.605 119.38 180) (unit 1)
+    (in_bom yes) (on_board yes) (dnp no)
+    (property "Reference" "CN3" (at 142.875 125.73 0)
+      (effects (font (size 1.27 1.27)) (justify left))
+    )
+    (property "Value" "Film End Eye" (at 144.145 128.27 0)
+      (effects (font (size 1.27 1.27)) (justify left))
+    )
+    (property "Footprint" "easyeda2kicad:CONN-TH_3P-P2.54_KF141R-2.54-3P" (at 141.605 109.22 0)
+      (effects (font (size 1.27 1.27)) hide)
+    )
+    (property "Datasheet" "https://lcsc.com/product-detail/New-Quadratic-Unclassified-Data_Cixi-Kefa-Elec-KF141R-2-54-3P_C475125.html" (at 141.605 106.68 0)
+      (effects (font (size 1.27 1.27)) hide)
+    )
+    (property "LCSC Part" "" (at 141.605 104.14 0)
+      (effects (font (size 1.27 1.27)) hide)
+    )

Commit message: Fixing BOM
Parts:
- J1, J2, TP7, TP8: now left out of the parts list
Changed lines of the file:
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@@
   )
   (symbol (lib_id "Connector_Generic:Conn_01x03") (at 116.205 73.66 0) (unit 1)
-    (in_bom yes) (on_board yes) (dnp no)
+    (in_bom no) (on_board yes) (dnp no)
     (property "Reference" "J2" (at 114.935 68.58 0)
       (effects (font (size 1.27 1.27)) (justify left))
@@
   )
   (symbol (lib_id "Connector:TestPoint") (at 200.025 121.92 180) (unit 1)
-    (in_bom yes) (on_board yes) (dnp no)
+    (in_bom no) (on_board yes) (dnp no)
     (property "Reference" "TP8" (at 204.597 125.476 0)
       (effects (font (size 1.27 1.27)) (justify left))
@@
   )
   (symbol (lib_id "Connector:TestPoint") (at 199.39 76.2 180) (unit 1)
-    (in_bom yes) (on_board yes) (dnp no)
+    (in_bom no) (on_board yes) (dnp no)
     (property "Reference" "TP7" (at 203.962 79.756 0)
       (effects (font (size 1.27 1.27)) (justify left))
@@
   )
   (symbol (lib_id "Connector_Generic:Conn_01x03") (at 117.475 119.38 0) (unit 1)
-    (in_bom yes) (on_board yes) (dnp no)
+    (in_bom no) (on_board yes) (dnp no)
     (property "Reference" "J1" (at 116.205 114.3 0)
       (effects (font (size 1.27 1.27)) (justify left))

Commit message: Add the missing BJP Transistor for the shaft eye
Parts:
- added Q2: SS8050, Package_TO_SOT_SMD:SOT-23, symbol Transistor_BJT:BC847
Connections:
- net GNDD: now also Q2.2 (E)
- net at R6.2, R8.1, U1.1: now also Q2.3 (C)
- net at CN2.2, R6.1: now also Q2.1 (B)
Changed lines of the file:
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@@
   (junction (at 98.425 81.28) (diameter 0) (color 0 0 0 0)
   )
+  (junction (at 157.48 85.09) (diameter 0) (color 0 0 0 0)
+  )
   (junction (at 183.515 119.38) (diameter 0) (color 0 0 0 0)
   )
@@
   (junction (at 106.045 73.66) (diameter 0) (color 0 0 0 0)
   )
+  (junction (at 148.59 73.66) (diameter 0) (color 0 0 0 0)
+  )
   (junction (at 107.315 124.46) (diameter 0) (color 0 0 0 0)
   )
@@
     (stroke (width 0) (type default))
   )
+  (wire (pts (xy 157.48 85.09) (xy 157.48 86.36))
+    (stroke (width 0) (type default))
+  )
+  (wire (pts (xy 148.59 73.66) (xy 149.86 73.66))
+    (stroke (width 0) (type default))
+  )
   (wire (pts (xy 146.685 111.76) (xy 146.685 116.84))
     (stroke (width 0) (type default))
@@
     (stroke (width 0) (type default))
   )
-  (wire (pts (xy 147.32 76.2) (xy 147.32 77.47))
-    (stroke (width 0) (type default))
-  )
   (wire (pts (xy 50.8 76.835) (xy 50.8 81.28))
     (stroke (width 0) (type default))
   )
+  (wire (pts (xy 146.05 85.09) (xy 157.48 85.09))
+    (stroke (width 0) (type default))
+  )
   (wire (pts (xy 107.315 109.22) (xy 107.315 111.76))
     (stroke (width 0) (type default))
@@
     (stroke (width 0) (type default))
   )
+  (wire (pts (xy 146.05 76.2) (xy 146.05 85.09))
+    (stroke (width 0) (type default))
+  )
+  (wire (pts (xy 148.59 80.01) (xy 149.86 80.01))
+    (stroke (width 0) (type default))
+  )
   (wire (pts (xy 98.425 81.28) (xy 106.045 81.28))
     (stroke (width 0) (type default))
@@
     (stroke (width 0) (type default))
   )
-  (wire (pts (xy 146.05 73.66) (xy 149.86 73.66))
+  (wire (pts (xy 146.05 73.66) (xy 148.59 73.66))
     (stroke (width 0) (type default))
   )
@@
     (stroke (width 0) (type default))
   )
+  (wire (pts (xy 148.59 73.66) (xy 148.59 80.01))
+    (stroke (width 0) (type default))
+  )
+  (wire (pts (xy 157.48 73.66) (xy 157.48 74.93))
+    (stroke (width 0) (type default))
+  )
   (wire (pts (xy 106.045 60.325) (xy 106.045 63.5))
     (stroke (width 0) (type default))
@@
     (stroke (width 0) (type default))
   )
-  (wire (pts (xy 146.05 76.2) (xy 147.32 76.2))
-    (stroke (width 0) (type default))
-  )
   (wire (pts (xy 111.125 63.5) (xy 106.045 63.5))
     (stroke (width 0) (type default))
@@
     (stroke (width 0) (type default))
   )
+  (wire (pts (xy 182.88 85.09) (xy 157.48 85.09))
+    (stroke (width 0) (type default))
+  )
   (wire (pts (xy 155.575 119.38) (xy 158.115 119.38))
     (stroke (width 0) (type default))
@@
     (stroke (width 0) (type default))
   )
-  (wire (pts (xy 182.88 81.28) (xy 182.88 82.55))
+  (wire (pts (xy 182.88 81.28) (xy 182.88 85.09))
     (stroke (width 0) (type default))
   )
@@
     )
   )
+  (symbol (lib_id "Transistor_BJT:BC847") (at 154.94 80.01 0) (unit 1)
+    (in_bom yes) (on_board yes) (dnp no)
+    (property "Reference" "Q2" (at 159.7914 78.8416 0)
+      (effects (font (size 1.27 1.27)) (justify left))
+    )
+    (property "Value" "SS8050" (at 159.7914 81.153 0)
+      (effects (font (size 1.27 1.27)) (justify left))
+    )
+    (property "Footprint" "Package_TO_SOT_SMD:SOT-23" (at 160.02 81.915 0)
+      (effects (font (size 1.27 1.27) italic) (justify left) hide)
+    )
+    (property "Datasheet" "https://datasheet.lcsc.com/lcsc/2303221100_Jiangsu-Changjing-Electronics-Technology-Co---Ltd--SS8050_C2150.pdf" (at 154.94 80.01 0)
+      (effects (font (size 1.27 1.27)) (justify left) hide)
+    )
+    (property "LCSC" "C2150" (at 154.94 80.01 0)
+      (effects (font (size 1.27 1.27)) hide)
+    )
+    (property "Inventory" "B" (at 154.94 80.01 0)
+      (effects (font (size 1.27 1.27)) hide)
+    )
+    (pin "1")
+    (pin "2")
+    (pin "3")
+    (instances
+      (project "scan-controller-kicad"
+        (path "/ab6dbce1-4ecf-44ae-8f33-5f07e4f43ca9"
+          (reference "Q2") (unit 1)
+        )
+        (path "/ab6dbce1-4ecf-44ae-8f33-5f07e4f43ca9/32afee9c-f78c-4810-b9e6-48288995c3da"
+          (reference "Q8") (unit 1)
+        )
+      )
+    )
+  )
   (symbol (lib_id "74xx:74HC14") (at 168.275 119.38 0) (unit 3)
     (in_bom yes) (on_board yes) (dnp no)
@@
     )
   )
-  (symbol (lib_id "power:GNDD") (at 147.32 77.47 0) (unit 1)
-    (in_bom yes) (on_board yes) (dnp no)
-    (property "Reference" "#PWR012" (at 147.32 83.82 0)
-      (effects (font (size 1.27 1.27)) hide)
-    )
-    (property "Value" "GNDD" (at 147.32 81.28 0)
-      (effects (font (size 1.27 1.27)))
-    )
-    (property "Footprint" "" (at 147.32 77.47 0)
-      (effects (font (size 1.27 1.27)) hide)
-    )
-    (property "Datasheet" "" (at 147.32 77.47 0)
+  (symbol (lib_id "power:GNDD") (at 157.48 86.36 0) (unit 1)
+    (in_bom yes) (on_board yes) (dnp no)
+    (property "Reference" "#PWR012" (at 157.48 92.71 0)
+      (effects (font (size 1.27 1.27)) hide)
+    )
+    (property "Value" "GNDD" (at 157.48 90.17 0)
+      (effects (font (size 1.27 1.27)))
+    )
+    (property "Footprint" "" (at 157.48 86.36 0)
+      (effects (font (size 1.27 1.27)) hide)
+    )
+    (property "Datasheet" "" (at 157.48 86.36 0)
       (effects (font (size 1.27 1.27)) hide)
     )
@@
         )
       )
-    )
-  )
-  (symbol (lib_id "power:GNDD") (at 182.88 82.55 0) (unit 1)
-    (in_bom yes) (on_board yes) (dnp no)
-    (property "Reference" "#PWR018" (at 182.88 88.9 0)
-      (effects (font (size 1.27 1.27)) hide)
-    )
-    (property "Value" "GNDD" (at 182.88 86.36 0)
-      (effects (font (size 1.27 1.27)))
-    )
-    (property "Footprint" "" (at 182.88 82.55 0)
-      (effects (font (size 1.27 1.27)) hide)
-    )
-    (property "Datasheet" "" (at 182.88 82.55 0)
-      (effects (font (size 1.27 1.27)) hide)
-    )
-    (pin "1")
-    (instances
-      (project "scan-controller-kicad"
-        (path "/ab6dbce1-4ecf-44ae-8f33-5f07e4f43ca9"
-          (reference "#PWR018") (unit 1)
-        )
-        (path "/ab6dbce1-4ecf-44ae-8f33-5f07e4f43ca9/32afee9c-f78c-4810-b9e6-48288995c3da"
-          (reference "#PWR027") (unit 1)
-        )
-      )

Commit message: Flipping J5/6 to have GND on Pin 1; Invert the Shaft Eye's ISR
Connections:
- net 3.3V-Eye1: now also J2.3 (Pin_3); no longer J2.1 (Pin_1)
- net 3.3V-Eye2: now also J1.3 (Pin_3); no longer J1.1 (Pin_1)
- net GND1: now also J2.1 (Pin_1); no longer J2.3 (Pin_3)
- net GND2: now also J1.1 (Pin_1); no longer J1.3 (Pin_3)
Changed lines of the file:
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@@
     )
   )
-  (symbol (lib_id "Connector_Generic:Conn_01x03") (at 116.205 73.66 0) (unit 1)
+  (symbol (lib_id "Connector_Generic:Conn_01x03") (at 116.205 73.66 0) (mirror x) (unit 1)
     (in_bom no) (on_board yes) (dnp no)
-    (property "Reference" "J2" (at 114.935 68.58 0)
-      (effects (font (size 1.27 1.27)) (justify left))
-    )
-    (property "Value" "Film End Eye" (at 107.315 80.01 0)
+    (property "Reference" "J2" (at 115.57 67.945 0)
+      (effects (font (size 1.27 1.27)) (justify left))
+    )
+    (property "Value" "Film End Eye" (at 112.395 78.74 0)
       (effects (font (size 1.27 1.27)) (justify left))
     )
@@
     )
   )
-  (symbol (lib_id "Connector_Generic:Conn_01x03") (at 117.475 119.38 0) (unit 1)
+  (symbol (lib_id "Connector_Generic:Conn_01x03") (at 117.475 119.38 0) (mirror x) (unit 1)
     (in_bom no) (on_board yes) (dnp no)
-    (property "Reference" "J1" (at 116.205 114.3 0)
-      (effects (font (size 1.27 1.27)) (justify left))
-    )
-    (property "Value" "Shaft Eye" (at 108.585 125.73 0)
-      (effects (font (size 1.27 1.27)) (justify left))
-    )
+    (property "Reference" "J1" (at 116.84 113.665 0)
+      (effects (font (size 1.27 1.27)) (justify left))
+    )
+    (property "Value" "Shaft Eye" (at 114.3 125.095 0)
+      (effects (font (size 1.27 1.27)) (justify left))
+    )

Commit message: Freeing up D4 (328) as it isn't needed
Parts:
- renumbered C1 to C12, C4 to C13, C5 to C14, J1 to J5, J2 to J6, Q2 to Q5, Q2 to Q8, R1 to R19, R5 to R20, R4 to R21, R10 to R22, R6 to R23, R7 to R24, R8 to R25, R9 to R26, R12 to R27, R13 to R28, TP7 to TP10, TP8 to TP11, U1 to U2, U2 to U3, U3 to U4
Connections:
- net Film End renamed Film End LED

Commit message: TPs renamed (using https://forum.kicad.info/t/answer-how-to-avoid-annotate-adding-number-but-still-label-pcb/38283/17)
Parts:
- TP10: footprint TestPoint:TestPoint_Pad_1.5x1.5mm -> Peacemans_Footprints:TestPoint_THTPad_1.5x1.5mm_Drill0.7mm_named; symbol Connector:TestPoint -> Peacemans_Teile:TestPoint_named; TP_Label (none) -> Shaft; now in the parts list
- TP11: footprint TestPoint:TestPoint_Pad_1.5x1.5mm -> Peacemans_Footprints:TestPoint_THTPad_1.5x1.5mm_Drill0.7mm_named; symbol Connector:TestPoint -> Peacemans_Teile:TestPoint_named; TP_Label (none) -> No Film; now in the parts list
Changed lines of the file:
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@@
     )
   )
-  (symbol (lib_id "Connector:TestPoint") (at 200.025 121.92 180) (unit 1)
-    (in_bom no) (on_board yes) (dnp no)
+  (symbol (lib_id "Peacemans_Teile:TestPoint_named") (at 200.025 121.92 180) (unit 1)
+    (in_bom yes) (on_board yes) (dnp no)
     (property "Reference" "TP11" (at 206.375 125.095 0)
       (effects (font (size 1.27 1.27)) (justify left))
@@
       (effects (font (size 1.27 1.27)) (justify left))
     )
-    (property "Footprint" "TestPoint:TestPoint_Pad_1.5x1.5mm" (at 194.945 121.92 0)
+    (property "Footprint" "Peacemans_Footprints:TestPoint_THTPad_1.5x1.5mm_Drill0.7mm_named" (at 194.945 121.92 0)
       (effects (font (size 1.27 1.27)) hide)
     )
@@
       (effects (font (size 1.27 1.27)) hide)
     )
-    (property "LCSC" "" (at 200.025 121.92 0)
-      (effects (font (size 1.27 1.27)) hide)
-    )
-    (property "Inventory" "" (at 200.025 121.92 0)
-      (effects (font (size 1.27 1.27)) hide)
+    (property "TP_Label" "No Film" (at 200.025 121.92 0)
+      (effects (font (size 1.27 1.27)))
     )
     (pin "1")
@@
     )
   )
-  (symbol (lib_id "Connector:TestPoint") (at 199.39 76.2 180) (unit 1)
-    (in_bom no) (on_board yes) (dnp no)
+  (symbol (lib_id "Peacemans_Teile:TestPoint_named") (at 199.39 76.2 180) (unit 1)
+    (in_bom yes) (on_board yes) (dnp no)
     (property "Reference" "TP10" (at 205.74 79.375 0)
       (effects (font (size 1.27 1.27)) (justify left))
@@
       (effects (font (size 1.27 1.27)) (justify left))
     )
-    (property "Footprint" "TestPoint:TestPoint_Pad_1.5x1.5mm" (at 194.31 76.2 0)
+    (property "Footprint" "Peacemans_Footprints:TestPoint_THTPad_1.5x1.5mm_Drill0.7mm_named" (at 194.31 76.2 0)
       (effects (font (size 1.27 1.27)) hide)
     )
@@
       (effects (font (size 1.27 1.27)) hide)
     )
-    (property "LCSC" "" (at 199.39 76.2 0)
-      (effects (font (size 1.27 1.27)) hide)
-    )
-    (property "Inventory" "" (at 199.39 76.2 0)
-      (effects (font (size 1.27 1.27)) hide)
-    )
-    (pin "1")
+    (property "TP_Label" "Shaft" (at 199.39 76.2 0)
+      (effects (font (size 1.27 1.27)))
+    )
+    (pin "1")

Commit message: Replacing D6 LED with 1N4148 Adding TPs for Lamp Current Fixing TP Labels and other Labels Add LED D9 that actually reflects Lamp status Add control LEDs for Eyes (makes mounting much easier) Add mini manual and tech specs on the back side
Parts:
- added D10: Shaft (re), LED_SMD:LED_0805_2012Metric, symbol Device:LED_Small
- added D3: No Film (re), LED_SMD:LED_0805_2012Metric, symbol Device:LED_Small
- added R18, R44: 300R, Resistor_SMD:R_0805_2012Metric, symbol Device:R_Small
Connections:
- net GNDD: now also D10.1 (K), D3.1 (K)
- net Main Shaft: no longer TP10.1
- net at R27.1, U2.2: now also TP10.1, R44.2
- net at R28.1, U2.6: now also TP11.1, R18.2
- net Film End LED renamed Film End
- net Film End: no longer TP11.1
- new net: D3.2 (A), R18.1
- new net: D10.2 (A), R44.1
Other:
- moved on the sheet: C13, TP10, TP11

Commit message: Reannotated
Parts:
- renumbered C12 to C20, C13 to C21, C14 to C22, CN3 to CN5, CN2 to CN6, D10 to D7, J5 to J2, J6 to J3, Q8 to Q5, Q5 to Q6, R21 to R1, R18 to R11, R23 to R20, R25 to R22, R27 to R24, R28 to R27, R44 to R29, R19 to R3, R26 to R30, R24 to R31, R20 to R5, R22 to R6, TP11 to TP3, U3 to U1, U4 to U2, U2 to U9
