File: scan-controller-kicad/sensors.kicad_sch (KiCad schematic)
At the start: 28 parts, among them CN5 Film End Eye, CN6 Shaft Eye, J2 Shaft Eye, J3 Film End Eye, Q5 SS8050, Q6 SS8050, U1 QRE1113, U2 QRE1113, U9 74LVC14

Commit message: Hiding some Refs the right way
Parts:
- R1, R3, R5, R6: footprint Resistor_SMD:R_0402_1005Metric -> Peacemans_Footprints:R_0402_1005Metric-noref; symbol Device:R_Small -> Peacemans_Teile:R_Small_0402-noref
Changed lines of the file:
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@@
     )
   )
-  (symbol (lib_id "Device:R_Small") (at 107.315 114.3 0) (unit 1)
+  (symbol (lib_id "Peacemans_Teile:R_Small_0402-noref") (at 107.315 114.3 0) (unit 1)
     (in_bom yes) (on_board yes) (dnp no)
     (property "Reference" "R1" (at 104.775 114.3 90)
@@
       (effects (font (size 1.27 1.27)) (justify left))
     )
-    (property "Footprint" "Resistor_SMD:R_0402_1005Metric" (at 107.315 114.3 0)
+    (property "Footprint" "Peacemans_Footprints:R_0402_1005Metric-noref" (at 107.315 114.3 0)
       (effects (font (size 1.27 1.27)) hide)
     )
@@
     )
   )
-  (symbol (lib_id "Device:R_Small") (at 90.805 68.58 0) (unit 1)
+  (symbol (lib_id "Peacemans_Teile:R_Small_0402-noref") (at 90.805 68.58 0) (unit 1)
     (in_bom yes) (on_board yes) (dnp no)
     (property "Reference" "R5" (at 93.345 68.58 90)
@@
       (effects (font (size 1.27 1.27)) (justify left))
     )
-    (property "Footprint" "Resistor_SMD:R_0402_1005Metric" (at 90.805 68.58 0)
+    (property "Footprint" "Peacemans_Footprints:R_0402_1005Metric-noref" (at 90.805 68.58 0)
       (effects (font (size 1.27 1.27)) hide)
     )
@@
     )
   )
-  (symbol (lib_id "Device:R_Small") (at 106.045 68.58 0) (unit 1)
+  (symbol (lib_id "Peacemans_Teile:R_Small_0402-noref") (at 106.045 68.58 0) (unit 1)
     (in_bom yes) (on_board yes) (dnp no)
     (property "Reference" "R6" (at 103.505 68.58 90)
@@
       (effects (font (size 1.27 1.27)) (justify left))
     )
-    (property "Footprint" "Resistor_SMD:R_0402_1005Metric" (at 106.045 68.58 0)
+    (property "Footprint" "Peacemans_Footprints:R_0402_1005Metric-noref" (at 106.045 68.58 0)
       (effects (font (size 1.27 1.27)) hide)
     )
@@
     )
   )
-  (symbol (lib_id "Device:R_Small") (at 92.075 114.3 0) (unit 1)
+  (symbol (lib_id "Peacemans_Teile:R_Small_0402-noref") (at 92.075 114.3 0) (unit 1)
     (in_bom yes) (on_board yes) (dnp no)
     (property "Reference" "R3" (at 94.615 114.3 90)
@@
       (effects (font (size 1.27 1.27)) (justify left))
     )
-    (property "Footprint" "Resistor_SMD:R_0402_1005Metric" (at 92.075 114.3 0)
-      (effects (font (size 1.27 1.27)) hide)
-    )
+    (property "Footprint" "Peacemans_Footprints:R_0402_1005Metric-noref" (at 92.075 114.3 0)
+      (effects (font (size 1.27 1.27)) hide)
+    )

Commit message: Updating 3p Terminal Blocks to some available type
Parts:
- CN5, CN6: footprint easyeda2kicad:CONN-TH_3P-P2.54_KF141R-2.54-3P -> easyeda2kicad:CONN-TH_3P-P2.54_DIBO_DB141R-2.54-3P; LCSC C475125 -> C2898755
Changed lines of the file:
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@@
       (effects (font (size 1.27 1.27)) (justify left))
     )
-    (property "Footprint" "easyeda2kicad:CONN-TH_3P-P2.54_KF141R-2.54-3P" (at 140.97 63.5 0)
+    (property "Footprint" "easyeda2kicad:CONN-TH_3P-P2.54_DIBO_DB141R-2.54-3P" (at 140.97 63.5 0)
       (effects (font (size 1.27 1.27)) hide)
     )
@@
       (effects (font (size 1.27 1.27)) hide)
     )
-    (property "LCSC" "C475125" (at 140.97 73.66 0)
+    (property "LCSC" "C2898755" (at 140.97 73.66 0)
       (effects (font (size 1.27 1.27)) hide)
     )
     (property "Inventory" "" (at 140.97 73.66 0)
+      (effects (font (size 1.27 1.27)) hide)
+    )
+    (property "Sim.Device" "C475125" (at 140.97 73.66 0)
       (effects (font (size 1.27 1.27)) hide)
     )
@@
       (effects (font (size 1.27 1.27)) (justify left))
     )
-    (property "Footprint" "easyeda2kicad:CONN-TH_3P-P2.54_KF141R-2.54-3P" (at 141.605 109.22 0)
+    (property "Footprint" "easyeda2kicad:CONN-TH_3P-P2.54_DIBO_DB141R-2.54-3P" (at 141.605 109.22 0)
       (effects (font (size 1.27 1.27)) hide)
     )
@@
       (effects (font (size 1.27 1.27)) hide)
     )
-    (property "LCSC" "C475125" (at 141.605 119.38 0)
+    (property "LCSC" "C2898755" (at 141.605 119.38 0)
       (effects (font (size 1.27 1.27)) hide)
     )
@@
       (effects (font (size 1.27 1.27)) hide)
     )
+    (property "Sim.Device" "C475125" (at 141.605 119.38 0)
+      (effects (font (size 1.27 1.27)) hide)
+    )
