File: scan-controller-kicad/scan-controller-kicad-backups/scan-controller-kicad-2023-11-09_001220/scan-controller-kicad.kicad_sch (KiCad schematic)
At the start: 101 parts, among them CN1 24V in, CN2 Shaft Eye, CN3 Film End Eye, CN4 Lamp, CN5 Fan, CN6 Motor, J1 Shaft Eye, J2 Film End Eye, J3 Raspi GPIO, J4 Raspi UART, J5 ICSP, J6 FTDI, Q1 IRF7470, Q2 BC848, Q5 BC817, Q6 IRLML2502, Q7 IRLML6402, SW1 Power, SW10 Rec, SW2 Lamp, SW3 Zoom, SW4 <<, SW5 <, SW6 Reset, SW7 Stop, SW8 >, SW9 >>, U1 74LVC14, U2 QRE1113, U3 QRE1113, U5 DRV8871DDA, U6 ATmega328P, Y1 8MHz

Commit message: Adding ZVD to protect the Raspi fro FTDI- or ICSP-Powering
Parts:
- added Q10, Q3: DMMT5401, Package_TO_SOT_SMD:SOT-23-6, symbol Device:Q_Dual_PNP_PNP_C1B1B2C2E2E1
- added Q11, Q4: DMG2305UX, Package_TO_SOT_SMD:SOT-23, symbol Device:Q_PMOS_GSD
- added R11, R35: 10K, Resistor_SMD:R_0805_2012Metric, symbol Device:R_Small
- added R14, R36: 47K, Resistor_SMD:R_0805_2012Metric, symbol Device:R_Small
- R18: value 47K -> 10K
Connections:
- net Zero Voltage Diode/K is gone; now on net 3.3V-RPi: Q7.2 (S), R17.1
- net +5V: now also Q3.5 (E2), Q3.6 (E1), Q4.2 (S), Q4.3 (D)
- net 3.3V-RPi: now also Q10.6 (E1), Q11.3 (D)
- net GND: now also R11.2, R14.2, R35.2, R36.2
- new net: Q3.4 (C2), Q4.1 (G), R14.1
- new net: Q10.4 (C2), Q11.1 (G), R36.1
- new net: Q10.5 (E2), Q11.2 (S)
- new net: Q10.1 (C1), Q10.2 (B1), Q10.3 (B2), R35.1
- new net: Q3.1 (C1), Q3.2 (B1), Q3.3 (B2), R11.1
Other:
- sheet Zero Voltage Diode: file ZVD.kicad_sch -> zero_voltage_diode.kicad_sch
- sheet Zero Voltage Diode ports: added none; removed A, K
- moved on the sheet: Q6, Q7, R16, R17, R18
