File: scan-controller-kicad/scan-controller-kicad-backups/scan-controller-kicad-2023-11-09_001220/zero_voltage_diode.kicad_sch (KiCad schematic)
At the start: 4 parts, among them Q3 DMMT5401, Q4 DMG2305UX

Commit message: Adding ZVD to protect the Raspi fro FTDI- or ICSP-Powering
Connections:
- net A renamed +5V
- net K renamed Raspi-5V
