File: scan-controller/scan-controller-kicad/scan-controller-kicad.kicad_pcb (KiCad board)
At the start: 2 copper layers, 122.2 x 113 mm, 144 parts, among them CN1 24V in, CN2 Motor, CN3 Fan, CN4 Lamp, CN5 Film End Eye, CN6 Shaft Eye, J1 FTDI, J2 Shaft Eye, J3 Film End Eye, J4 Target, J5 ICSP, J6 Raspi UART, J7 Raspi GPIO, Q1 IRF7470, Q2 IRLML2502, Q3 IRLML6402, Q4 DMG2305UX, Q5 SS8050, Q6 SS8050, Q7 DMMT5401, Q8 SS8050, SW1 Power, SW10 >>, SW11 Rec, SW2 Target, SW3 Reset, SW4 Lamp, SW5 <<, SW6 Zoom, SW7 Stop, SW8 <, SW9 >, U1 QRE1113, U2 QRE1113, U3 78L05, U4 DRV8871DDA, U5 ATmega328P, U6 TL431, U7 XL4015, U8 LM358, U9 74LVC14, Y1 8MHz

Commit message: Switching back to Rev-B (newer Displays have their outputs on the left hand side)
Parts:
- moved D1 72.9 mm to (130.1, 58.1), turned to -90 degrees
- moved R7 67.0 mm to (130.1, 63.7), turned to -90 degrees
- moved SW1 66.2 mm to (136.3, 59.3), turned to 180 degrees
- moved RV4 47.5 mm to (149.9, 64.6), turned to 180 degrees
- moved RV5 45.3 mm to (165.6, 64.6), turned to 180 degrees
- moved D7 42.2 mm to (154.9, 118.9), turned to 0 degrees
- moved TP10 38.4 mm to (158.0, 116.6), turned to 90 degrees
- moved R29 36.9 mm to (154.9, 115.6), turned to 180 degrees
- moved D3 12.0 mm to (131.8, 108.5), turned to 0 degrees
- moved R11 11.5 mm to (138.7, 110.0)
- moved TP3 2.05 mm to (131.8, 112.8)
Routing:
- net /A6: track 56.1 -> 85.7 mm, vias 1 -> 2
- net Net-(R24-Pad1): track 51.2 -> 30.0 mm
- net /SCL: track 161.2 -> 145.5 mm, vias 9 -> 6
- net /A3: track 45.4 -> 50.8 mm, vias 2 -> 1
- net Net-(R11-Pad2): track 28.5 -> 33.6 mm, vias 4 -> 6
- net /A2: track 35.4 -> 39.8 mm, vias 0 -> 1
- net 3.3V-uC: track 63.4 -> 60.2 mm
- net Net-(J1-Pin_6): track 37.6 -> 36.0 mm, vias 1 -> 0
- net /A0: track 102.5 -> 101.5 mm, vias 4 -> 3
- net Net-(D7-A): track 4.31 -> 3.31 mm
- net Net-(R21-Pad2): track 20.2 -> 21.0 mm
- net /~{RST}: track 92.2 -> 91.5 mm, vias 9 -> 7
- net Net-(D1-A): track 4.30 -> 3.75 mm

Commit message: Initial Rev.C work
Parts:
- added R41: 47K, Resistor_SMD:R_0805_2012Metric, F.Cu at (209.4, 57.9)
- moved D1 10.4 mm to (130.9, 47.8)
- moved R7 10.4 mm to (130.9, 53.4)
- moved SW1 10.4 mm to (137.1, 49.0)
- moved RV3 10.3 mm to (201.6, 52.6)
- moved RV1 10.2 mm to (190.5, 52.6)
- moved RV2 10.2 mm to (179.1, 52.6)
- moved J3 6.59 mm to (230.1, 54.3)
- moved REF** 6.59 mm to (227.6, 46.7)
- moved REF** 6.59 mm to (227.6, 55.9)
- moved J2 6.59 mm to (218.4, 54.3)
- moved R1 6.59 mm to (212.9, 48.3)
- moved R3 6.59 mm to (218.9, 48.3)
- moved R5 6.59 mm to (230.6, 48.3)
- moved R6 6.59 mm to (224.5, 48.3)
- moved REF** 6.59 mm to (215.9, 55.9)
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Routing:
- net Net-(D5-K): track 88.1 -> 99.0 mm
- net Net-(U8A--): track 59.2 -> 69.8 mm
- net Net-(R17-Pad2): track 42.3 -> 52.9 mm
- net /Drivers/Lamp-GND: track 38.9 -> 49.5 mm
- net 24VDC: track 124.1 -> 133.5 mm
- net Net-(C15-Pad1): track 81.6 -> 89.5 mm
- net /GPIO17: track 111.3 -> 118.5 mm
- net 3.3V-uC: track 60.2 -> 65.3 mm
- net /A6: track 85.7 -> 89.0 mm
- net GND: track 83.4 -> 86.1 mm
Other:
- board size 122.2 x 113 mm -> 122.2 x 112.8 mm

Commit message: Extend the board and improve usability
Parts:
- added REFe: MountingHole_3.2mm_M3_Pad_Via, MountingHole:MountingHole_3.2mm_M3_Pad_Via, F.Cu at (139.8, 60.2)
- RV4, RV5: footprint easyeda2kicad:RES-TH_RK09K1110A0J -> easyeda2kicad:RES-TH_RK09K1110A0J_short
- moved RV4 4.19 mm to (149.9, 60.5)
- moved RV5 4.06 mm to (165.6, 60.6)
- moved J1 3.89 mm to (122.7, 61.0)
- moved RV2 2.29 mm to (181.4, 52.6)
- moved RV1 1.27 mm to (191.8, 52.6)
- moved RV3 0.55 mm to (202.2, 52.6)
Routing:
- net /SCL: track 145.5 -> 155.6 mm
- net 3.3V-uC: track 65.3 -> 70.9 mm
- net /A6: track 89.0 -> 93.2 mm
- net /A2: track 39.8 -> 43.9 mm
- net /A3: track 50.8 -> 54.3 mm
- net /TX: track 39.7 -> 40.5 mm
- net /Drivers/Lamp-GND: track 49.5 -> 50.0 mm
- net Net-(R17-Pad2): track 52.9 -> 53.4 mm
- net Net-(U8A--): track 69.8 -> 70.3 mm
Other:
- board text added: "DTR"
- board text added: "GND"
- board text added: "Rx"
- board text added: "Tx"
- board text added: "UART"
- board text added: "VDC"
- board text removed: "FTDI"

Commit message: Looking good, just the new 5VDC source is missing
Parts:
- moved SW3 16.6 mm to (124.7, 79.8), turned to -90 degrees
Routing:
- net /~{RST}: track 91.5 -> 103.7 mm
- net Net-(C15-Pad1): track 89.3 -> 91.8 mm
Other:
- board text added: "4.3{dblquote} Display"

Commit message: Routing WIP
Parts:
- removed Q8: SS8050, Package_TO_SOT_SMD:SOT-23
- removed R38: 2K2, Resistor_SMD:R_0805_2012Metric
- added C25: 10u/50V, Capacitor_SMD:C_1210_3225Metric, F.Cu at (145.4, 84.4)
- added C26: 100n/50V, Capacitor_SMD:C_0805_2012Metric, F.Cu at (145.4, 77.8)
- added C27: 10u, Capacitor_SMD:C_0805_2012Metric, F.Cu at (136.2, 70.7)
- added D10: SS54, Diode_SMD:D_SMA, F.Cu at (215.6, 107.5)
- added D9: PMEG6020ER, Diode_SMD:D_SOD-123F, F.Cu at (141.5, 77.1)
- added L2: 10uH, easyeda2kicad:IND-SMD_L4.4-W4.2, F.Cu at (145.4, 71.9)
- added R42: 10K, Resistor_SMD:R_0805_2012Metric, F.Cu at (140.5, 70.7)
- added R43: 2K7, Resistor_SMD:R_0805_2012Metric, F.Cu at (141.0, 84.4)
- added RV6: 25K, easyeda2kicad:RES-ADJ-TH_3P-L10.0-W10.0-P2.50-L, F.Cu at (137.7, 77.3)
- added U10: LGS5145, easyeda2kicad:SOT-23-6_L2.9-W1.7-P0.95-LS2.8-BL, F.Cu at (145.4, 80.8)
- moved R8 4.72 mm to (160.0, 92.5), turned to -90 degrees
- moved R9 4.41 mm to (159.8, 88.6), turned to 0 degrees
- moved Q1 4.35 mm to (161.8, 83.8)
- moved C15 0.77 mm to (206.8, 106.4)
Connections:
- CN3 pad 1: Net-(D8-A) -> GND
- CN3 pad 3: 5V-RPi -> Net-(D10-K)
- D8 pad 1: 5V-RPi -> Net-(D10-A)
- D8 pad 2: Net-(D8-A) -> GND
Routing:
- net 5V-RPi: track 49.5 -> 9.17 mm
- net /D8: track 71.9 -> 103.3 mm, vias 2 -> 4
- net 24VDC: track 133.5 -> 160.8 mm
- net GND: track 86.1 -> 107.3 mm, vias 3 -> 4
- net Net-(D8-A): track 19.2 -> 0.00 mm, vias 1 -> 0
- net Net-(D10-A): track 0.00 -> 16.5 mm
- net Net-(D10-K): track 0.00 -> 11.1 mm
- net Net-(D9-K): track 0.00 -> 10.7 mm
- net /A6: track 93.2 -> 103.8 mm, vias 2 -> 3
- net Net-(U10-FB): track 0.00 -> 9.75 mm
- net /SCL: track 155.6 -> 164.3 mm
- net /A2: track 43.9 -> 51.9 mm
- net Net-(R42-Pad2): track 0.00 -> 7.38 mm
- net /A3: track 54.3 -> 61.0 mm
- net Net-(Q8-B): track 3.87 -> 0.00 mm
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Other:
- board text added: "Fan Speed"

Commit message: DRC happy!
Parts:
- moved TP6 0.51 mm to (159.5, 102.9)
- moved TP7 0.51 mm to (159.5, 97.0)
- moved TP5 0.51 mm to (159.5, 100.3)
- turned RV6 to -90 degrees
Routing:
- net Net-(D10-A): track 16.5 -> 119.8 mm, vias 0 -> 2
- net /D8: track 103.3 -> 36.3 mm
- net /SCL: track 164.3 -> 163.8 mm
- net /SDA: track 100.2 -> 100.7 mm
- net /~{RST}: track 103.7 -> 103.9 mm, vias 7 -> 9
- net 24VDC: vias 0 -> 2
- net /A6: vias 3 -> 2
