File: scan-controller/scan-controller-kicad/scan-controller-kicad.kicad_pcb (KiCad board)
At the start: 2 copper layers, 122.2 x 112.8 mm, 154 parts, among them CN1 24V in, CN2 Motor, CN3 Fan, CN4 Lamp, CN5 Film End Eye, CN6 Shaft Eye, J1 FTDI, J2 Shaft Eye, J3 Film End Eye, J4 Target, J5 ICSP, J6 Raspi UART, J7 Raspi GPIO, Q1 IRF7470, Q2 IRLML2502, Q3 IRLML6402, Q4 DMG2305UX, Q5 SS8050, Q6 SS8050, Q7 DMMT5401, SW1 Power, SW10 >>, SW11 Rec, SW2 Target, SW3 Reset, SW4 Lamp, SW5 <<, SW6 Zoom, SW7 Stop, SW8 <, SW9 >, U1 QRE1113, U10 LGS5145, U2 QRE1113, U3 78L05, U4 DRV8871DDA, U5 ATmega328P, U6 TL431, U7 XL4015, U8 LM358, U9 74LVC14, Y1 8MHz

Commit message: Adding a Gate Driver and making the MOSFET tougher. DRC happy!
Parts:
- added C28: 100n, Capacitor_SMD:C_0402_1005Metric, F.Cu at (149.6, 84.6)
- added U11: MCP1416, Package_TO_SOT_SMD:SOT-23-5, F.Cu at (152.4, 85.0)
- Q1: value IRF7470 -> CS12N06AE-G
- R8: value 150R -> 10R
- moved R8 8.29 mm to (156.2, 85.1), turned to 90 degrees
- moved R9 0.51 mm to (159.8, 88.1)
Connections:
- R8 pad 2: /D9 -> Net-(U11-OUT)
Routing:
- net 5V-RPi: track 9.17 -> 88.9 mm, vias 0 -> 2
- net /D9: track 80.5 -> 85.9 mm
- net GND: track 107.3 -> 112.2 mm
- net Net-(U11-OUT): track 0.00 -> 2.71 mm
- net Net-(Q1-G): track 6.50 -> 5.44 mm

Commit message: weaker mousebites. removed orphaned traces and vias
Parts:
- REF** (x2): value Eye_Mousebites -> Eye_Mousebites_weaker; footprint Peacemans_Footprints:Eye_Mousebites -> Peacemans_Footprints:Eye_Mousebites_weaker
Routing:
- net /A0: track 101.5 -> 100.2 mm
- net Net-(R37-Pad2): track 17.1 -> 16.0 mm
- net Net-(R32-Pad2): track 17.0 -> 16.1 mm
- net /D5: track 74.9 -> 75.8 mm
- net Net-(R37-Pad1): track 16.8 -> 16.0 mm
- net Net-(R21-Pad2): track 21.0 -> 20.1 mm
- net /A6: track 103.8 -> 103.1 mm
- net Net-(J3-Pin_2): track 8.21 -> 7.63 mm
- net Net-(J2-Pin_2): track 8.21 -> 7.62 mm
- net 3.3V-uC: track 70.9 -> 70.3 mm
- net /SDA: track 100.7 -> 100.2 mm

Commit message: Rev. C, as ordered
Changed lines of the file:
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@@
         (effects (font (size 1 1) (thickness 0.15)))
     )
-    (pad "" np_thru_hole circle (at -3.75 0) (size 0.5 0.5) (drill 0.6) (layers "F&B.Cu" "*.Mask"))
-    (pad "" np_thru_hole circle (at -3 0) (size 0.5 0.5) (drill 0.6) (layers "F&B.Cu" "*.Mask"))
-    (pad "" np_thru_hole circle (at -2.25 0) (size 0.5 0.5) (drill 0.6) (layers "F&B.Cu" "*.Mask"))
-    (pad "" np_thru_hole circle (at -1.5 0) (size 0.5 0.5) (drill 0.6) (layers "F&B.Cu" "*.Mask"))
-    (pad "" np_thru_hole circle (at -0.75 0) (size 0.5 0.5) (drill 0.6) (layers "F&B.Cu" "*.Mask"))
-    (pad "" np_thru_hole circle (at 0 0) (size 0.5 0.5) (drill 0.6) (layers "F&B.Cu" "*.Mask"))
-    (pad "" np_thru_hole circle (at 0.75 0) (size 0.5 0.5) (drill 0.6) (layers "F&B.Cu" "*.Mask"))
-    (pad "" np_thru_hole circle (at 1.5 0) (size 0.5 0.5) (drill 0.6) (layers "F&B.Cu" "*.Mask"))
-    (pad "" np_thru_hole circle (at 2.25 0) (size 0.5 0.5) (drill 0.6) (layers "F&B.Cu" "*.Mask"))
-    (pad "" np_thru_hole circle (at 3 0) (size 0.5 0.5) (drill 0.6) (layers "F&B.Cu" "*.Mask"))
-    (pad "" np_thru_hole circle (at 3.75 0) (size 0.5 0.5) (drill 0.6) (layers "F&B.Cu" "*.Mask"))
-    (group "" (id 738983a3-dac3-400c-bb32-40ff424d399c)
+    (pad "" np_thru_hole circle (at -3.75 0) (size 0.5 0.5) (drill 0.55) (layers "F&B.Cu" "*.Mask"))
+    (pad "" np_thru_hole circle (at -3 0) (size 0.5 0.5) (drill 0.55) (layers "F&B.Cu" "*.Mask"))
+    (pad "" np_thru_hole circle (at -2.25 0) (size 0.5 0.5) (drill 0.55) (layers "F&B.Cu" "*.Mask"))
+    (pad "" np_thru_hole circle (at -1.5 0) (size 0.5 0.5) (drill 0.55) (layers "F&B.Cu" "*.Mask"))
+    (pad "" np_thru_hole circle (at -0.75 0) (size 0.5 0.5) (drill 0.55) (layers "F&B.Cu" "*.Mask"))
+    (pad "" np_thru_hole circle (at 0 0) (size 0.5 0.5) (drill 0.55) (layers "F&B.Cu" "*.Mask"))
+    (pad "" np_thru_hole circle (at 0.75 0) (size 0.5 0.5) (drill 0.55) (layers "F&B.Cu" "*.Mask"))
+    (pad "" np_thru_hole circle (at 1.5 0) (size 0.5 0.5) (drill 0.55) (layers "F&B.Cu" "*.Mask"))
+    (pad "" np_thru_hole circle (at 2.25 0) (size 0.5 0.5) (drill 0.55) (layers "F&B.Cu" "*.Mask"))
+    (pad "" np_thru_hole circle (at 3 0) (size 0.5 0.5) (drill 0.55) (layers "F&B.Cu" "*.Mask"))
+    (pad "" np_thru_hole circle (at 3.75 0) (size 0.5 0.5) (drill 0.55) (layers "F&B.Cu" "*.Mask"))
+    (group "" (id ca347249-9ab3-4959-b5ec-ecb4288b718f)
       (members
-        09aebba8-7c39-4580-a249-72b7adaf4ad0
-        148e4c0c-8bcb-4ad5-a337-48a889f44938
-        29deec68-be90-4287-9a85-0b84b1140f7c
-        42cd1eaa-e139-4b9f-8171-813002857409
-        5b4ccc14-c871-43a9-bd0d-affbf8e87808
-        6025f7ad-ed76-4483-9031-ba61be994a4c
-        7999d9c7-0e48-49f0-8caa-ff23cd56041b
-        8b99e973-b9f2-4415-8285-bd50aa890eb9
-        91bfd9e9-b32c-403f-9726-c239753c3fa0
-        d8f9ed6f-3cbb-4467-8253-3f68aad2a615
-        e4297b9e-c6ff-4c90-9ede-cfe66cc629fd
+        0074b195-33b6-47f6-b4b5-653f560f5519
+        110f74f8-9242-47a8-85e9-4c5e2b062943
+        783a3ae6-92b2-40cb-837c-d15285b6a09e
+        ac25e4e5-81e1-44f8-8327-5ffcdebb08b2
+        cbc7385f-85a5-40e1-9300-bf3f3d6782fe
+        cd31d2e0-a602-4dc2-8cdc-03f59f89efa9
+        cf4dc2fe-bfb6-4b3b-b292-89f57ba8867f
+        d90c09af-584b-4dc9-bee3-91a1333d192f
+        e949d99b-1a79-4c36-9903-6be69f5c5e1d
+        fab99fc8-8058-430c-b309-33d4ed500f82
+        fcf27ddc-4d20-4919-a69d-c27c7ae9ff2b
       )
     )
@@
         (effects (font (size 1 1) (thickness 0.15)))
     )
-    (pad "" np_thru_hole circle (at -3.75 0) (size 0.5 0.5) (drill 0.6) (layers "F&B.Cu" "*.Mask"))
-    (pad "" np_thru_hole circle (at -3 0) (size 0.5 0.5) (drill 0.6) (layers "F&B.Cu" "*.Mask"))
-    (pad "" np_thru_hole circle (at -2.25 0) (size 0.5 0.5) (drill 0.6) (layers "F&B.Cu" "*.Mask"))
-    (pad "" np_thru_hole circle (at -1.5 0) (size 0.5 0.5) (drill 0.6) (layers "F&B.Cu" "*.Mask"))
-    (pad "" np_thru_hole circle (at -0.75 0) (size 0.5 0.5) (drill 0.6) (layers "F&B.Cu" "*.Mask"))
-    (pad "" np_thru_hole circle (at 0 0) (size 0.5 0.5) (drill 0.6) (layers "F&B.Cu" "*.Mask"))
-    (pad "" np_thru_hole circle (at 0.75 0) (size 0.5 0.5) (drill 0.6) (layers "F&B.Cu" "*.Mask"))
-    (pad "" np_thru_hole circle (at 1.5 0) (size 0.5 0.5) (drill 0.6) (layers "F&B.Cu" "*.Mask"))
-    (pad "" np_thru_hole circle (at 2.25 0) (size 0.5 0.5) (drill 0.6) (layers "F&B.Cu" "*.Mask"))
-    (pad "" np_thru_hole circle (at 3 0) (size 0.5 0.5) (drill 0.6) (layers "F&B.Cu" "*.Mask"))
-    (pad "" np_thru_hole circle (at 3.75 0) (size 0.5 0.5) (drill 0.6) (layers "F&B.Cu" "*.Mask"))
-    (group "" (id 30b5dd98-92d9-4865-889c-fc856d1b0c20)
+    (pad "" np_thru_hole circle (at -3.75 0) (size 0.5 0.5) (drill 0.55) (layers "F&B.Cu" "*.Mask"))
+    (pad "" np_thru_hole circle (at -3 0) (size 0.5 0.5) (drill 0.55) (layers "F&B.Cu" "*.Mask"))
+    (pad "" np_thru_hole circle (at -2.25 0) (size 0.5 0.5) (drill 0.55) (layers "F&B.Cu" "*.Mask"))
+    (pad "" np_thru_hole circle (at -1.5 0) (size 0.5 0.5) (drill 0.55) (layers "F&B.Cu" "*.Mask"))
+    (pad "" np_thru_hole circle (at -0.75 0) (size 0.5 0.5) (drill 0.55) (layers "F&B.Cu" "*.Mask"))
+    (pad "" np_thru_hole circle (at 0 0) (size 0.5 0.5) (drill 0.55) (layers "F&B.Cu" "*.Mask"))
+    (pad "" np_thru_hole circle (at 0.75 0) (size 0.5 0.5) (drill 0.55) (layers "F&B.Cu" "*.Mask"))
+    (pad "" np_thru_hole circle (at 1.5 0) (size 0.5 0.5) (drill 0.55) (layers "F&B.Cu" "*.Mask"))
+    (pad "" np_thru_hole circle (at 2.25 0) (size 0.5 0.5) (drill 0.55) (layers "F&B.Cu" "*.Mask"))
+    (pad "" np_thru_hole circle (at 3 0) (size 0.5 0.5) (drill 0.55) (layers "F&B.Cu" "*.Mask"))
+    (pad "" np_thru_hole circle (at 3.75 0) (size 0.5 0.5) (drill 0.55) (layers "F&B.Cu" "*.Mask"))
+    (group "" (id e3a692bd-40ee-4333-b5ec-3c7b25295802)
       (members
-        19540b9e-914c-4896-9be6-086950708c2b
-        25d855d8-fb21-4f05-b131-c783c8530257
-        308b3530-a8d5-4116-a4d3-4c92a4e0c129
-        4801acef-8b06-4d92-b25c-ff0930fe6271
-        79f2135d-d0ae-40f0-af1c-1cc3b793b09a
-        7a447944-f7fd-4302-bfe2-b24250dcf90a
-        97f96a46-cd1e-4336-8ab3-e7fcd8057df8
-        af0133d0-43af-4f09-8949-8f94cf1bf510
-        b228b6cf-6716-4317-ad90-4a235ecc26d9
-        ece7295c-39bb-4afb-9f42-37caac3007ac
-        f4dcf078-0d06-416d-831b-c6e0b88cfcd1
+        4265dbf4-814e-4c63-9c85-3ed8733ac4d3
+        5158fee9-928e-4c14-a2f2-d3f256b03801
+        54e8116a-3278-4183-a2d9-aab7b55e5000
+        5df63d4b-a007-4bc3-a15e-2b4495d0ac9f
+        5e6b4129-5b59-480a-8ead-2f32a5ce6903
+        64bc6a67-c80a-4b2b-b292-72d191ac2424
+        98decc65-9ccf-40c2-914a-eedc07543c6a
+        a6e122b3-8ea8-4447-9ed3-2a5b3e145dd4
+        b56f2577-794f-466d-b723-d86d16b562ae
+        ba9b5b55-116a-44ed-b5f8-9ce1433b6b9c
+        e869b6f2-8bc9-4748-b191-85d48f49e2ca
       )
     )

Commit message: minor layout tweaks, todos
Routing:
- net /A1: track 119.2 -> 116.7 mm
Changed lines of the file:
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@@
     (fp_line (start 1 0.625) (end -1 0.625)
       (stroke (width 0.1) (type solid)) (layer "F.Fab"))
-    (pad "1" smd roundrect (at -0.9125 0 180) (size 1.025 1.4) (layers "F.Cu" "F.Paste" "F.Mask") (roundrect_rratio 0.243902)
+    (pad "1" smd roundrect (at -0.9125 0 180) (size 1.025 1.4) (layers "F.Cu" "F.Paste" "F.Mask") (roundrect_rratio 0.243902439)
       (net 2 "GND") (pintype "passive"))
-    (pad "2" smd roundrect (at 0.9125 0 180) (size 1.025 1.4) (layers "F.Cu" "F.Paste" "F.Mask") (roundrect_rratio 0.243902)
+    (pad "2" smd roundrect (at 0.9125 0 180) (size 1.025 1.4) (layers "F.Cu" "F.Paste" "F.Mask") (roundrect_rratio 0.243902439)
       (net 1 "24VDC") (pintype "passive"))
     (model "${KICAD6_3DMODEL_DIR}/Resistor_SMD.3dshapes/R_0805_2012Metric.wrl"
@@
     (fp_line (start 1 0.625) (end -1 0.625)
       (stroke (width 0.1) (type solid)) (layer "F.Fab"))
-    (pad "1" smd roundrect (at -0.9125 0 180) (size 1.025 1.4) (layers "F.Cu" "F.Paste" "F.Mask") (roundrect_rratio 0.243902)
+    (pad "1" smd roundrect (at -0.9125 0 180) (size 1.025 1.4) (layers "F.Cu" "F.Paste" "F.Mask") (roundrect_rratio 0.243902439)
       (net 129 "Net-(D10-A)") (pintype "passive"))
-    (pad "2" smd roundrect (at 0.9125 0 180) (size 1.025 1.4) (layers "F.Cu" "F.Paste" "F.Mask") (roundrect_rratio 0.243902)
+    (pad "2" smd roundrect (at 0.9125 0 180) (size 1.025 1.4) (layers "F.Cu" "F.Paste" "F.Mask") (roundrect_rratio 0.243902439)
       (net 127 "Net-(R42-Pad2)") (pintype "passive"))
     (model "${KICAD6_3DMODEL_DIR}/Resistor_SMD.3dshapes/R_0805_2012Metric.wrl"
@@
     (fp_line (start 1 0.625) (end -1 0.625)
       (stroke (width 0.1) (type solid)) (layer "F.Fab"))
-    (pad "1" smd roundrect (at -0.9125 0 90) (size 1.025 1.4) (layers "F.Cu" "F.Paste" "F.Mask") (roundrect_rratio 0.243902)
+    (pad "1" smd roundrect (at -0.9125 0 90) (size 1.025 1.4) (layers "F.Cu" "F.Paste" "F.Mask") (roundrect_rratio 0.243902439)
       (net 2 "GND") (pintype "passive"))
-    (pad "2" smd roundrect (at 0.9125 0 90) (size 1.025 1.4) (layers "F.Cu" "F.Paste" "F.Mask") (roundrect_rratio 0.243902)
+    (pad "2" smd roundrect (at 0.9125 0 90) (size 1.025 1.4) (layers "F.Cu" "F.Paste" "F.Mask") (roundrect_rratio 0.243902439)
       (net 128 "Net-(U10-FB)") (pintype "passive"))
     (model "${KICAD6_3DMODEL_DIR}/Resistor_SMD.3dshapes/R_0805_2012Metric.wrl"
@@
     (fp_line (start 1.6 1.25) (end -1.6 1.25)
       (stroke (width 0.1) (type solid)) (layer "F.Fab"))
-    (pad "1" smd roundrect (at -1.475 0 180) (size 1.15 2.7) (layers "F.Cu" "F.Paste" "F.Mask") (roundrect_rratio 0.217391)
+    (pad "1" smd roundrect (at -1.475 0 180) (size 1.15 2.7) (layers "F.Cu" "F.Paste" "F.Mask") (roundrect_rratio 0.2173913043)
       (net 1 "24VDC") (pintype "passive"))
-    (pad "2" smd roundrect (at 1.475 0 180) (size 1.15 2.7) (layers "F.Cu" "F.Paste" "F.Mask") (roundrect_rratio 0.217391)
+    (pad "2" smd roundrect (at 1.475 0 180) (size 1.15 2.7) (layers "F.Cu" "F.Paste" "F.Mask") (roundrect_rratio 0.2173913043)
       (net 2 "GND") (pintype "passive"))
     (model "${KICAD6_3DMODEL_DIR}/Capacitor_SMD.3dshapes/C_1210_3225Metric.wrl"
@@
   (segment (start 150.363593 111.801763) (end 149.215593 112.949763) (width 0.25) (layer "F.Cu") (net 5))
   (segment (start 141.931593 99.487763) (end 139.055593 99.487763) (width 0.25) (layer "F.Cu") (net 5))
+  (segment (start 142.244459 101.236763) (end 143.625593 101.236763) (width 0.25) (layer "F.Cu") (net 5))
   (segment (start 136.111093 130.729763) (end 136.111093 130.325263) (width 0.25) (layer "F.Cu") (net 5))
   (segment (start 185.7 132) (end 185.7 132.05867) (width 0.25) (layer "F.Cu") (net 5))
-  (segment (start 142.410593 101.236763) (end 143.625593 101.236763) (width 0.25) (layer "F.Cu") (net 5))
   (segment (start 185.7 132.05867) (end 186.911093 133.269763) (width 0.25) (layer "F.Cu") (net 5))
   (segment (start 125.222 66.04) (end 122.682 66.04) (width 0.25) (layer "F.Cu") (net 5))
@@
   (segment (start 135.96033 98.6125) (end 136.007593 98.659763) (width 0.25) (layer "F.Cu") (net 5))
   (segment (start 137.211593 115.619763) (end 137.211593 115.301763) (width 0.25) (layer "F.Cu") (net 5))
+  (segment (start 142.185593 101.177897) (end 142.244459 101.236763) (width 0.25) (layer "F.Cu") (net 5))
   (segment (start 130.862 54.2845) (end 130.862 60.4) (width 0.25) (layer "F.Cu") (net 5))
   (segment (start 228.122967 60.677784) (end 228.027284 60.677784) (width 0.25) (layer "F.Cu") (net 5))
@@
   (segment (start 196.658593 137.234763) (end 186.608593 137.234763) (width 0.25) (layer "F.Cu") (net 32))
   (segment (start 153.717879 96.186977) (end 154.608093 95.296763) (width 0.25) (layer "F.Cu") (net 32))
-  (segment (start 152.125593 95.874407) (end 152.703237 95.296763) (width 0.25) (layer "F.Cu") (net 32))
   (segment (start 183.474593 137.718763) (end 159.723093 137.718763) (width 0.25) (layer "F.Cu") (net 32))
+  (segment (start 152.237191 97.236763) (end 153.286977 96.186977) (width 0.25) (layer "F.Cu") (net 32))
   (segment (start 153.787593 108.377763) (end 153.787593 104.313763) (width 0.25) (layer "F.Cu") (net 32))
   (segment (start 186.608593 137.234763) (end 185.283593 135.909763) (width 0.25) (layer "F.Cu") (net 32))
-  (segment (start 152.703237 95.296763) (end 154.608093 95.296763) (width 0.25) (layer "F.Cu") (net 32))
-  (segment (start 152.125593 97.236763) (end 152.125593 95.874407) (width 0.25) (layer "F.Cu") (net 32))
   (segment (start 197.983593 135.909763) (end 196.658593 137.234763) (width 0.25) (layer "F.Cu") (net 32))
   (segment (start 159.723093 137.718763) (end 159.629593 137.625263) (width 0.25) (layer "F.Cu") (net 32))
+  (segment (start 152.125593 97.236763) (end 152.237191 97.236763) (width 0.25) (layer "F.Cu") (net 32))
   (segment (start 153.286977 96.186977) (end 153.717879 96.186977) (width 0.25) (layer "F.Cu") (net 32))
   (segment (start 185.283593 135.909763) (end 183.474593 137.718763) (width 0.25) (layer "F.Cu") (net 32))

Commit message: Minor aesthetics-changes (only) for a Rev.D
Other:
- board text added: "For detailed instructions, see www.filmkorn.org The Controller is powered by the Raspberry Pi. Projector Motor, Fan and Lamp/LED get powered via external Power: Use 12-36 VAC or VDC, e.g. from projector transformer. LED Contant Current Output can be adjusted from 1.5-32V/0-5A, depending on external power supplied."
- board text removed: "For detailed instructions, see www.filmkorn.org The Controller and the Fan are powered by the Raspberry Pi. Projector Motor and Lamp/LED get powered via external Power: Use 12-36 VAC or VDC, e.g. from projector transformer. LED Contant Current Output can be adjusted from 1.5-32V/0-5A, depending on external power supplied."
Changed lines of the file:
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@@
   (gr_arc (start 205.243965 44.704016) (mid 208.469119 46.047341) (end 209.804 49.276)
     (stroke (width 0.1) (type default)) (layer "Edge.Cuts"))
-  (gr_text "For detailed instructions, see www.filmkorn.org\nThe Controller and the Fan are powered by the Raspberry Pi.\nProjector Motor and Lamp/LED get powered via external\nPower: Use 12-36 VAC or VDC, e.g. from projector transformer.\nLED Contant Current Output can be adjusted from 1.5-32V/0-5A, \ndepending on external power supplied." (at 207.518 89.154) (layer "B.SilkS")
+  (gr_text "For detailed instructions, see www.filmkorn.org\nThe Controller is powered by the Raspberry Pi.\nProjector Motor, Fan and Lamp/LED get powered via external\nPower: Use 12-36 VAC or VDC, e.g. from projector transformer.\nLED Contant Current Output can be adjusted from 1.5-32V/0-5A, \ndepending on external power supplied." (at 207.518 89.154) (layer "B.SilkS")
     (effects (font (size 1.5 1.5) (thickness 0.3) bold) (justify left bottom mirror))
   )
@@
     (effects (font (size 1.8 1.8) (thickness 0.3) bold) (justify left bottom))
   )
-  (gr_text_box "Filmkorn-Scanner\nby filmkorn.org 2024 • Rev. C"
+  (gr_text_box "Filmkorn-Scanner\nby filmkorn.org 2024 • Rev. D"
     (start 129.032 185.674) (end 119.732 133.374) (angle 270) (layer "B.SilkS")
       (effects (font (size 2 2) (thickness 0.2)) (justify left top mirror))
   )
-  (gr_text_box "Filmkorn-Scanner\nby filmkorn.org 2024 • Rev. C"
+  (gr_text_box "Filmkorn-Scanner\nby filmkorn.org 2024 • Rev. D"
     (start 129.032 82.816) (end 119.732 135.116) (angle 270) (layer "F.SilkS")
       (effects (font (size 2 2) (thickness 0.2)) (justify left top))
@@
   (segment (start 179.899695 85.263263) (end 182.163263 85.263263) (width 0.25) (layer "B.Cu") (net 42))
   (segment (start 157.254 88.646) (end 166.878 88.646) (width 0.25) (layer "B.Cu") (net 42))
+  (segment (start 205.359 84.963) (end 204.495503 84.099503) (width 0.25) (layer "B.Cu") (net 42))
   (segment (start 146.464356 99.319763) (end 149.129593 99.319763) (width 0.25) (layer "B.Cu") (net 42))
   (segment (start 170.224 85.3) (end 179.862958 85.3) (width 0.25) (layer "B.Cu") (net 42))
   (segment (start 149.129593 99.319763) (end 149.129593 97.759854) (width 0.25) (layer "B.Cu") (net 42))
-  (segment (start 205.359 84.963) (end 204.296 83.9) (width 0.25) (layer "B.Cu") (net 42))
-  (segment (start 204.296 83.9) (end 201.3 83.9) (width 0.25) (layer "B.Cu") (net 42))
+  (segment (start 204.495503 84.099503) (end 201.3 84.099503) (width 0.25) (layer "B.Cu") (net 42))
   (segment (start 179.862958 85.3) (end 179.899695 85.263263) (width 0.25) (layer "B.Cu") (net 42))
   (segment (start 182.163263 85.263263) (end 182.6 85.7) (width 0.25) (layer "B.Cu") (net 42))

Commit message: Renaming Post-MOSFET TP Motor GND to Lamp GND. Doh!
Changed lines of the file:
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@@
         (effects (font (size 1 1) (thickness 0.15)))
     )
-    (fp_text user "${TP_Label}" (at -0.508 -2.286) (layer "F.SilkS" knockout)
+    (fp_text user "Lamp GND" (at -0.508 -2.286) (layer "F.SilkS" knockout)
         (effects (font (size 1 1) (thickness 0.15)))
     )
