File: scan-controller/scan-controller-kicad/scan-controller-kicad.kicad_pcb (KiCad board)
At the start: 4 copper layers, 122.2 x 112.8 mm, 167 parts, among them CN1 24V in, CN2 Motor, CN3 Fan, CN4 Lamp, CN5 Film End Eye, CN6 Shaft Eye, J1 FTDI, J2 Shaft Eye, J3 Film End Eye, J4 Resolution, J5 ICSP, J6 Raspi UART, J7 Raspi GPIO, J8 Target, Q1 CS12N06AE-G, Q2 IRLML2502, Q3 IRLML6402, Q4 DMG2305UX, Q5 SS8050, Q6 SS8050, Q7 DMMT5401, SW1 Power, SW10 >>, SW11 Rec, SW12 Target, SW2 Resolution, SW3 Reset, SW4 Lamp, SW5 <<, SW6 Zoom, SW7 Stop, SW8 <, SW9 >, U1 QRE1113, U10 LGS5145, U11 MCP1416, U2 QRE1113, U3 78L05, U4 DRV8871DDA, U5 ATmega328P, U6 TL431, U7 XL4015, U8 LM358, U9 74LVC14, Y1 8MHz

Commit message: Bigger Ears, DRc not quite happy yet
Parts:
- R1, R3, R5, R6: footprint Peacemans_Teile:R_0402_1005Metric-noref -> Resistor_SMD:R_0603_1608Metric
- moved REF** 1.88 mm to (215.9, 44.8)
- moved REF** 1.88 mm to (227.6, 44.8)
- moved R1 1.66 mm to (212.7, 46.6)
- moved R6 1.66 mm to (224.4, 46.6)
- moved R3 1.66 mm to (219.1, 46.6)
- moved R5 1.66 mm to (230.8, 46.6)
- moved U1 0.86 mm to (215.9, 49.6)
- moved U2 0.86 mm to (227.6, 49.6)
- moved J2 0.40 mm to (218.4, 53.8)
- moved J3 0.40 mm to (230.1, 53.8)
Routing:
- net unconnected-(CN3-Pad2): track 5.08 -> 0.00 mm
- net GND2: track 0.00 -> 2.98 mm, vias 0 -> 2
- net GND1: track 0.00 -> 2.98 mm, vias 0 -> 2
- net Net-(J2-Pin_2): track 7.62 -> 7.73 mm, vias 1 -> 0
- net Net-(J3-Pin_2): track 7.63 -> 7.72 mm, vias 1 -> 0
- net /A3: vias 2 -> 1
- added copper zone on In2.Cu, net /Sensors/3.3V-Eye1
- added copper zone on In2.Cu, net /Sensors/3.3V-Eye2
- added copper zone on In1.Cu, net GND1
- added copper zone on In1.Cu, net GND2
- removed copper zone on B.Cu, net /Sensors/3.3V-Eye1
- removed copper zone on B.Cu, net /Sensors/3.3V-Eye2
- removed copper zone on F.Cu, net GND1
- removed copper zone on F.Cu, net GND2
Other:
- board size 122.2 x 112.8 mm -> 122.2 x 115.1 mm

Commit message: DRC much happier
Parts:
- moved C5 0.13 mm to (133.5, 102.4)
- moved C7 0.13 mm to (136.5, 101.9)
- moved C9 0.13 mm to (136.5, 105.4)

Commit message: DRC mostly happy
Parts:
- removed TP17, TP18: TestPoint, Peacemans_Teile:TestPoint_THTPad_1.5x1.5mm_Drill0.7mm_named
Routing:
- net GND: track 125.1 -> 136.9 mm, vias 75 -> 83

Commit message: Massive LampGND
Parts:
- moved TP9 24.7 mm to (188.5, 81.4)
- moved TP4 11.2 mm to (130.7, 107.4)
- moved TP8 5.04 mm to (157.5, 113.3)
- moved TP10 0.51 mm to (130.7, 104.1)
- moved D7 0.38 mm to (121.5, 104.4)
- moved TP3 0.13 mm to (130.7, 101.0)
- renumbered REF** to H1, REFee to H2, REF** to H3, REFe to H4
Routing:
- net Net-(D10-A): track 120.1 -> 146.0 mm
- net 5V-RPi: track 88.9 -> 114.6 mm
- net Net-(D10-K): track 26.5 -> 11.1 mm
- net Net-(U5-PD7): track 7.05 -> 17.7 mm
- net Net-(U5-PB2): track 10.0 -> 15.4 mm
- net Net-(R11-Pad2): track 40.9 -> 45.8 mm, vias 6 -> 8
- net Net-(D3-A): track 16.4 -> 19.7 mm
- net 3.3V-RPi: track 195.0 -> 197.6 mm
- net Net-(D7-A): track 15.8 -> 18.2 mm
- net Net-(J1-Pin_6): track 39.4 -> 41.4 mm
- net Net-(D5-K): track 99.2 -> 97.7 mm
- net Net-(C15-Pad1): track 92.0 -> 90.8 mm
- net Net-(R24-Pad1): track 38.4 -> 38.9 mm

Commit message: Major refactoring to better EMV in progress
Parts:
- added R46: 10K, Resistor_SMD:R_1206_3216Metric, F.Cu at (186.2, 64.4)
- added R47: 10K, Resistor_SMD:R_1206_3216Metric, F.Cu at (279.0, 77.9)
- added R48: 100K, Resistor_SMD:R_0805_2012Metric, F.Cu at (209.2, 58.9)
- H1, H2, H3, H4: value MountingHole_3.2mm_M3_Pad_Via -> MountingHole
- R41: value 47K -> 10K; footprint Resistor_SMD:R_0805_2012Metric -> Resistor_SMD:R_1206_3216Metric
- moved TP9 74.8 mm to (255.3, 47.8)
- moved C16 33.1 mm to (163.8, 100.6), turned to -90 degrees
- moved U7 32.7 mm to (187.2, 84.7), turned to 0 degrees
- moved D5 30.2 mm to (166.9, 108.1)
- moved R41 28.1 mm to (186.3, 73.9), turned to 90 degrees
- moved C19 28.1 mm to (182.9, 77.6)
- moved R10 27.2 mm to (172.2, 109.7)
- moved R18 24.6 mm to (167.0, 104.5), turned to 180 degrees
- moved C15 23.7 mm to (184.0, 99.8), turned to 0 degrees
- moved C3 19.4 mm to (163.6, 94.0), turned to 90 degrees
- moved U8 17.2 mm to (167.8, 97.5), turned to 90 degrees
- moved C1 16.6 mm to (172.0, 95.0), turned to -90 degrees
- moved C14 15.2 mm to (175.0, 87.1), turned to 90 degrees
- moved D4 14.2 mm to (171.9, 82.5), turned to 90 degrees
- moved C12 13.1 mm to (175.5, 103.1), turned to 90 degrees
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Routing:
- net 24VDC: track 161.0 -> 51.0 mm, vias 2 -> 17
- net Net-(D5-K): track 97.7 -> 33.9 mm
- net Net-(U8A--): track 70.3 -> 20.2 mm, vias 1 -> 0
- net Net-(R17-Pad2): track 53.4 -> 9.67 mm, vias 1 -> 0
- net /D6: track 77.6 -> 35.9 mm, vias 4 -> 2
- net /D5: track 75.7 -> 34.2 mm, vias 4 -> 2
- net /Drivers/Lamp-GND: track 49.5 -> 9.65 mm, vias 1 -> 0
- net Net-(U8A-+): track 55.4 -> 27.6 mm, vias 1 -> 0
- net Net-(U3-OUT): track 47.0 -> 25.2 mm, vias 4 -> 2
- net Net-(C15-Pad1): track 90.8 -> 106.4 mm, vias 1 -> 0
- net Net-(D4-K): track 39.4 -> 51.5 mm
- net Net-(D10-A): track 146.0 -> 152.8 mm
- net 3.3V-uC: track 50.2 -> 56.9 mm
- net Net-(U6-K): track 26.1 -> 32.3 mm, vias 3 -> 0
- net GND: track 136.8 -> 141.8 mm, vias 83 -> 78
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- added copper zone on In2.Cu, net 24VDC
- removed copper zone on F.Cu, net 24VDC
