File: scan-controller/scan-controller-kicad/drivers.kicad_sch (KiCad schematic)
At the start: 53 parts, among them CN2 Motor, CN3 Fan, CN4 Lamp, Q1 CS12N06AE-G, U10 LGS5145, U11 MCP1416, U3 78L05, U4 DRV8871DDA, U6 TL431, U7 XL4015, U8 LM358

Commit message: R8 -> 1K
Parts:
- R8: value 10R -> 1K; LCSC C17415 -> C17513
Changed lines of the file:
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@@
 			)
 		)
-		(property "Value" "10R"
+		(property "Value" "1K"
 			(at 173.355 58.42 0)
 			(effects
@@
 			)
 		)
-		(property "LCSC" "C17415"
+		(property "LCSC" "C17513"
 			(at 169.545 59.055 0)
 			(effects

Commit message: Add C31 to U9 to form another low pass
Parts:
- added C30: 100n, Capacitor_SMD:C_0805_2012Metric, symbol Device:C_Small
Connections:
- net GNDD: now also C30.1
- net at Q1.4 (G), R8.1, R9.1: now also C30.2
Other:
- moved on the sheet: C1, C12, C14, C15, C16, C19, C2, C28, C29, C3, CN4, D4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

Commit message: reassigned customfootprints to now gobal library
Parts:
- TP14, TP15, TP16, TP17, TP18, TP9: footprint Peacemans_Footprints:TestPoint_THTPad_1.5x1.5mm_Drill0.7mm_named -> Peacemans_Teile:TestPoint_THTPad_1.5x1.5mm_Drill0.7mm_named
Changed lines of the file:
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@@
 			)
 		)
-		(property "Footprint" "Peacemans_Footprints:TestPoint_THTPad_1.5x1.5mm_Drill0.7mm_named"
+		(property "Footprint" "Peacemans_Teile:TestPoint_THTPad_1.5x1.5mm_Drill0.7mm_named"
 			(at 227.965 134.62 0)
 			(effects
@@
 			)
 		)
-		(property "Footprint" "Peacemans_Footprints:TestPoint_THTPad_1.5x1.5mm_Drill0.7mm_named"
+		(property "Footprint" "Peacemans_Teile:TestPoint_THTPad_1.5x1.5mm_Drill0.7mm_named"
 			(at 258.445 34.925 0)
 			(effects
@@
 			)
 		)
-		(property "Footprint" "Peacemans_Footprints:TestPoint_THTPad_1.5x1.5mm_Drill0.7mm_named"
+		(property "Footprint" "Peacemans_Teile:TestPoint_THTPad_1.5x1.5mm_Drill0.7mm_named"
 			(at 197.485 83.82 0)
 			(effects
@@
 			)
 		)
-		(property "Footprint" "Peacemans_Footprints:TestPoint_THTPad_1.5x1.5mm_Drill0.7mm_named"
+		(property "Footprint" "Peacemans_Teile:TestPoint_THTPad_1.5x1.5mm_Drill0.7mm_named"
 			(at 266.065 53.34 0)
 			(effects
@@
 			)
 		)
-		(property "Footprint" "Peacemans_Footprints:TestPoint_THTPad_1.5x1.5mm_Drill0.7mm_named"
+		(property "Footprint" "Peacemans_Teile:TestPoint_THTPad_1.5x1.5mm_Drill0.7mm_named"
 			(at 267.335 34.925 0)
 			(effects
@@
 			)
 		)
-		(property "Footprint" "Peacemans_Footprints:TestPoint_THTPad_1.5x1.5mm_Drill0.7mm_named"
+		(property "Footprint" "Peacemans_Teile:TestPoint_THTPad_1.5x1.5mm_Drill0.7mm_named"
 			(at 228.6 116.205 0)
 			(effects

Commit message: Massive rearrangement :)
Other:
- moved on the sheet: CN3
Changed lines of the file:
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@@
 	)
 	(junction
-		(at 227.965 123.19)
+		(at 237.49 46.355)
 		(diameter 0)
 		(color 0 0 0 0)
 	)
 	(junction
-		(at 237.49 46.355)
+		(at 182.245 83.82)
 		(diameter 0)
 		(color 0 0 0 0)
 	)
 	(junction
-		(at 182.245 83.82)
+		(at 193.675 83.82)
 		(diameter 0)
 		(color 0 0 0 0)
 	)
 	(junction
-		(at 193.675 83.82)
+		(at 228.6 129.54)
 		(diameter 0)
 		(color 0 0 0 0)
@@
 	)
 	(junction
-		(at 227.965 129.54)
-		(diameter 0)
-		(color 0 0 0 0)
-	)
-	(junction
 		(at 208.915 118.11)
 		(diameter 0)
@@
 	)
 	(junction
-		(at 227.965 118.11)
+		(at 219.075 139.7)
 		(diameter 0)
 		(color 0 0 0 0)
 	)
 	(junction
-		(at 219.075 139.7)
+		(at 170.18 76.2)
 		(diameter 0)
 		(color 0 0 0 0)
 	)
 	(junction
-		(at 170.18 76.2)
+		(at 228.6 118.11)
 		(diameter 0)
 		(color 0 0 0 0)
 	)
 	(no_connect
-		(at 227.965 120.65)
+		(at 231.14 120.65)
 	)
 	(wire
@@
 	(wire
 		(pts
+			(xy 231.14 118.11) (xy 228.6 118.11)
+		)
+		(stroke
+			(width 0)
+			(type default)
+		)
+	)
+	(wire
+		(pts
 			(xy 166.37 60.325) (xy 165.735 60.325)
 		)
@@
 	(wire
 		(pts
-			(xy 227.965 111.125) (xy 227.965 118.11)
+			(xy 228.6 111.76) (xy 228.6 118.11)
 		)
 		(stroke
@@
 	(wire
 		(pts
-			(xy 226.06 118.11) (xy 227.965 118.11)
+			(xy 226.06 118.11) (xy 228.6 118.11)
 		)
 		(stroke
@@
 	(wire
 		(pts
-			(xy 227.965 123.19) (xy 227.965 129.54)
-		)
-		(stroke
-			(width 0)
-			(type default)
-		)
-	)
-	(wire
-		(pts
 			(xy 147.955 40.64) (xy 147.955 39.37)
 		)
@@
 	(wire
 		(pts
-			(xy 227.965 122.555) (xy 227.965 123.19)
+			(xy 228.6 123.19) (xy 228.6 129.54)
 		)
 		(stroke
@@
 	(wire
 		(pts
-			(xy 227.965 129.54) (xy 227.965 139.7)
+			(xy 228.6 129.54) (xy 228.6 139.7)
 		)
 		(stroke
@@
 	(wire
 		(pts
-			(xy 228.6 111.125) (xy 227.965 111.125)
-		)
-		(stroke
-			(width 0)
-			(type default)
-		)
-	)
-	(wire
-		(pts
 			(xy 177.8 83.82) (xy 182.245 83.82)
 		)
@@
 	(wire
 		(pts
-			(xy 227.965 139.7) (xy 219.075 139.7)
+			(xy 228.6 139.7) (xy 219.075 139.7)
 		)
 		(stroke
@@
 	(wire
 		(pts
+			(xy 228.6 123.19) (xy 231.14 123.19)
+		)
+		(stroke
+			(width 0)
+			(type default)
+		)
+	)
+	(wire
+		(pts
 			(xy 250.825 43.815) (xy 250.825 48.26)
 		)
@@
 	(symbol
 		(lib_id "easyeda2kicad:KF141R-2.54-3P")
-		(at 233.045 120.65 0)
+		(at 236.22 120.65 0)
 		(mirror x)
 		(unit 1)
@@
 		(dnp no)
 		(property "Reference" "CN3"
-			(at 231.775 127 0)
+			(at 234.95 127 0)
 			(effects
 				(font
@@
 		)
 		(property "Value" "Fan"
-			(at 232.41 114.3 0)
+			(at 235.585 114.3 0)
 			(effects
 				(font
@@
 		)
 		(property "Footprint" "easyeda2kicad:CONN-TH_3P-P2.54_DIBO_DB141R-2.54-3P"
-			(at 233.045 110.49 0)
+			(at 236.22 110.49 0)
 			(effects
 				(font
@@
 		)
 		(property "Datasheet" "https://lcsc.com/product-detail/New-Quadratic-Unclassified-Data_Cixi-Kefa-Elec-KF141R-2-54-3P_C475125.html"
-			(at 233.045 107.95 0)
+			(at 236.22 107.95 0)
 			(effects
 				(font
@@
 		)
 		(property "Description" ""
-			(at 233.045 120.65 0)
+			(at 236.22 120.65 0)
 			(effects
 				(font
@@
 		)
 		(property "LCSC Part" ""
-			(at 233.045 105.41 0)
+			(at 236.22 105.41 0)
 			(effects
 				(font
@@
 		)
 		(property "LCSC" "C2898755"
-			(at 233.045 120.65 0)
+			(at 236.22 120.65 0)
 			(effects
 				(font
@@
 		)
 		(property "Inventory" ""
-			(at 233.045 120.65 0)
+			(at 236.22 120.65 0)
 			(effects
 				(font
@@
 		)
 		(property "Sim.Device" "C475125"
-			(at 233.045 120.65 0)
+			(at 236.22 120.65 0)
 			(effects
 				(font
@@
 	(symbol
 		(lib_id "Peacemans_Teile:TestPoint_named")
-		(at 227.965 129.54 270)
+		(at 228.6 129.54 270)
 		(unit 1)
 		(exclude_from_sim no)
@@
 		(dnp no)
 		(property "Reference" "TP17"
-			(at 234.823 129.54 0)
+			(at 235.458 129.54 0)
 			(effects
 				(font
@@
 		)
 		(property "Value" "TestPoint"
-			(at 233.045 129.54 0)
+			(at 233.68 129.54 0)
 			(effects
 				(font
@@
 		)
 		(property "Footprint" "Peacemans_Teile:TestPoint_THTPad_1.5x1.5mm_Drill0.7mm_named"
-			(at 227.965 134.62 0)
+			(at 228.6 134.62 0)
 			(effects
 				(font
@@
 		)
 		(property "Datasheet" "~"
-			(at 227.965 134.62 0)
+			(at 228.6 134.62 0)
 			(effects
 				(font
@@
 		)
 		(property "Description" ""
-			(at 227.965 129.54 0)
+			(at 228.6 129.54 0)
 			(effects
 				(font
@@
 		)
 		(property "TP_Label" "Fan -"
-			(at 233.045 131.445 90)
+			(at 233.68 131.445 90)
 			(effects
 				(font
 					(size 1.27 1.27)
 				)
+				(hide yes)
 			)
 		)
@@
 	(symbol
 		(lib_id "Peacemans_Teile:TestPoint_named")
-		(at 228.6 111.125 270)
+		(at 228.6 111.76 270)
 		(unit 1)
 		(exclude_from_sim no)
@@
 		(dnp no)
 		(property "Reference" "TP18"
-			(at 235.458 111.125 0)
+			(at 235.458 111.76 0)
 			(effects
 				(font
@@
 		)
 		(property "Value" "TestPoint"
-			(at 233.68 111.125 0)
+			(at 233.68 111.76 0)
 			(effects
 				(font
@@
 		)
 		(property "Footprint" "Peacemans_Teile:TestPoint_THTPad_1.5x1.5mm_Drill0.7mm_named"
-			(at 228.6 116.205 0)
+			(at 228.6 116.84 0)
 			(effects
 				(font
@@
 		)
 		(property "Datasheet" "~"
-			(at 228.6 116.205 0)
+			(at 228.6 116.84 0)
 			(effects
 				(font
@@
 		)
 		(property "Description" ""
-			(at 228.6 111.125 0)
+			(at 228.6 111.76 0)
 			(effects
 				(font
@@
 		)
 		(property "TP_Label" "Fan +"
-			(at 232.918 109.093 90)
+			(at 232.918 109.728 90)
 			(effects
 				(font
 					(size 1.27 1.27)
 				)
+				(hide yes)
 			)
 		)

Commit message: DRC mostly happy
Parts:
- removed TP17, TP18: TestPoint, Peacemans_Teile:TestPoint_THTPad_1.5x1.5mm_Drill0.7mm_named, symbol Peacemans_Teile:TestPoint_named
Changed lines of the file:
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@@
 	)
 	(junction
-		(at 228.6 129.54)
-		(diameter 0)
-		(color 0 0 0 0)
-	)
-	(junction
 		(at 156.21 83.82)
 		(diameter 0)
@@
 		(color 0 0 0 0)
 	)
-	(junction
-		(at 228.6 118.11)
-		(diameter 0)
-		(color 0 0 0 0)
-	)
 	(no_connect
 		(at 231.14 120.65)
@@
 	(wire
 		(pts
-			(xy 231.14 118.11) (xy 228.6 118.11)
+			(xy 226.06 118.11) (xy 231.14 118.11)
 		)
 		(stroke
@@
 	(wire
 		(pts
-			(xy 228.6 111.76) (xy 228.6 118.11)
-		)
-		(stroke
-			(width 0)
-			(type default)
-		)
-	)
-	(wire
-		(pts
 			(xy 198.755 130.81) (xy 198.755 132.715)
 		)
@@
 	(wire
 		(pts
-			(xy 226.06 118.11) (xy 228.6 118.11)
-		)
-		(stroke
-			(width 0)
-			(type default)
-		)
-	)
-	(wire
-		(pts
 			(xy 182.245 78.105) (xy 182.245 83.82)
 		)
@@
 	(wire
 		(pts
-			(xy 228.6 123.19) (xy 228.6 129.54)
-		)
-		(stroke
-			(width 0)
-			(type default)
-		)
-	)
-	(wire
-		(pts
 			(xy 246.38 94.615) (xy 246.38 99.06)
 		)
@@
 	(wire
 		(pts
-			(xy 228.6 129.54) (xy 228.6 139.7)
+			(xy 228.6 123.19) (xy 228.6 139.7)
 		)
 		(stroke
@@
 	(symbol
 		(lib_id "Peacemans_Teile:TestPoint_named")
-		(at 228.6 129.54 270)
-		(unit 1)
-		(exclude_from_sim no)
-		(in_bom yes)
-		(on_board yes)
-		(dnp no)
-		(property "Reference" "TP17"
-			(at 235.458 129.54 0)
-			(effects
-				(font
-					(size 1.27 1.27)
-				)
-				(hide yes)
-			)
-		)
-		(property "Value" "TestPoint"
-			(at 233.68 129.54 0)
-			(effects
-				(font
-					(size 1.27 1.27)
-				)
-				(hide yes)
-			)
-		)
-		(property "Footprint" "Peacemans_Teile:TestPoint_THTPad_1.5x1.5mm_Drill0.7mm_named"
-			(at 228.6 134.62 0)
-			(effects
-				(font
-					(size 1.27 1.27)
-				)
-				(hide yes)
-			)
-		)
-		(property "Datasheet" "~"
-			(at 228.6 134.62 0)
-			(effects
-				(font
-					(size 1.27 1.27)
-				)
-				(hide yes)
-			)
-		)
-		(property "Description" ""
-			(at 228.6 129.54 0)
-			(effects
-				(font
-					(size 1.27 1.27)
-				)
-				(hide yes)
-			)
-		)
-		(property "TP_Label" "Fan -"
-			(at 233.68 131.445 90)
-			(effects
-				(font
-					(size 1.27 1.27)
-				)
-				(hide yes)
-			)
-		)
-		(pin "1"
-		)
-		(instances
-			(project "scan-controller-kicad"
-				(path "/ab6dbce1-4ecf-44ae-8f33-5f07e4f43ca9/f199f7c1-4da9-41da-ae5e-c136f90f6de6"
-					(reference "TP17")
-					(unit 1)
-				)
-			)
-		)
-	)
-	(symbol
-		(lib_id "Peacemans_Teile:TestPoint_named")
 		(at 253.365 34.925 0)
 		(unit 1)
@@
 					(unit 1)
 				)
-			)
-		)
-	)
-	(symbol
-		(lib_id "Peacemans_Teile:TestPoint_named")
-		(at 228.6 111.76 270)
-		(unit 1)
-		(exclude_from_sim no)
-		(in_bom yes)
-		(on_board yes)
-		(dnp no)
-		(property "Reference" "TP18"
-			(at 235.458 111.76 0)
-			(effects
-				(font
-					(size 1.27 1.27)
-				)
-				(hide yes)
-			)
-		)
-		(property "Value" "TestPoint"
-			(at 233.68 111.76 0)
-			(effects
-				(font
-					(size 1.27 1.27)
-				)
-				(hide yes)
-			)
-		)
-		(property "Footprint" "Peacemans_Teile:TestPoint_THTPad_1.5x1.5mm_Drill0.7mm_named"
-			(at 228.6 116.84 0)
-			(effects
-				(font
-					(size 1.27 1.27)
-				)
-				(hide yes)
-			)
-		)
-		(property "Datasheet" "~"
-			(at 228.6 116.84 0)
-			(effects
-				(font
-					(size 1.27 1.27)
-				)
-				(hide yes)
-			)
-		)
-		(property "Description" ""
-			(at 228.6 111.76 0)
-			(effects
-				(font
-					(size 1.27 1.27)
-				)
-				(hide yes)
-			)
-		)
-		(property "TP_Label" "Fan +"
-			(at 232.918 109.728 90)
-			(effects
-				(font
-					(size 1.27 1.27)
-				)
-				(hide yes)
-			)
-		)
-		(pin "1"
-		)
-		(instances
-			(project "scan-controller-kicad"
-				(path "/ab6dbce1-4ecf-44ae-8f33-5f07e4f43ca9/f199f7c1-4da9-41da-ae5e-c136f90f6de6"
-					(reference "TP18")
-					(unit 1)
-				)

Commit message: Major refactoring to better EMV in progress
Parts:
- added C33: 1u, Capacitor_SMD:C_0805_2012Metric, symbol Device:C_Small
- added R46, R47: 10K, Resistor_SMD:R_1206_3216Metric, symbol Device:R_Small
- C2: value 470u -> 220u; LCSC C90272 -> (none)
Connections:
- net 24VDC: now also C33.1, R46.2
- net GNDD: now also R46.1
- net Lamp-GND: no longer C1.2, C12.2, C15.2, C19.2, C2.2, C3.2, D4.2 (A), Q1.5 (D), Q1.6 (D), Q1.7 (D), Q1.8 (D), R16.2, R18.1, RV1.3, TP9.1, U3.2 (GND), U6.3 (A), U7.1 (GND), U8.4 (V-)
- net at C15.1, C19.1, CN4.3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: now also R47.2
- new net: C1.2, C12.2, C15.2, C19.2, C2.2, C3.2, C33.2, D4.2 (A), Q1.5 (D), Q1.6 (D), Q1.7 (D), Q1.8 (D), R16.2, R18.1, R47.1, RV1.3, TP9.1, U3.2 (GND), U6.3 (A), U7.1 (GND), U8.4 (V-)
Other:
- note added: "Bleeder (against GNDD to not pull drain up)"
- note added: "Move to switch post buck"
- note added: "Snubber von SW nach GND: SW-RC-GND. C = 680p bis 2.2n C0G oder X7R, >100 V R = 4.7 bis 22, 0.25W 1n/10 probieren"
- note added: "Wenn dauerversorgt nach Q1 move, In mit 47k Pulldown versehen 100R Serie als EMI Schutz"
- moved on the sheet: C1, C12, C14, C15, C16, C19, C2, C25, C26, C27, C28, C29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

Commit message: Refactored LED Driver: Switch behind the buck, reduce EMV
Parts:
- removed C29: 100n, Capacitor_SMD:C_0805_2012Metric, symbol Device:C_Small
- added C34: 1n, Capacitor_SMD:C_0805_2012Metric, symbol Device:C_Small
- added R48: 100K, Resistor_SMD:R_0805_2012Metric, symbol Device:R_Small
- added R49: 47K, Resistor_SMD:R_0805_2012Metric, symbol Device:R_Small
Connections:
- net GNDD: now also C1.2, C12.2, C15.2, C19.2, C2.2, C3.2, C33.2, D4.2 (A), R16.2, R18.1, R47.1, RV1.3, U3.2 (GND), U6.3 (A), U7.1 (GND), U8.4 (V-), R49.2; no longer Q1.1 (S), Q1.2 (S), Q1.3 (S)
- net Lamp: now also R49.1
- net at R18.2, U8.3 (+): now also Q1.1 (S), Q1.2 (S), Q1.3 (S), C34.1, R48.2; no longer CN4.1, TP14.1
- new net: C34.2, CN4.1, Q1.5 (D), Q1.6 (D), Q1.7 (D), Q1.8 (D), R48.1, TP14.1
- now unconnected: TP9.1
Other:
- note removed: "Bleeder (against GNDD to not pull drain up)"
- note removed: "Move to switch post buck"
- note removed: "Snubber von SW nach GND: SW-RC-GND. C = 680p bis 2.2n C0G oder X7R, >100 V R = 4.7 bis 22, 0.25W 1n/10 probieren"
- note removed: "Wenn dauerversorgt nach Q1 move, In mit 47k Pulldown versehen 100R Serie als EMI Schutz"
- moved on the sheet: C1, C12, C14, C15, C16, C17, C18, C19, C2, C28, C3, C30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
