File: scan-controller/scan-controller-kicad/drivers.kicad_sch (KiCad schematic)
At the start: 56 parts, among them CN2 Motor, CN3 Fan, CN4 Lamp, Q1 CS12N06AE-G, U10 LGS5145, U11 MCP1416, U3 NH6375A50P, U4 DRV8871DDA, U6 TL431, U7 XL4015, U8 LM358

Commit message: Rev.E
Co-authored-by: Cursor <cursoragent@cursor.com>
Parts:
- D9: LCSC C2687553 -> C52146084; LCSC Part (none) -> C2687553
Changed lines of the file:
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@@
 			)
 		)
-		(property "LCSC" "C2687553"
+		(property "LCSC" "C52146084"
 			(at 107.95 166.37 0)
 			(effects
 				(font
+					(size 1.27 1.27)
+				)
+				(hide yes)
+			)
+		)
+		(property "LCSC Part" "C2687553"
+			(at 107.95 166.37 90)
+			(effects
+				(font
