File: scan-controller/scan-controller-kicad/scan-controller-kicad.kicad_sch (KiCad schematic)
At the start: 36 parts, among them CN1 24V in, J1 FTDI, J5 ICSP, J6 Raspi UART, J7 Raspi GPIO, Q2 IRLML2502, Q3 IRLML6402, SW3 Reset, U5 ATmega328P, Y1 8MHz

Commit message: Switching back to Rev-B (newer Displays have their outputs on the left hand side)
Parts:
- removed R41: 47K, Resistor_SMD:R_0805_2012Metric, symbol Device:R_Small
Other:
- note added: "eKamerakabel-Schlitz? Target Schalter größer? FTDI Masse kennzeichnen Exp/Current prüfen KSQ LEDs nötig? Shaft LED als Einbauhilfe Taster durch SMD ersetzen"
- note removed: "FTDI Pins kennzeichnen R platzieren Extra GND"
- moved on the sheet: Q2, Q3, R14, R15, R33

Commit message: Initial Rev.C work
Parts:
- added R41: 47K, Resistor_SMD:R_0805_2012Metric, symbol Device:R_Small
Connections:
- net 24VDC: now also R41.2
- net GND: now also R41.1
Other:
- note added: "UART Pins kennzeichnen Shaft LED platzieren PCB nach oben erweitern Rev D Reset Taster verlegen"
- note removed: "eKamerakabel-Schlitz? Target Schalter größer? FTDI Masse kennzeichnen Exp/Current prüfen KSQ LEDs nötig? Shaft LED als Einbauhilfe Taster durch SMD ersetzen"
Changed lines of the file:
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@@
   (junction (at 93.98 145.415) (diameter 0) (color 0 0 0 0)
   )
+  (junction (at 57.15 23.495) (diameter 0) (color 0 0 0 0)
+  )
   (junction (at 108.585 89.535) (diameter 0) (color 0 0 0 0)
   )
@@
   (junction (at 164.465 92.71) (diameter 0) (color 0 0 0 0)
   )
-  (junction (at 54.61 41.275) (diameter 0) (color 0 0 0 0)
+  (junction (at 61.595 41.275) (diameter 0) (color 0 0 0 0)
   )
   (junction (at 108.585 94.615) (diameter 0) (color 0 0 0 0)
@@
   )
   (junction (at 188.595 66.04) (diameter 0) (color 0 0 0 0)
+  )
+  (junction (at 57.15 41.275) (diameter 0) (color 0 0 0 0)
   )
   (junction (at 164.465 97.79) (diameter 0) (color 0 0 0 0)
@@
     (stroke (width 0) (type default))
   )
-  (wire (pts (xy 54.61 41.275) (xy 57.15 41.275))
+  (wire (pts (xy 61.595 41.275) (xy 64.135 41.275))
     (stroke (width 0) (type default))
   )
@@
     (stroke (width 0) (type default))
   )
+  (wire (pts (xy 57.15 23.495) (xy 57.15 28.575))
+    (stroke (width 0) (type default))
+  )
   (wire (pts (xy 205.105 82.55) (xy 203.835 82.55))
     (stroke (width 0) (type default))
@@
     (stroke (width 0) (type default))
   )
-  (wire (pts (xy 48.26 23.495) (xy 49.53 23.495))
+  (wire (pts (xy 48.26 23.495) (xy 57.15 23.495))
     (stroke (width 0) (type default))
   )
@@
     (stroke (width 0) (type default))
   )
+  (wire (pts (xy 48.26 41.275) (xy 57.15 41.275))
+    (stroke (width 0) (type default))
+  )
   (wire (pts (xy 85.725 97.155) (xy 86.995 97.155))
     (stroke (width 0) (type default))
@@
     (stroke (width 0) (type default))
   )
-  (wire (pts (xy 54.61 41.275) (xy 48.26 41.275))
-    (stroke (width 0) (type default))
-  )
   (wire (pts (xy 120.015 95.25) (xy 120.015 94.615))
     (stroke (width 0) (type default))
@@
     (stroke (width 0) (type default))
   )
+  (wire (pts (xy 57.15 23.495) (xy 62.23 23.495))
+    (stroke (width 0) (type default))
+  )
   (wire (pts (xy 85.725 130.175) (xy 95.885 130.175))
     (stroke (width 0) (type default))
@@
     (stroke (width 0) (type default))
   )
-  (wire (pts (xy 57.15 41.275) (xy 57.15 42.545))
+  (wire (pts (xy 64.135 41.275) (xy 64.135 42.545))
     (stroke (width 0) (type default))
   )
@@
     (stroke (width 0) (type default))
   )
+  (wire (pts (xy 57.15 41.275) (xy 61.595 41.275))
+    (stroke (width 0) (type default))
+  )
   (wire (pts (xy 132.715 64.135) (xy 132.715 69.85))
     (stroke (width 0) (type default))
@@
   )
   (wire (pts (xy 108.585 135.255) (xy 110.49 135.255))
+    (stroke (width 0) (type default))
+  )
+  (wire (pts (xy 57.15 33.655) (xy 57.15 41.275))
     (stroke (width 0) (type default))
   )
@@
     (effects (font (size 1 1)) (justify left bottom))
   )
-  (text "eKamerakabel-Schlitz?\nTarget Schalter größer?\nFTDI Masse kennzeichnen\nExp/Current prüfen\nKSQ LEDs nötig?\nShaft LED als Einbauhilfe\nTaster durch SMD ersetzen"
-    (at 59.69 189.865 0)
+  (text "UART Pins kennzeichnen\nShaft LED platzieren\nPCB nach oben erweitern\nRev D\nReset Taster verlegen"
+    (at 208.915 34.29 0)
     (effects (font (size 1.27 1.27)) (justify left bottom))
   )
-  (label "GNDD" (at 57.15 42.545 0) (fields_autoplaced)
+  (label "GNDD" (at 64.135 42.545 0) (fields_autoplaced)
     (effects (font (size 1.27 1.27)) (justify left bottom))
   )
@@
     )
   )
-  (global_label "24VDC" (shape input) (at 49.53 23.495 0) (fields_autoplaced)
+  (global_label "24VDC" (shape input) (at 62.23 23.495 0) (fields_autoplaced)
     (effects (font (size 1.27 1.27)) (justify left))
-    (property "Intersheetrefs" "${INTERSHEET_REFS}" (at 58.5628 23.495 0)
+    (property "Intersheetrefs" "${INTERSHEET_REFS}" (at 71.2628 23.495 0)
       (effects (font (size 1.27 1.27)) (justify left) hide)
     )
@@
     )
   )
+  (symbol (lib_id "Device:R_Small") (at 57.15 31.115 180) (unit 1)
+    (in_bom yes) (on_board yes) (dnp no)
+    (property "Reference" "R41" (at 60.325 29.845 0)
+      (effects (font (size 1.27 1.27)))
+    )
+    (property "Value" "47K" (at 60.325 32.385 0)
+      (effects (font (size 1.27 1.27)))
+    )
+    (property "Footprint" "Resistor_SMD:R_0805_2012Metric" (at 57.15 31.115 0)
+      (effects (font (size 1.27 1.27)) hide)
+    )
+    (property "Datasheet" "~" (at 57.15 31.115 0)
+      (effects (font (size 1.27 1.27)) hide)
+    )
+    (property "LCSC" "C17713" (at 57.15 31.115 0)
+      (effects (font (size 1.27 1.27)) hide)
+    )
+    (property "Inventory" "B" (at 57.15 31.115 0)
+      (effects (font (size 1.27 1.27)) hide)
+    )
+    (pin "1")
+    (pin "2")
+    (instances
+      (project "scan-controller-kicad"
+        (path "/ab6dbce1-4ecf-44ae-8f33-5f07e4f43ca9"
+          (reference "R41") (unit 1)
+        )
+      )
+    )
+  )
   (symbol (lib_id "Device:R_Small") (at 121.285 59.055 90) (unit 1)
     (in_bom yes) (on_board yes) (dnp no)
@@
     )
   )
-  (symbol (lib_id "power:GNDD") (at 65.405 43.18 0) (unit 1)
-    (in_bom yes) (on_board yes) (dnp no)
-    (property "Reference" "#PWR03" (at 65.405 49.53 0)
-      (effects (font (size 1.27 1.27)) hide)
-    )
-    (property "Value" "GNDD" (at 65.405 46.99 0)
-      (effects (font (size 1.27 1.27)))
-    )
-    (property "Footprint" "" (at 65.405 43.18 0)
-      (effects (font (size 1.27 1.27)) hide)
-    )
-    (property "Datasheet" "" (at 65.405 43.18 0)
+  (symbol (lib_id "power:GNDD") (at 72.39 43.18 0) (unit 1)
+    (in_bom yes) (on_board yes) (dnp no)
+    (property "Reference" "#PWR03" (at 72.39 49.53 0)
+      (effects (font (size 1.27 1.27)) hide)
+    )
+    (property "Value" "GNDD" (at 72.39 46.99 0)
+      (effects (font (size 1.27 1.27)))
+    )
+    (property "Footprint" "" (at 72.39 43.18 0)
+      (effects (font (size 1.27 1.27)) hide)
+    )
+    (property "Datasheet" "" (at 72.39 43.18 0)
       (effects (font (size 1.27 1.27)) hide)
     )
@@
     )
   )
-  (symbol (lib_id "power:PWR_FLAG") (at 65.405 43.18 0) (unit 1)
+  (symbol (lib_id "power:PWR_FLAG") (at 72.39 43.18 0) (unit 1)
     (in_bom yes) (on_board yes) (dnp no) (fields_autoplaced)
-    (property "Reference" "#FLG02" (at 65.405 41.275 0)
-      (effects (font (size 1.27 1.27)) hide)
-    )
-    (property "Value" "PWR_FLAG" (at 65.405 38.735 0)
-      (effects (font (size 1.27 1.27)) hide)
-    )
-    (property "Footprint" "" (at 65.405 43.18 0)
-      (effects (font (size 1.27 1.27)) hide)
-    )
-    (property "Datasheet" "~" (at 65.405 43.18 0)
+    (property "Reference" "#FLG02" (at 72.39 41.275 0)
+      (effects (font (size 1.27 1.27)) hide)
+    )
+    (property "Value" "PWR_FLAG" (at 72.39 38.735 0)
+      (effects (font (size 1.27 1.27)) hide)
+    )
+    (property "Footprint" "" (at 72.39 43.18 0)
+      (effects (font (size 1.27 1.27)) hide)
+    )
+    (property "Datasheet" "~" (at 72.39 43.18 0)
       (effects (font (size 1.27 1.27)) hide)
     )
@@
     )
   )
-  (symbol (lib_id "Peacemans_Teile:TestPoint_named") (at 54.61 41.275 180) (unit 1)
-    (in_bom yes) (on_board yes) (dnp no)
-    (property "Reference" "TP2" (at 55.88 49.53 0)
+  (symbol (lib_id "Peacemans_Teile:TestPoint_named") (at 61.595 41.275 180) (unit 1)
+    (in_bom yes) (on_board yes) (dnp no)
+    (property "Reference" "TP2" (at 62.865 49.53 0)
       (effects (font (size 1.27 1.27)) (justify left) hide)
     )
-    (property "Value" "GND" (at 56.515 46.99 0)
+    (property "Value" "GND" (at 63.5 46.99 0)
       (effects (font (size 1.27 1.27)) (justify left))
     )
-    (property "Footprint" "Peacemans_Footprints:TestPoint_THTPad_1.5x1.5mm_Drill0.7mm_named" (at 49.53 41.275 0)
-      (effects (font (size 1.27 1.27)) hide)
-    )
-    (property "Datasheet" "~" (at 49.53 41.275 0)
-      (effects (font (size 1.27 1.27)) hide)
-    )
-    (property "TP_Label" "GND" (at 54.61 41.275 0)
-      (effects (font (size 1.27 1.27)))
-    )
+    (property "Footprint" "Peacemans_Footprints:TestPoint_THTPad_1.5x1.5mm_Drill0.7mm_named" (at 56.515 41.275 0)
+      (effects (font (size 1.27 1.27)) hide)
+    )
+    (property "Datasheet" "~" (at 56.515 41.275 0)
+      (effects (font (size 1.27 1.27)) hide)
+    )
+    (property "TP_Label" "GND" (at 61.595 41.275 0)
+      (effects (font (size 1.27 1.27)))
+    )

Commit message: Extend the board and improve usability
Other:
- note added: "UART Pins kennzeichnen Shaft LED platzieren PCB nach oben erweitern Rev D Reset Taster verlegen Better 5V Source?"
- note removed: "UART Pins kennzeichnen Shaft LED platzieren PCB nach oben erweitern Rev D Reset Taster verlegen"
Changed lines of the file:
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@@
     (effects (font (size 1 1)) (justify left bottom))
   )
-  (text "UART Pins kennzeichnen\nShaft LED platzieren\nPCB nach oben erweitern\nRev D\nReset Taster verlegen"
+  (text "UART Pins kennzeichnen\nShaft LED platzieren\nPCB nach oben erweitern\nRev D\nReset Taster verlegen\nBetter 5V Source?"
     (at 208.915 34.29 0)
     (effects (font (size 1.27 1.27)) (justify left bottom))

Commit message: Looking good, just the new 5VDC source is missing
Other:
- note added: "Create a Better 5V Source?"
- note removed: "UART Pins kennzeichnen Shaft LED platzieren PCB nach oben erweitern Rev D Reset Taster verlegen Better 5V Source?"
Changed lines of the file:
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@@
     (effects (font (size 1 1)) (justify left bottom))
   )
-  (text "UART Pins kennzeichnen\nShaft LED platzieren\nPCB nach oben erweitern\nRev D\nReset Taster verlegen\nBetter 5V Source?"
-    (at 208.915 34.29 0)
+  (text "Create a Better 5V Source?" (at 208.915 34.29 0)
     (effects (font (size 1.27 1.27)) (justify left bottom))
   )

Commit message: Adding a Gate Driver and making the MOSFET tougher. DRC happy!
Other:
- note removed: "Create a Better 5V Source?"
Changed lines of the file:
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@@
     (effects (font (size 1 1)) (justify left bottom))
-  )
-  (text "Create a Better 5V Source?" (at 208.915 34.29 0)
-    (effects (font (size 1.27 1.27)) (justify left bottom))
   )
   (label "GNDD" (at 64.135 42.545 0) (fields_autoplaced)

Commit message: minor layout tweaks, todos
Other:
- note added: "Todo: - RV6 Label Pos - Backside text (Fan Power) - Projector background (zonefill) - C2/4 Zonefill - Name: Filmkorn-Raw-Scanner"
Changed lines of the file:
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@@
     (effects (font (size 1 1)) (justify left bottom))
+  )
+  (text "Todo:\n- RV6 Label Pos\n- Backside text (Fan Power)\n- Projector background (zonefill)\n- C2/4 Zonefill\n- Name: Filmkorn-Raw-Scanner\n"
+    (at 201.93 29.845 0)
+    (effects (font (size 1.27 1.27)) (justify left bottom))
   )
   (label "GNDD" (at 64.135 42.545 0) (fields_autoplaced)

Commit message: Cosmetic PCB Changes (not in sync with netlist yet)
Other:
- note removed: "Todo: - RV6 Label Pos - Backside text (Fan Power) - Projector background (zonefill) - C2/4 Zonefill - Name: Filmkorn-Raw-Scanner"
Changed lines of the file:
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@@
     (effects (font (size 1 1)) (justify left bottom))
-  )
-  (text "Todo:\n- RV6 Label Pos\n- Backside text (Fan Power)\n- Projector background (zonefill)\n- C2/4 Zonefill\n- Name: Filmkorn-Raw-Scanner\n"
-    (at 201.93 29.845 0)
-    (effects (font (size 1.27 1.27)) (justify left bottom))
   )
   (label "GNDD" (at 64.135 42.545 0) (fields_autoplaced)
