File: scan-controller/scan-controller-kicad/scan-controller-kicad.kicad_sch (KiCad schematic)
At the start: 38 parts, among them CN1 24V in, J1 FTDI, J5 ICSP, J6 Raspi UART, J7 Raspi GPIO, Q2 IRLML2502, Q3 IRLML6402, SW3 Reset, U5 ATmega328P, Y1 8MHz

Commit message: Rev.E
Co-authored-by: Cursor <cursoragent@cursor.com>
Parts:
- J7: now left out of the parts list
- R51: LCSC C17414 -> C17477
Changed lines of the file:
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@@
 		(unit 1)
 		(exclude_from_sim no)
-		(in_bom yes)
+		(in_bom no)
 		(on_board yes)
 		(dnp no)
@@
 			)
 		)
-		(property "LCSC" "C17414"
+		(property "LCSC" "C17477"
 			(at 234.95 80.01 0)
 			(effects
