File: scan-controller/scan-controller-kicad/userinterface.kicad_sch (KiCad schematic)
At the start: 29 parts, among them J4 Target, SW1 Power, SW10 >>, SW11 Rec, SW2 Target, SW4 Lamp, SW5 <<, SW6 Zoom, SW7 Stop, SW8 <, SW9 >

Commit message: Switching back to Rev-B (newer Displays have their outputs on the left hand side)
Other:
- moved on the sheet: C13, D1, J4, R13, R2, R21, R23, R25, R28, R32, R35, R37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

Commit message: Routing WIP
Parts:
- RV4, RV5: footprint easyeda2kicad:RES-TH_RK09K1110A0J -> easyeda2kicad:RES-TH_RK09K1110A0J_short
Changed lines of the file:
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@@
       (effects (font (size 1.27 1.27)) (justify right))
     )
-    (property "Footprint" "easyeda2kicad:RES-TH_RK09K1110A0J" (at 163.195 112.395 0)
+    (property "Footprint" "easyeda2kicad:RES-TH_RK09K1110A0J_short" (at 163.195 112.395 0)
       (effects (font (size 1.27 1.27)) hide)
     )
@@
       (effects (font (size 1.27 1.27)) (justify right))
     )
-    (property "Footprint" "easyeda2kicad:RES-TH_RK09K1110A0J" (at 180.975 119.38 0)
-      (effects (font (size 1.27 1.27)) hide)
-    )
+    (property "Footprint" "easyeda2kicad:RES-TH_RK09K1110A0J_short" (at 180.975 119.38 0)
+      (effects (font (size 1.27 1.27)) hide)
+    )

Commit message: Cosmetic PCB Changes (not in sync with netlist yet)
Connections:
- net 3.3V-uC: now also RV4.3, RV5.3; no longer RV4.1, RV5.1
- net GNDD: now also RV4.1, RV5.1; no longer RV4.3, RV5.3
Changed lines of the file:
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@@
     )
   )
-  (symbol (lib_id "Device:R_Potentiometer_Small") (at 163.195 112.395 0) (unit 1)
-    (in_bom yes) (on_board yes) (dnp no)
-    (property "Reference" "RV5" (at 167.64 115.57 0)
+  (symbol (lib_id "Device:R_Potentiometer_Small") (at 163.195 112.395 0) (mirror x) (unit 1)
+    (in_bom yes) (on_board yes) (dnp no)
+    (property "Reference" "RV5" (at 167.64 109.22 0)
       (effects (font (size 1.27 1.27)) (justify right))
     )
@@
     )
   )
-  (symbol (lib_id "Device:R_Potentiometer_Small") (at 180.975 119.38 0) (unit 1)
-    (in_bom yes) (on_board yes) (dnp no)
-    (property "Reference" "RV4" (at 185.42 122.555 0)
+  (symbol (lib_id "Device:R_Potentiometer_Small") (at 180.975 119.38 0) (mirror x) (unit 1)
+    (in_bom yes) (on_board yes) (dnp no)
+    (property "Reference" "RV4" (at 185.42 116.205 0)
       (effects (font (size 1.27 1.27)) (justify right))
     )
