File: scan-controller/scan-controller-kicad/userinterface.kicad_sch (KiCad schematic)
At the start: 29 parts, among them J4 Target, SW1 Power, SW10 >>, SW11 Rec, SW2 Target, SW4 Lamp, SW5 <<, SW6 Zoom, SW7 Stop, SW8 <, SW9 >

Commit message: Raspi Power LED
Parts:
- added D11: Raspi Power, LED_SMD:LED_0805_2012Metric, symbol Device:LED_Small
- added R38: 3K3, Resistor_SMD:R_0805_2012Metric, symbol Device:R_Small
Connections:
- net GNDD: now also D11.1 (K)
- new net: D11.2 (A), R38.1
- new net 3.3V-RPi: R38.2
Other:
- moved on the sheet: C13, D1, R7

Commit message: R2/R4 -> 10K
Parts:
- R2, R4: value 47K -> 10K; LCSC C17713 -> C17414
Changed lines of the file:
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@@
 			)
 		)
-		(property "Value" "47K"
+		(property "Value" "10K"
 			(at 163.195 52.07 0)
 			(effects
@@
 			)
 		)
-		(property "LCSC" "C17713"
+		(property "LCSC" "C17414"
 			(at 168.91 50.165 0)
 			(effects
@@
 			)
 		)
-		(property "Value" "47K"
+		(property "Value" "10K"
 			(at 163.195 35.56 0)
 			(effects
@@
 			)
 		)
-		(property "LCSC" "C17713"
+		(property "LCSC" "C17414"
 			(at 168.91 33.655 0)
 			(effects

Commit message: Rename Target Switch to Resolution, add actual Target Switch
Parts:
- added J8: Target, Connector_PinHeader_2.54mm:PinHeader_1x03_P2.54mm_Vertical, symbol Connector_Generic:Conn_01x03
- added R44, R45: 10K, Resistor_SMD:R_0805_2012Metric, symbol Device:R_Small
- added SW12: Target, easyeda2kicad:SW-SMD_3P-P1.50_L2.7-W6.6, symbol Switch:SW_SPDT
- J4, SW2: value Target -> Resolution
Connections:
- net 3.3V-uC: now also J8.3 (Pin_3), R44.1
- net GNDD: now also J8.1 (Pin_1), R45.2
- net Storage Target renamed Resolution
- new net: R44.2, SW12.1 (A)
- new net: R45.1, SW12.3 (C)
- new net Target: J8.2 (Pin_2), SW12.2 (B)
Other:
- moved on the sheet: J4, R2, R4, SW2

Commit message: Initial 4 plane version
Parts:
- SW12: footprint easyeda2kicad:SW-SMD_3P-P1.50_L2.7-W6.6 -> easyeda2kicad:SW-TH_SS-12F23-G040; LCSC C319020 -> C17179527
- SW2: footprint easyeda2kicad:SW-SMD_3P-P1.50_L2.7-W6.6 -> easyeda2kicad:SW-TH_5P-P4.70_SS-12D11-G040; LCSC C319020 -> C17179527
Changed lines of the file:
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@@
 			)
 		)
-		(property "Footprint" "easyeda2kicad:SW-SMD_3P-P1.50_L2.7-W6.6"
-			(at 221.615 41.275 0)
-			(effects
-				(font
-					(size 1.27 1.27)
-				)
-				(hide yes)
-			)
-		)
-		(property "Datasheet" "https://datasheet.lcsc.com/lcsc/2110151630_XKB-Connectivity-SK-3296S-01-L1_C319020.pdf"
+		(property "Footprint" "easyeda2kicad:SW-TH_SS-12F23-G040"
+			(at 221.615 41.275 0)
+			(effects
+				(font
+					(size 1.27 1.27)
+				)
+				(hide yes)
+			)
+		)
+		(property "Datasheet" "https://jlcpcb.com/api/file/downloadByFileSystemAccessId/8602925046717968384"
 			(at 221.615 41.275 0)
 			(effects
@@
 			)
 		)
-		(property "LCSC" "C319020"
+		(property "LCSC" "C17179527"
 			(at 221.615 41.275 0)
 			(effects
@@
 			)
 		)
-		(property "Footprint" "easyeda2kicad:SW-SMD_3P-P1.50_L2.7-W6.6"
-			(at 174.625 41.275 0)
-			(effects
-				(font
-					(size 1.27 1.27)
-				)
-				(hide yes)
-			)
-		)
-		(property "Datasheet" "https://datasheet.lcsc.com/lcsc/2110151630_XKB-Connectivity-SK-3296S-01-L1_C319020.pdf"
+		(property "Footprint" "easyeda2kicad:SW-TH_5P-P4.70_SS-12D11-G040"
+			(at 174.625 41.275 0)
+			(effects
+				(font
+					(size 1.27 1.27)
+				)
+				(hide yes)
+			)
+		)
+		(property "Datasheet" "https://jlcpcb.com/api/file/downloadByFileSystemAccessId/8602925046717968384"
 			(at 174.625 41.275 0)
 			(effects
@@
 			)
 		)
-		(property "LCSC" "C319020"
-			(at 174.625 41.275 0)
-			(effects
+		(property "LCSC" "C17179527"
+			(at 174.625 41.275 0)
+			(effects

Commit message: Massive rearrangement :)
Parts:
- SW12: footprint easyeda2kicad:SW-TH_SS-12F23-G040 -> easyeda2kicad:SW-TH_5P-P4.70_SS-12D11-G040
Changed lines of the file:
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@@
 			)
 		)
-		(property "Footprint" "easyeda2kicad:SW-TH_SS-12F23-G040"
+		(property "Footprint" "easyeda2kicad:SW-TH_5P-P4.70_SS-12D11-G040"
 			(at 221.615 41.275 0)
 			(effects

Commit message: Massive LampGND
Parts:
- added H1, H2, H3, H4: MountingHole, MountingHole_3.2mm_M3_Pad_Via, symbol Mechanical:MountingHole

Commit message: Major refactoring to better EMV in progress
Parts:
- H1, H2, H3, H4: footprint MountingHole_3.2mm_M3_Pad_Via -> MountingHole:MountingHole_3.2mm_M3_Pad_Via
Changed lines of the file:
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@@
 			)
 		)
-		(property "Footprint" "MountingHole_3.2mm_M3_Pad_Via"
+		(property "Footprint" "MountingHole:MountingHole_3.2mm_M3_Pad_Via"
 			(at 266.7 144.78 0)
 			(effects
@@
 			)
 		)
-		(property "Footprint" "MountingHole_3.2mm_M3_Pad_Via"
+		(property "Footprint" "MountingHole:MountingHole_3.2mm_M3_Pad_Via"
 			(at 266.7 160.02 0)
 			(effects
@@
 			)
 		)
-		(property "Footprint" "MountingHole_3.2mm_M3_Pad_Via"
+		(property "Footprint" "MountingHole:MountingHole_3.2mm_M3_Pad_Via"
 			(at 266.7 149.86 0)
 			(effects
@@
 			)
 		)
-		(property "Footprint" "MountingHole_3.2mm_M3_Pad_Via"
+		(property "Footprint" "MountingHole:MountingHole_3.2mm_M3_Pad_Via"
 			(at 266.7 154.94 0)
 			(effects
