File: scan-controller/scan-controller-kicad/userinterface.kicad_sch (KiCad schematic)
At the start: 39 parts, among them J4 Resolution, J8 Target, SW1 Power, SW10 >>, SW11 Rec, SW12 Target, SW2 Resolution, SW4 Lamp, SW5 <<, SW6 Zoom, SW7 Stop, SW8 <, SW9 >

Commit message: ERC happy!
Parts:
- SW10, SW11, SW4, SW5, SW6, SW7, SW8, SW9: LCSC Part (none) -> C93156
Other:
- moved on the sheet: J4, J8, R13, R2, R21, R23, R25, R28, R32, R35, R37, R39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
