File: scan-controller/scan-controller-kicad/userinterface.kicad_sch (KiCad schematic)
At the start: 39 parts, among them J4 Resolution, J8 Target, SW1 Power, SW10 >>, SW11 Rec, SW12 Target, SW2 Resolution, SW4 Lamp, SW5 <<, SW6 Zoom, SW7 Stop, SW8 <, SW9 >

Commit message: Rev.E
Co-authored-by: Cursor <cursoragent@cursor.com>
Parts:
- R38: value 3K3 -> 300R; LCSC C26010 -> C17617
Changed lines of the file:
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@@
 			)
 		)
-		(property "Value" "3K3"
+		(property "Value" "300R"
 			(at 208.28 68.58 90)
 			(effects
@@
 			)
 		)
-		(property "LCSC" "C26010"
+		(property "LCSC" "C17617"
 			(at 210.82 71.12 0)
 			(effects
