File: scan-controller/scan-controller-kicad/ZVD.kicad_sch (KiCad schematic)
At the start: 4 parts, among them Q4 DMG2305UX, Q7 DMMT5401

Commit message: ERC happy!
Other:
- moved on the sheet: Q4, Q7A, Q7B, R34, R36
