File: scan-controller/scan-controller-kicad/sensors.kicad_sch (KiCad schematic)
At the start: 28 parts, among them CN5 Film End Eye, CN6 Shaft Eye, J2 Shaft Eye, J3 Film End Eye, Q5 SS8050, Q6 SS8050, U1 QRE1113, U2 QRE1113, U9 74LVC14

Commit message: Add C31 to U9 to form another low pass
Parts:
- added C31: 100n, Capacitor_SMD:C_0805_2012Metric, symbol Device:C_Small
Connections:
- net GNDD: now also C31.2
- net at Q6.3 (C), R30.1, R31.2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: now also C31.1
Other:
- moved on the sheet: C22, CN5, D3, Q6, R11, R27, R30, R31, TP3, U9C, U9D

Commit message: reassigned customfootprints to now gobal library
Parts:
- R1, R3, R5, R6: footprint Peacemans_Footprints:R_0402_1005Metric-noref -> Peacemans_Teile:R_0402_1005Metric-noref
- TP10, TP3: footprint Peacemans_Footprints:TestPoint_THTPad_1.5x1.5mm_Drill0.7mm_named -> Peacemans_Teile:TestPoint_THTPad_1.5x1.5mm_Drill0.7mm_named
- U1, U2: footprint Peacemans_Footprints:QRE1113GR-slim -> Peacemans_Teile:QRE1113GR-slim
Changed lines of the file:
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@@
 			)
 		)
-		(property "Footprint" "Peacemans_Footprints:R_0402_1005Metric-noref"
+		(property "Footprint" "Peacemans_Teile:R_0402_1005Metric-noref"
 			(at 107.315 114.3 0)
 			(effects
@@
 			)
 		)
-		(property "Footprint" "Peacemans_Footprints:QRE1113GR-slim"
+		(property "Footprint" "Peacemans_Teile:QRE1113GR-slim"
 			(at 98.425 81.28 0)
 			(effects
@@
 			)
 		)
-		(property "Footprint" "Peacemans_Footprints:TestPoint_THTPad_1.5x1.5mm_Drill0.7mm_named"
+		(property "Footprint" "Peacemans_Teile:TestPoint_THTPad_1.5x1.5mm_Drill0.7mm_named"
 			(at 171.45 121.285 0)
 			(effects
@@
 			)
 		)
-		(property "Footprint" "Peacemans_Footprints:QRE1113GR-slim"
+		(property "Footprint" "Peacemans_Teile:QRE1113GR-slim"
 			(at 99.695 127 0)
 			(effects
@@
 			)
 		)
-		(property "Footprint" "Peacemans_Footprints:R_0402_1005Metric-noref"
+		(property "Footprint" "Peacemans_Teile:R_0402_1005Metric-noref"
 			(at 90.805 68.58 0)
 			(effects
@@
 			)
 		)
-		(property "Footprint" "Peacemans_Footprints:R_0402_1005Metric-noref"
+		(property "Footprint" "Peacemans_Teile:R_0402_1005Metric-noref"
 			(at 106.045 68.58 0)
 			(effects
@@
 			)
 		)
-		(property "Footprint" "Peacemans_Footprints:R_0402_1005Metric-noref"
+		(property "Footprint" "Peacemans_Teile:R_0402_1005Metric-noref"
 			(at 92.075 114.3 0)
 			(effects
@@
 			)
 		)
-		(property "Footprint" "Peacemans_Footprints:TestPoint_THTPad_1.5x1.5mm_Drill0.7mm_named"
+		(property "Footprint" "Peacemans_Teile:TestPoint_THTPad_1.5x1.5mm_Drill0.7mm_named"
 			(at 170.18 75.565 0)
 			(effects

Commit message: Remove Pin numbers from mechanical pins, add unplaced U9 units as NC
Parts:
- added unit 5 of U9
- added unit 6 of U9
- U9: Inventory E -> (none); LCSC C6065 -> (none)
Connections:
- no-connect marks 0 -> 6
Changed lines of the file:
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@@
 		(color 0 0 0 0)
 	)
+	(no_connect
+		(at 45.72 151.13)
+	)
+	(no_connect
+		(at 72.39 116.84)
+	)
+	(no_connect
+		(at 38.1 88.9)
+	)
+	(no_connect
+		(at 60.96 135.89)
+	)
+	(no_connect
+		(at 45.72 135.89)
+	)
+	(no_connect
+		(at 60.96 151.13)
+	)
 	(wire
 		(pts
@@
 			)
 		)
-		(property "Datasheet" "https://datasheet.lcsc.com/lcsc/2304140030_Nexperia-74LVC14AD-118_C6065.pdf"
-			(at 50.8 97.79 0)
-			(effects
-				(font
-					(size 1.27 1.27)
-				)
-				(hide yes)
-			)
-		)
-		(property "Description" ""
-			(at 50.8 97.79 0)
-			(effects
-				(font
-					(size 1.27 1.27)
-				)
-				(hide yes)
-			)
-		)
-		(property "LCSC" "C6065"
+		(property "Datasheet" "http://www.ti.com/lit/gpn/sn74HC14"
 			(at 50.8 97.79 0)
 			(effects
@@
 			)
 		)
-		(property "Inventory" "E"
+		(property "Description" "Hex inverter schmitt trigger"
 			(at 50.8 97.79 0)
 			(effects
@@
 			)
 		)
-		(property "Datasheet" "https://datasheet.lcsc.com/lcsc/2304140030_Nexperia-74LVC14AD-118_C6065.pdf"
+		(property "Datasheet" "http://www.ti.com/lit/gpn/sn74HC14"
 			(at 167.64 73.66 0)
 			(effects
@@
 			)
 		)
-		(property "Description" ""
-			(at 167.64 73.66 0)
-			(effects
-				(font
-					(size 1.27 1.27)
-				)
-				(hide yes)
-			)
-		)
-		(property "LCSC" "C6065"
-			(at 167.64 73.66 0)
-			(effects
-				(font
-					(size 1.27 1.27)
-				)
-				(hide yes)
-			)
-		)
-		(property "Inventory" "E"
+		(property "Description" "Hex inverter schmitt trigger"
 			(at 167.64 73.66 0)
 			(effects
@@
 	)
 	(symbol
+		(lib_id "74xx:74HC14")
+		(at 53.34 135.89 0)
+		(unit 5)
+		(exclude_from_sim no)
+		(in_bom yes)
+		(on_board yes)
+		(dnp no)
+		(fields_autoplaced yes)
+		(property "Reference" "U9"
+			(at 53.34 127 0)
+			(effects
+				(font
+					(size 1.27 1.27)
+				)
+			)
+		)
+		(property "Value" "74LVC14"
+			(at 53.34 129.54 0)
+			(effects
+				(font
+					(size 1.27 1.27)
+				)
+			)
+		)
+		(property "Footprint" "Package_SO:SOIC-14_3.9x8.7mm_P1.27mm"
+			(at 53.34 135.89 0)
+			(effects
+				(font
+					(size 1.27 1.27)
+				)
+				(hide yes)
+			)
+		)
+		(property "Datasheet" "http://www.ti.com/lit/gpn/sn74HC14"
+			(at 53.34 135.89 0)
+			(effects
+				(font
+					(size 1.27 1.27)
+				)
+				(hide yes)
+			)
+		)
+		(property "Description" "Hex inverter schmitt trigger"
+			(at 53.34 135.89 0)
+			(effects
+				(font
+					(size 1.27 1.27)
+				)
+				(hide yes)
+			)
+		)
+		(pin "8"
+		)
+		(pin "7"
+		)
+		(pin "1"
+		)
+		(pin "9"
+		)
+		(pin "5"
+		)
+		(pin "6"
+		)
+		(pin "4"
+		)
+		(pin "3"
+		)
+		(pin "10"
+		)
+		(pin "14"
+		)
+		(pin "2"
+		)
+		(pin "12"
+		)
+		(pin "11"
+		)
+		(pin "13"
+		)
+		(instances
+			(project ""
+				(path "/ab6dbce1-4ecf-44ae-8f33-5f07e4f43ca9/32afee9c-f78c-4810-b9e6-48288995c3da"
+					(reference "U9")
+					(unit 5)
+				)
+			)
+		)
+	)
+	(symbol
 		(lib_id "Peacemans_Teile:R_Small_0402-noref")
 		(at 107.315 114.3 0)
@@
 			)
 		)
-		(property "Datasheet" "https://datasheet.lcsc.com/lcsc/2304140030_Nexperia-74LVC14AD-118_C6065.pdf"
-			(at 168.91 119.38 0)
-			(effects
-				(font
-					(size 1.27 1.27)
-				)
-				(hide yes)
-			)
-		)
-		(property "Description" ""
-			(at 168.91 119.38 0)
-			(effects
-				(font
-					(size 1.27 1.27)
-				)
-				(hide yes)
-			)
-		)
-		(property "LCSC" "C6065"
+		(property "Datasheet" "http://www.ti.com/lit/gpn/sn74HC14"
 			(at 168.91 119.38 0)
 			(effects
@@
 			)
 		)
-		(property "Inventory" "E"
+		(property "Description" "Hex inverter schmitt trigger"
 			(at 168.91 119.38 0)
 			(effects
@@
 			)
 		)
-		(property "Datasheet" "https://datasheet.lcsc.com/lcsc/2304140030_Nexperia-74LVC14AD-118_C6065.pdf"
-			(at 191.77 73.66 0)
-			(effects
-				(font
-					(size 1.27 1.27)
-				)
-				(hide yes)
-			)
-		)
-		(property "Description" ""
-			(at 191.77 73.66 0)
-			(effects
-				(font
-					(size 1.27 1.27)
-				)
-				(hide yes)
-			)
-		)
-		(property "LCSC" "C6065"
+		(property "Datasheet" "http://www.ti.com/lit/gpn/sn74HC14"
 			(at 191.77 73.66 0)
 			(effects
@@
 			)
 		)
-		(property "Inventory" "E"
+		(property "Description" "Hex inverter schmitt trigger"
 			(at 191.77 73.66 0)
 			(effects
@@
 	)
 	(symbol
+		(lib_id "74xx:74HC14")
+		(at 53.34 151.13 0)
+		(unit 6)
+		(exclude_from_sim no)
+		(in_bom yes)
+		(on_board yes)
+		(dnp no)
+		(fields_autoplaced yes)
+		(property "Reference" "U9"
+			(at 53.34 142.24 0)
+			(effects
+				(font
+					(size 1.27 1.27)
+				)
+			)
+		)
+		(property "Value" "74LVC14"
+			(at 53.34 144.78 0)
+			(effects
+				(font
+					(size 1.27 1.27)
+				)
+			)
+		)
+		(property "Footprint" "Package_SO:SOIC-14_3.9x8.7mm_P1.27mm"
+			(at 53.34 151.13 0)
+			(effects
+				(font
+					(size 1.27 1.27)
+				)
+				(hide yes)
+			)
+		)
+		(property "Datasheet" "http://www.ti.com/lit/gpn/sn74HC14"
+			(at 53.34 151.13 0)
+			(effects
+				(font
+					(size 1.27 1.27)
+				)
+				(hide yes)
+			)
+		)
+		(property "Description" "Hex inverter schmitt trigger"
+			(at 53.34 151.13 0)
+			(effects
+				(font
+					(size 1.27 1.27)
+				)
+				(hide yes)
+			)
+		)
+		(pin "8"
+		)
+		(pin "7"
+		)
+		(pin "1"
+		)
+		(pin "9"
+		)
+		(pin "5"
+		)
+		(pin "6"
+		)
+		(pin "4"
+		)
+		(pin "3"
+		)
+		(pin "10"
+		)
+		(pin "14"
+		)
+		(pin "2"
+		)
+		(pin "12"
+		)
+		(pin "11"
+		)
+		(pin "13"
+		)
+		(instances
+			(project ""
+				(path "/ab6dbce1-4ecf-44ae-8f33-5f07e4f43ca9/32afee9c-f78c-4810-b9e6-48288995c3da"
+					(reference "U9")
+					(unit 6)
+				)
+			)
+		)
+	)
+	(symbol
 		(lib_id "Peacemans_Teile:R_Small_0402-noref")
 		(at 92.075 114.3 0)
@@
 			)
 		)
-		(property "Datasheet" "https://datasheet.lcsc.com/lcsc/2304140030_Nexperia-74LVC14AD-118_C6065.pdf"
+		(property "Datasheet" "http://www.ti.com/lit/gpn/sn74HC14"
 			(at 193.04 119.38 0)
 			(effects
@@
 			)
 		)
-		(property "Description" ""
-			(at 193.04 119.38 0)
-			(effects
-				(font
-					(size 1.27 1.27)
-				)
-				(hide yes)
-			)
-		)
-		(property "LCSC" "C6065"
-			(at 193.04 119.38 0)
-			(effects
-				(font
-					(size 1.27 1.27)
-				)
-				(hide yes)
-			)
-		)
-		(property "Inventory" "E"
+		(property "Description" "Hex inverter schmitt trigger"
 			(at 193.04 119.38 0)
 			(effects

Commit message: Bigger Ears, DRc not quite happy yet
Parts:
- R1, R6: footprint Peacemans_Teile:R_0402_1005Metric-noref -> Resistor_SMD:R_0603_1608Metric; LCSC C25792 -> C25819
- R3, R5: footprint Peacemans_Teile:R_0402_1005Metric-noref -> Resistor_SMD:R_0603_1608Metric; LCSC C25076 -> C22775
Changed lines of the file:
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@@
 			)
 		)
-		(property "Footprint" "Peacemans_Teile:R_0402_1005Metric-noref"
+		(property "Footprint" "Resistor_SMD:R_0603_1608Metric"
 			(at 107.315 114.3 0)
 			(effects
@@
 			)
 		)
-		(property "LCSC" "C25792"
+		(property "LCSC" "C25819"
 			(at 107.315 114.3 0)
 			(effects
@@
 			)
 		)
-		(property "Footprint" "Peacemans_Teile:R_0402_1005Metric-noref"
+		(property "Footprint" "Resistor_SMD:R_0603_1608Metric"
 			(at 90.805 68.58 0)
 			(effects
@@
 			)
 		)
-		(property "LCSC" "C25076"
+		(property "LCSC" "C22775"
 			(at 90.805 68.58 0)
 			(effects
@@
 			)
 		)
-		(property "Footprint" "Peacemans_Teile:R_0402_1005Metric-noref"
+		(property "Footprint" "Resistor_SMD:R_0603_1608Metric"
 			(at 106.045 68.58 0)
 			(effects
@@
 			)
 		)
-		(property "LCSC" "C25792"
+		(property "LCSC" "C25819"
 			(at 106.045 68.58 0)
 			(effects
@@
 			)
 		)
-		(property "Footprint" "Peacemans_Teile:R_0402_1005Metric-noref"
+		(property "Footprint" "Resistor_SMD:R_0603_1608Metric"
 			(at 92.075 114.3 0)
 			(effects
@@
 			)
 		)
-		(property "LCSC" "C25076"
+		(property "LCSC" "C22775"
 			(at 92.075 114.3 0)
 			(effects

Commit message: ERC happy!
Parts:
- U1, U2: footprint Peacemans_Teile:QRE1113GR-slim -> OptoDevice:OnSemi_CASE100AQ
Connections:
- no-connect marks 6 -> 4
Other:
- moved on the sheet: C21, J2, J3, R1, R11, R29, R3, R5, R6, TP10, TP3, U1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
