File: scan-controller/scan-controller-kicad/sensors.kicad_sch (KiCad schematic)
At the start: 29 parts, among them CN5 Film End Eye, CN6 Shaft Eye, J2 Shaft Eye, J3 Film End Eye, Q5 SS8050, Q6 SS8050, U1 QRE1113, U2 QRE1113, U9 74LVC14

Commit message: Merge tracks
Parts:
- U1, U2: footprint OptoDevice:OnSemi_CASE100AQ -> easyeda2kicad:OPTO-SMD_QRE1113GR
Changed lines of the file:
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@@
 			)
 		)
-		(property "Footprint" "OptoDevice:OnSemi_CASE100AQ"
+		(property "Footprint" "easyeda2kicad:OPTO-SMD_QRE1113GR"
 			(at 99.06 81.28 0)
 			(effects
@@
 			)
 		)
-		(property "Footprint" "OptoDevice:OnSemi_CASE100AQ"
+		(property "Footprint" "easyeda2kicad:OPTO-SMD_QRE1113GR"
 			(at 100.33 127 0)
 			(effects
